Commit message: Fix hand controller

File: kortex_description/grippers/robotiq_2f_85/urdf/robotiq_kortex.ros2_control.xacro (robot description, xacro)
@@ -17,16 +17,9 @@
         </xacro:unless>
       </hardware>
-      <joint name="robotiq_85_left_knuckle_joint">
-        <command_interface name="position">
-          <param name="min">0</param>
-          <param name="max">1.0</param>
-        </command_interface>
-        <command_interface name="velocity">
-          <param name="min">-2.0/param>
-          <param name="max">2.0</param>
-        </command_interface>
-        <state_interface name="position"/>
-        <state_interface name="velocity"/>
-        <state_interface name="effort"/>
+      <joint name="${prefix}finger_joint">
+          <param name="initial_position">0.0</param>
+          <command_interface name="position" />
+          <state_interface name="position"/>
+          <state_interface name="velocity"/>
       </joint>
     </ros2_control>
