Commit message: Have the gripper opening

File: kortex_description/grippers/robotiq_2f_85/urdf/robotiq_arg2f_85_model_macro.xacro (robot description, xacro)
@@ -166,5 +166,5 @@
       <child link="${prefix}left_outer_knuckle" />
       <axis xyz="1 0 0" />
-      <limit lower="0" upper="0.8" velocity="2.0" effort="1000" />
+      <limit lower="0" upper="100" velocity="2.0" effort="1000" />
     </joint>
     <xacro:finger_joints prefix="${prefix}" fingerprefix="left" reflect="1.0"/>

Commit message: Updated the config so that it's range is 0 - 100

File: kortex_description/grippers/robotiq_2f_85/urdf/robotiq_arg2f_85_model_macro.xacro (robot description, xacro)
@@ -137,5 +137,5 @@
       <child link="${prefix}${fingerprefix}_inner_knuckle" />
       <axis xyz="1 0 0" />
-      <limit lower="0" upper="0.8757" velocity="2.0" effort="1000" />
+      <limit lower="0" upper="100.0" velocity="2.0" effort="1000" />
       <mimic joint="${prefix}finger_joint" multiplier="1" offset="0" />
     </joint>
@@ -147,5 +147,5 @@
       <child link="${prefix}${fingerprefix}_inner_finger" />
       <axis xyz="1 0 0" />
-      <limit lower="-0.8757" upper="0.8757" velocity="2.0" effort="1000" />
+      <limit lower="-100.0" upper="100.0" velocity="2.0" effort="1000" />
       <mimic joint="${prefix}finger_joint" multiplier="-1" offset="0" />
     </joint>
@@ -176,5 +176,5 @@
       <child link="${prefix}right_outer_knuckle" />
       <axis xyz="1 0 0" />
-      <limit lower="0" upper="0.81" velocity="2.0" effort="1000" />
+      <limit lower="0" upper="100" velocity="2.0" effort="1000" />
       <mimic joint="${prefix}finger_joint" multiplier="1" offset="0" />
     </joint>

Commit message: Added an action server for the gripper (#14)
* Fixed a error with an arg

* Updated the name of open / close gripper group to be the same as the Ur5

* Added hand_controller to movit controllers.yaml

* Added a gripper driver for the 85 gripper

* cleanup some code

* Have the gripper opening

* Updated the srdf so that open / close are the correct value

* Updated the config so that it's range is 0 - 100

* Working gripper action server

* Working gripper action server

* Removed an unused comment

* Updated the copy write

* linting

* linting

* removed un-used testing files

* swapped the open / close the other way around

File: kortex_description/grippers/robotiq_2f_85/urdf/robotiq_arg2f_85_model_macro.xacro (robot description, xacro)
@@ -137,5 +137,5 @@
       <child link="${prefix}${fingerprefix}_inner_knuckle" />
       <axis xyz="1 0 0" />
-      <limit lower="0" upper="0.8757" velocity="2.0" effort="1000" />
+      <limit lower="0" upper="100.0" velocity="2.0" effort="1000" />
       <mimic joint="${prefix}finger_joint" multiplier="1" offset="0" />
     </joint>
@@ -147,5 +147,5 @@
       <child link="${prefix}${fingerprefix}_inner_finger" />
       <axis xyz="1 0 0" />
-      <limit lower="-0.8757" upper="0.8757" velocity="2.0" effort="1000" />
+      <limit lower="-100.0" upper="100.0" velocity="2.0" effort="1000" />
       <mimic joint="${prefix}finger_joint" multiplier="-1" offset="0" />
     </joint>
@@ -166,5 +166,5 @@
       <child link="${prefix}left_outer_knuckle" />
       <axis xyz="1 0 0" />
-      <limit lower="0" upper="0.8" velocity="2.0" effort="1000" />
+      <limit lower="0" upper="100" velocity="2.0" effort="1000" />
     </joint>
     <xacro:finger_joints prefix="${prefix}" fingerprefix="left" reflect="1.0"/>
@@ -176,5 +176,5 @@
       <child link="${prefix}right_outer_knuckle" />
       <axis xyz="1 0 0" />
-      <limit lower="0" upper="0.81" velocity="2.0" effort="1000" />
+      <limit lower="0" upper="100" velocity="2.0" effort="1000" />
       <mimic joint="${prefix}finger_joint" multiplier="1" offset="0" />
     </joint>

Commit message: Fixed the gripper bug where it never successed

File: kortex_description/grippers/robotiq_2f_85/urdf/robotiq_arg2f_85_model_macro.xacro (robot description, xacro)
@@ -137,5 +137,5 @@
       <child link="${prefix}${fingerprefix}_inner_knuckle" />
       <axis xyz="1 0 0" />
-      <limit lower="0" upper="100.0" velocity="2.0" effort="1000" />
+      <limit lower="0" upper="0.8" velocity="2.0" effort="1000" />
       <mimic joint="${prefix}finger_joint" multiplier="1" offset="0" />
     </joint>
@@ -147,5 +147,5 @@
       <child link="${prefix}${fingerprefix}_inner_finger" />
       <axis xyz="1 0 0" />
-      <limit lower="-100.0" upper="100.0" velocity="2.0" effort="1000" />
+      <limit lower="-0.8" upper="0.8" velocity="2.0" effort="1000" />
       <mimic joint="${prefix}finger_joint" multiplier="-1" offset="0" />
     </joint>
@@ -166,5 +166,5 @@
       <child link="${prefix}left_outer_knuckle" />
       <axis xyz="1 0 0" />
-      <limit lower="0" upper="100" velocity="2.0" effort="1000" />
+      <limit lower="0" upper="0.8" velocity="2.0" effort="1000" />
     </joint>
     <xacro:finger_joints prefix="${prefix}" fingerprefix="left" reflect="1.0"/>
@@ -176,5 +176,5 @@
       <child link="${prefix}right_outer_knuckle" />
       <axis xyz="1 0 0" />
-      <limit lower="0" upper="100" velocity="2.0" effort="1000" />
+      <limit lower="0" upper="0.8" velocity="2.0" effort="1000" />
       <mimic joint="${prefix}finger_joint" multiplier="1" offset="0" />
     </joint>
