Commit message: Revert "Merge pull request #1 from PickNikRobotics/pr-robotiq_driver"
This reverts commit 77d7e71b6cc7eea06eccff2cbcf3862cfbd5f2df, reversing
changes made to 5ed5a8d1dde4ffadd0132043c894c1832153da47.

File: kortex_description/grippers/robotiq_2f_85/urdf/robotiq_2f_85_macro.xacro (robot description, xacro)
@@ -4,12 +4,4 @@
     <xacro:include filename="$(find kortex_description)/grippers/robotiq_2f_85/urdf/robotiq_arg2f_85_model_macro.xacro" />
     <xacro:robotiq_arg2f_85 parent="${parent}" prefix="${prefix}"/>
-    <!-- ros2 control include -->
-    <xacro:include filename="$(find kortex_description)/grippers/robotiq_2f_85/urdf/robotiq_kortex.ros2_control.xacro" />
-    <xacro:robotiq_kortex_ros2_control
-      name="KortexGripperInterfaceHardware" prefix="${prefix}"
-      use_fake_hardware="${use_fake_hardware}"
-      fake_sensor_commands="${fake_sensor_commands}"
-      tf_prefix=""
-      robot_ip="${robot_ip}" />
   </xacro:macro>
 </robot>

File: kortex_move_it_config/gen3_robotiq_2f_85_move_it_config/config/7dof/gen3_robotiq_2f_85.srdf.xacro (robot description, xacro)
@@ -6,9 +6,9 @@
 <robot name="gen3_robotiq_2f_85" xmlns:xacro="http://www.ros.org/wiki/xacro">
     <xacro:arg name="prefix" default="" />
-    <!--GROUPS - Representation of a set of joints and links. This can be useful for specifying DOF to plan for, defining arms, end effectors, etc-->
-    <!--LINKS - When a link is specified, the parent joint of that link (if it exists) is automatically included-->
-    <!--JOINTS - When a joint is specified, the child link of that joint (which will always exist) is automatically included-->
-    <!--CHAINS - When a chain is specified, all the links along the chain (including endpoints) are included in the group. Additionally, all the joints that are parents to included links are also included. This means that joints along the chain and the parent joint of the base link are included in the group-->
-    <!--SUBGROUPS - Groups can also be formed by referencing to already defined group names-->
+    <!--GROUPS: Representation of a set of joints and links. This can be useful for specifying DOF to plan for, defining arms, end effectors, etc-->
+    <!--LINKS: When a link is specified, the parent joint of that link (if it exists) is automatically included-->
+    <!--JOINTS: When a joint is specified, the child link of that joint (which will always exist) is automatically included-->
+    <!--CHAINS: When a chain is specified, all the links along the chain (including endpoints) are included in the group. Additionally, all the joints that are parents to included links are also included. This means that joints along the chain and the parent joint of the base link are included in the group-->
+    <!--SUBGROUPS: Groups can also be formed by referencing to already defined group names-->
     <group name="arm">
         <joint name="$(arg prefix)joint_1" />
@@ -35,5 +35,5 @@
         <joint name="$(arg prefix)right_inner_finger_pad_joint" />
     </group>
-    <!--GROUP STATES - Purpose - Define a named state for a particular group, in terms of joint values. This is useful to define states like 'folded arms'-->
+    <!--GROUP STATES: Purpose: Define a named state for a particular group, in terms of joint values. This is useful to define states like 'folded arms'-->
     <group_state name="home" group="arm">
         <joint name="$(arg prefix)joint_1" value="0" />
@@ -72,5 +72,5 @@
     </group_state>
     <group_state name="closed" group="gripper">
-        <joint name="$(arg prefix)left_inner_finger_joint" value="-0.8" />
+        <joint name="$(arg prefix)left_inner_finger_joint" value="0.8" />
         <joint name="$(arg prefix)right_inner_knuckle_joint" value="0.8" />
         <joint name="$(arg prefix)finger_joint" value="0.8" />
@@ -79,7 +79,7 @@
         <joint name="$(arg prefix)right_outer_knuckle_joint" value="0.8" />
     </group_state>
-    <!--END EFFECTOR - Purpose - Represent information about an end effector.-->
+    <!--END EFFECTOR: Purpose: Represent information about an end effector.-->
     <end_effector name="gripper" parent_link="$(arg prefix)base_link" group="gripper" />
-    <!--PASSIVE JOINT - Purpose - this element is used to mark joints that are not actuated-->
+    <!--PASSIVE JOINT: Purpose: this element is used to mark joints that are not actuated-->
     <passive_joint name="$(arg prefix)left_inner_finger_joint" />
     <passive_joint name="$(arg prefix)left_inner_knuckle_joint" />
@@ -87,5 +87,5 @@
     <passive_joint name="$(arg prefix)right_outer_knuckle_joint" />
     <passive_joint name="$(arg prefix)right_inner_finger_joint" />
-    <!--DISABLE COLLISIONS - By default it is assumed that any link of the robot could potentially come into collision with any other link in the robot. This tag disables collision checking between a specified pair of links. -->
+    <!--DISABLE COLLISIONS: By default it is assumed that any link of the robot could potentially come into collision with any other link in the robot. This tag disables collision checking between a specified pair of links. -->
     <disable_collisions link1="$(arg prefix)base_link" link2="$(arg prefix)forearm_link" reason="Never" />
     <disable_collisions link1="$(arg prefix)base_link" link2="$(arg prefix)half_arm_1_link" reason="Never" />

Commit message: define command interface

File: kortex_description/grippers/robotiq_2f_85/urdf/robotiq_2f_85_macro.xacro (robot description, xacro)
@@ -26,15 +26,11 @@
         <origin xyz="0 0 0" rpy="0 0 0" />
     </xacro:robotiq_gripper>
-    <xacro:if value="${use_internal_bus_gripper_comm}">
-      <xacro:if value="${not include_ros2_control}">
-        <joint name="${prefix}robotiq_85_left_knuckle_joint">
-          <command_interface name="position" />
-          <state_interface name="position">
-            <param name="initial_value">0.7929</param>
-          </state_interface>
-          <state_interface name="velocity"/>
-        </joint>
-      </xacro:if>
-    </xacro:if>
+    <joint name="${prefix}robotiq_85_left_knuckle_joint">
+      <command_interface name="position" />
+      <state_interface name="position">
+        <param name="initial_value">0.7929</param>
+      </state_interface>
+      <state_interface name="velocity"/>
+    </joint>
   </xacro:macro>
 </robot>
