Commit message: Fix joint value for left_inner_finger_joint

File: kortex_move_it_config/gen3_robotiq_2f_85_move_it_config/config/7dof/gen3_robotiq_2f_85.srdf.xacro (robot description, xacro)
@@ -72,5 +72,5 @@
     </group_state>
     <group_state name="closed" group="gripper">
-        <joint name="$(arg prefix)left_inner_finger_joint" value="0.8" />
+        <joint name="$(arg prefix)left_inner_finger_joint" value="-0.8" />
         <joint name="$(arg prefix)right_inner_knuckle_joint" value="0.8" />
         <joint name="$(arg prefix)finger_joint" value="0.8" />
