Commit message: Propagate parameter for gripper comm to xacro file.

File: kortex_description/robots/gen3.xacro (robot description, xacro)
@@ -11,6 +11,7 @@
     <xacro:arg name="use_fake_hardware" default="true" />
     <xacro:arg name="fake_sensor_commands" default="true" />
+    <xacro:arg name="use_internal_bus_gripper_comm" default="false" />
     <xacro:include filename="$(find kortex_description)/robots/kortex_robot.xacro" />
     <link name="world" />
-    <xacro:load_robot parent="world" arm="$(arg arm)" gripper="$(arg gripper)" dof="$(arg dof)" vision="$(arg vision)" robot_ip="$(arg robot_ip)" sim="$(arg sim)" prefix="$(arg prefix)" use_fake_hardware="$(arg use_fake_hardware)" fake_sensor_commands="$(arg fake_sensor_commands)" />
+    <xacro:load_robot parent="world" arm="$(arg arm)" gripper="$(arg gripper)" dof="$(arg dof)" vision="$(arg vision)" robot_ip="$(arg robot_ip)" sim="$(arg sim)" prefix="$(arg prefix)" use_fake_hardware="$(arg use_fake_hardware)" fake_sensor_commands="$(arg fake_sensor_commands)" use_internal_bus_gripper_comm="$(arg use_internal_bus_gripper_comm)" />
 </robot>

File: kortex_description/robots/kortex_robot.xacro (robot description, xacro)
@@ -1,5 +1,5 @@
 <?xml version="1.0"?>
 <robot xmlns:xacro="http://ros.org/wiki/xacro">
-    <xacro:macro name="load_robot" params="parent arm gripper dof vision robot_ip sim prefix use_fake_hardware fake_sensor_commands">
+    <xacro:macro name="load_robot" params="parent arm gripper dof vision robot_ip sim prefix use_fake_hardware fake_sensor_commands use_internal_bus_gripper_comm:=false">
         <!-- Files to include -->
         <xacro:include filename="$(find kortex_description)/arms/${arm}/${dof}dof/urdf/${arm}_macro.xacro" />
@@ -17,5 +17,5 @@
         <!-- Run the macros -->
         <!-- Load the arm -->
-        <xacro:load_arm parent="${parent}" dof="${dof}" vision="${vision}" robot_ip="${robot_ip}" prefix="${prefix}" use_fake_hardware="${use_fake_hardware}" fake_sensor_commands="${fake_sensor_commands}">
+        <xacro:load_arm parent="${parent}" dof="${dof}" vision="${vision}" robot_ip="${robot_ip}" prefix="${prefix}" use_fake_hardware="${use_fake_hardware}" fake_sensor_commands="${fake_sensor_commands}" use_internal_bus_gripper_comm="${use_internal_bus_gripper_comm}">
             <origin xyz="0 0 0" rpy="0 0 0"/>
         </xacro:load_arm>
