Commit message: Break initial_positions out into a yaml file

File: kortex_description/robots/kinova.urdf.xacro (robot description, xacro)
@@ -32,4 +32,8 @@
   <!-- import main macro -->
   <xacro:include filename="$(find kortex_description)/robots/kortex_robot.xacro" />
+  <!-- initial position for simulations (Mock Hardware, Gazebo, Ignition) -->
+  <xacro:arg name="initial_positions_file" default="$(find kortex_description)/config/initial_positions.yaml"/>
+  <!-- convert to property to use substitution in function -->
+  <xacro:property name="initial_positions_file" default="$(arg initial_positions_file)"/>
   <!-- create link fixed to the "world" -->
   <link name="world" />
@@ -56,5 +60,6 @@
     sim_gazebo="$(arg sim_gazebo)"
     sim_ignition="$(arg sim_ignition)"
-    sim_isaac="$(arg sim_isaac)" >
+    sim_isaac="$(arg sim_isaac)"
+    initial_positions="${xacro.load_yaml(initial_positions_file)}" >
     <origin xyz="0 0 0" rpy="0 0 0" />  <!-- position robot in the world -->
   </xacro:load_robot>
