Commit message: case is important

File: kortex_description/arms/gen3/7dof/urdf/GEN3_URDF_V12_vision.urdf (robot description, URDF)
Before this commit: robot GEN3_URDF_V12, 9 links, 8 joints
Links:
- link Bracelet_Link: geometry collision mesh filename=package://kortex_description/arms/gen3/7dof/meshes/braclet_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; visual mesh filename=package://kortex_description/arms/gen3/7dof/meshes/braclet_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

Commit message: so is spelling

File: kortex_description/arms/gen3/7dof/urdf/GEN3_URDF_V12_vision.urdf (robot description, URDF)
Before this commit: robot GEN3_URDF_V12, 9 links, 8 joints
Links:
- link Bracelet_Link: geometry collision mesh filename=package://kortex_description/arms/gen3/7dof/meshes/bracelet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; visual mesh filename=package://kortex_description/arms/gen3/7dof/meshes/bracelet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
