Commit message: Only include <ros2_control> xacro stuff once

File: kortex_description/arms/gen3/7dof/urdf/kortex.ros2_control.xacro (robot description, xacro)
@@ -108,4 +108,9 @@
         <state_interface name="effort"/>
       </joint>
+      <!-- TODO(andyz) - make this optional -->
+      <joint name="${prefix}finger_joint">
+        <command_interface name="position"/>
+        <state_interface name="position"/>
+      </joint>
     </ros2_control>
   </xacro:macro>

Commit message: fix ros2_control xacros

File: kortex_description/arms/gen3/7dof/urdf/kortex.ros2_control.xacro (robot description, xacro)
@@ -156,11 +156,4 @@
         <state_interface name="effort"/>
       </joint>
-      <xacro:if value="${use_internal_bus_gripper_comm}">
-      <joint name="${prefix}finger_joint">
-        <command_interface name="position"/>
-        <state_interface name="position"/>
-        <state_interface name="velocity"/>
-      </joint>
-      </xacro:if>
     </ros2_control>
   </xacro:macro>

File: kortex_description/grippers/robotiq_2f_85/urdf/robotiq_2f_85_macro.xacro (robot description, xacro)
@@ -8,5 +8,6 @@
     sim_ignition:=false
     sim_isaac:=false">
-    <xacro:include filename="$(find robotiq_description)/urdf/robotiq_gripper_macro.urdf.xacro" />
+    <xacro:include filename="$(find robotiq_description)/urdf/robotiq_2f_85_macro.urdf.xacro" />
+    <!-- Hardware talks directly to the gripper so we don't need ros2_control unless we are simulating -->
     <xacro:property name="include_ros2_control" value="false"/>
     <xacro:if value="${sim_ignition or sim_isaac or use_fake_hardware}">
@@ -17,5 +18,5 @@
         prefix="${prefix}"
         parent="${parent}"
-        include_ros2_control="${not include_ros2_control}"
+        include_ros2_control="${include_ros2_control}"
         use_fake_hardware="$(arg use_fake_hardware)"
         fake_sensor_commands="$(arg fake_sensor_commands)"

Commit message: Convert package to use robotiq_description and update xacros (#95)
* Convert package to use robotiq_description and update xacros

* fix ros2_control xacros

* update package.xml

* remove URDF files

* add sim_isaac arg to gen3.xacro

File: kortex_description/arms/gen3/7dof/urdf/kortex.ros2_control.xacro (robot description, xacro)
@@ -8,4 +8,5 @@
     sim_gazebo:=false
     sim_ignition:=false
+    sim_isaac:=false
     use_internal_bus_gripper_comm:=false
     tf_prefix
@@ -26,4 +27,9 @@
           <plugin>ign_ros2_control/IgnitionSystem</plugin>
         </xacro:if>
+        <xacro:if value="${sim_isaac}">
+          <plugin>topic_based_ros2_control/TopicBasedSystem</plugin>
+          <param name="joint_commands_topic">/isaac_joint_commands</param>
+          <param name="joint_states_topic">/isaac_joint_states</param>
+        </xacro:if>
         <xacro:if value="${use_fake_hardware}">
           <plugin>fake_components/GenericSystem</plugin>
@@ -31,5 +37,5 @@
           <param name="state_following_offset">0.0</param>
         </xacro:if>
-        <xacro:unless value="${use_fake_hardware or sim_gazebo or sim_ignition}">
+        <xacro:unless value="${use_fake_hardware or sim_gazebo or sim_ignition or sim_isaac}">
           <plugin>kortex2_driver/KortexMultiInterfaceHardware</plugin>
           <param name="robot_ip">${robot_ip}</param>
@@ -150,11 +156,4 @@
         <state_interface name="effort"/>
       </joint>
-      <xacro:if value="${use_internal_bus_gripper_comm}">
-      <joint name="${prefix}finger_joint">
-        <command_interface name="position"/>
-        <state_interface name="position"/>
-        <state_interface name="velocity"/>
-      </joint>
-      </xacro:if>
     </ros2_control>
   </xacro:macro>

File: kortex_description/grippers/robotiq_2f_85/urdf/robotiq_2f_85_macro.xacro (robot description, xacro)
@@ -1,7 +1,28 @@
 <?xml version="1.0"?>
 <robot name="robotiq_arg2f_85_model" xmlns:xacro="http://ros.org/wiki/xacro">
-  <xacro:macro name="load_gripper" params="parent prefix">
-    <xacro:include filename="$(find kortex_description)/grippers/robotiq_2f_85/urdf/robotiq_arg2f_85_model_macro.xacro" />
-    <xacro:robotiq_arg2f_85 parent="${parent}" prefix="${prefix}"/>
+  <xacro:macro name="load_gripper" params="
+    parent
+    prefix
+    use_fake_hardware:=false
+    fake_sensor_commands:=false
+    sim_ignition:=false
+    sim_isaac:=false">
+    <xacro:include filename="$(find robotiq_description)/urdf/robotiq_2f_85_macro.urdf.xacro" />
+    <!-- Hardware talks directly to the gripper so we don't need ros2_control unless we are simulating -->
+    <xacro:property name="include_ros2_control" value="false"/>
+    <xacro:if value="${sim_ignition or sim_isaac or use_fake_hardware}">
+      <xacro:property name="include_ros2_control" value="true"/>
+    </xacro:if>
+    <xacro:robotiq_gripper
+        name="RobotiqGripperHardwareInterface"
+        prefix="${prefix}"
+        parent="${parent}"
+        include_ros2_control="${include_ros2_control}"
+        use_fake_hardware="$(arg use_fake_hardware)"
+        fake_sensor_commands="$(arg fake_sensor_commands)"
+        sim_ignition="$(arg sim_ignition)"
+        sim_isaac="$(arg sim_isaac)">
+        <origin xyz="0 0 0" rpy="0 0 0" />
+    </xacro:robotiq_gripper>
   </xacro:macro>
 </robot>

File: kortex_description/robots/gen3.xacro (robot description, xacro)
@@ -4,5 +4,5 @@
     <xacro:arg name="arm" default="gen3" />
     <xacro:arg name="dof" default="7" />
-    <xacro:arg name="vision" default="true" />
+    <xacro:arg name="vision" default="false" />
     <xacro:arg name="robot_ip" default="192.168.11.11" />
     <xacro:arg name="username" default="admin" />
@@ -13,5 +13,7 @@
     <xacro:arg name="connection_inactivity_timeout_ms" default="2000" />
     <xacro:arg name="gripper" default="" />
-    <xacro:arg name="sim" default="false" />
+    <xacro:arg name="sim_gazebo" default="false" />
+    <xacro:arg name="sim_ignition" default="false" />
+    <xacro:arg name="sim_issac" default="false" />
     <xacro:arg name="prefix" default="" />
     <xacro:arg name="use_fake_hardware" default="true" />
@@ -20,20 +22,25 @@
     <xacro:include filename="$(find kortex_description)/robots/kortex_robot.xacro" />
     <link name="world" />
-    <xacro:load_robot parent="world"
-                      arm="$(arg arm)"
-                      gripper="$(arg gripper)"
-                      dof="$(arg dof)"
-                      vision="$(arg vision)"
-                      robot_ip="$(arg robot_ip)"
-                      username="$(arg username)"
-                      password="$(arg password)"
-                      port="$(arg port)"
-                      port_realtime="$(arg port_realtime)"
-                      session_inactivity_timeout_ms="$(arg session_inactivity_timeout_ms)"
-                      connection_inactivity_timeout_ms="$(arg connection_inactivity_timeout_ms)"
-                      sim="$(arg sim)"
-                      prefix="$(arg prefix)"
-                      use_fake_hardware="$(arg use_fake_hardware)"
-                      fake_sensor_commands="$(arg fake_sensor_commands)"
-                      use_internal_bus_gripper_comm="$(arg use_internal_bus_gripper_comm)" />
+    <xacro:load_robot
+        parent="world"
+        arm="$(arg arm)"
+        gripper="$(arg gripper)"
+        dof="$(arg dof)"
+        vision="$(arg vision)"
+        robot_ip="$(arg robot_ip)"
+        username="$(arg username)"
+        password="$(arg password)"
+        port="$(arg port)"
+        port_realtime="$(arg port_realtime)"
+        session_inactivity_timeout_ms="$(arg session_inactivity_timeout_ms)"
+        connection_inactivity_timeout_ms="$(arg connection_inactivity_timeout_ms)"
+        use_internal_bus_gripper_comm="$(arg use_internal_bus_gripper_comm)"
+        prefix="$(arg prefix)"
+        use_fake_hardware="$(arg use_fake_hardware)"
+        fake_sensor_commands="$(arg fake_sensor_commands)"
+        sim_gazebo="$(arg sim_gazebo)"
+        sim_ignition="$(arg sim_ignition)"
+        sim_issac="$(arg sim_isaac)" >
+        <origin xyz="0 0 0" rpy="0 0 0" />  <!-- position robot in the world -->
+    </xacro:load_robot>
 </robot>

File: kortex_description/robots/kortex_robot.xacro (robot description, xacro)
@@ -20,5 +20,6 @@
     fake_sensor_commands:=false
     sim_gazebo:=false
-    sim_ignition:=false" >
+    sim_ignition:=false
+    sim_isaac:=false" >
     <!-- Include and load arm macro files -->
     <xacro:include filename="$(find kortex_description)/arms/${arm}/${dof}dof/urdf/${arm}_macro.xacro" />
@@ -40,5 +41,6 @@
       fake_sensor_commands="${fake_sensor_commands}"
       sim_gazebo="${sim_gazebo}"
-      sim_ignition="${sim_ignition}" >
+      sim_ignition="${sim_ignition}"
+      sim_isaac="${sim_isaac}" >
       <xacro:insert_block name="origin" />
     </xacro:load_arm>
@@ -57,17 +59,12 @@
       <xacro:include filename="$(find kortex_description)/grippers/${gripper}/urdf/${gripper}_macro.xacro" />
       <!-- last_arm_link is defined in "$(find kortex_description)/arms/${arm}/urdf/${arm}_macro.xacro" -->
-      <xacro:load_gripper parent="${prefix}${last_arm_link}"  prefix="${prefix}"/>
+      <xacro:load_gripper
+        parent="${prefix}${last_arm_link}"
+        prefix="${prefix}"
+        use_fake_hardware="${use_fake_hardware}"
+        fake_sensor_commands="${fake_sensor_commands}"
+        sim_ignition="${sim_ignition}"
+        sim_isaac="${sim_isaac}"/>
     </xacro:unless>
-    <!-- Load the Gazebo transmissions and gazebo_ros_control plugin -->
-    <xacro:if value="${sim_gazebo or sim_ignition}">
-      <!-- Arm transmission elements-->
-      <xacro:include filename="$(find kortex_description)/arms/${arm}/${dof}dof/urdf/${arm}_transmission_macro.xacro" />
-      <xacro:load_gazebo_arm_transmissions prefix="${prefix}"/>
-      <!-- Gripper transmission elements if there is a gripper-->
-      <xacro:unless value="${not gripper}">
-        <xacro:include filename="$(find kortex_description)/grippers/${gripper}/urdf/${gripper}_transmission_macro.xacro" />
-        <xacro:load_gazebo_gripper_transmissions prefix="${prefix}"/>
-      </xacro:unless>
-    </xacro:if>
   </xacro:macro>
 </robot>

Commit message: Defined command interface in the correct spot

File: kortex_description/arms/gen3/7dof/urdf/kortex.ros2_control.xacro (robot description, xacro)
@@ -161,4 +161,11 @@
         <state_interface name="effort"/>
       </joint>
+      <xacro:if value="${use_internal_bus_gripper_comm}">
+        <joint name="${prefix}${gripper_joint_name}">
+          <command_interface name="position" />
+          <state_interface name="position"/>
+          <state_interface name="velocity"/>
+        </joint>
+      </xacro:if>
     </ros2_control>
   </xacro:macro>

File: kortex_description/grippers/robotiq_2f_85/urdf/robotiq_2f_85_macro.xacro (robot description, xacro)
@@ -26,11 +26,4 @@
         <origin xyz="0 0 0" rpy="0 0 0" />
     </xacro:robotiq_gripper>
-    <joint name="${prefix}robotiq_85_left_knuckle_joint">
-      <command_interface name="position" />
-      <state_interface name="position">
-        <param name="initial_value">0.7929</param>
-      </state_interface>
-      <state_interface name="velocity"/>
-    </joint>
   </xacro:macro>
 </robot>

Commit message: Fix mock_hardware and enable simulating gen3_lite

File: kortex_description/arms/gen3/7dof/urdf/kortex.ros2_control.xacro (robot description, xacro)
@@ -135,11 +135,4 @@
         <state_interface name="effort"/>
       </joint>
-      <xacro:if value="${use_internal_bus_gripper_comm}">
-        <joint name="${prefix}${gripper_joint_name}">
-          <command_interface name="position" />
-          <state_interface name="position"/>
-          <state_interface name="velocity"/>
-        </joint>
-      </xacro:if>
     </ros2_control>
   </xacro:macro>

File: kortex_description/grippers/gen3_lite_2f/urdf/gen3_lite_2f_macro.xacro (robot description, xacro)
@@ -11,4 +11,14 @@
     isaac_joint_states:=/isaac_joint_states
     use_internal_bus_gripper_comm:=true">
+    <xacro:include filename="$(find kortex_description)/grippers/gen3_lite_2f/urdf/gen3_lite_2f.ros2_control.xacro" />
+    <xacro:gripper_ros2_control
+      prefix="${prefix}"
+      use_fake_hardware="${use_fake_hardware}"
+      fake_sensor_commands="${fake_sensor_commands}"
+      sim_ignition="${sim_ignition}"
+      sim_isaac="${sim_isaac}"
+      isaac_joint_commands="${isaac_joint_commands}"
+      isaac_joint_states="${isaac_joint_states}"
+      use_internal_bus_gripper_comm="${use_internal_bus_gripper_comm}"/>
     <!-- Tool frame used by the arm -->
     <link name="${prefix}tool_frame"/>

File: kortex_description/grippers/robotiq_2f_140/urdf/robotiq_2f_140_macro.xacro (robot description, xacro)
@@ -9,5 +9,6 @@
     sim_isaac:=false
     isaac_joint_commands:=/isaac_joint_commands
-    isaac_joint_states:=/isaac_joint_states">
+    isaac_joint_states:=/isaac_joint_states
+    use_internal_bus_gripper_comm:=false">
     <xacro:include filename="$(find robotiq_description)/urdf/robotiq_2f_140_macro.urdf.xacro" />
     <!-- Hardware talks directly to the gripper so we don't need ros2_control unless we are simulating -->
@@ -29,4 +30,13 @@
         <origin xyz="0 0 0" rpy="0 0 0" />
     </xacro:robotiq_gripper>
+    <!-- When running hardware we need to set the ros2_control command and state interfaces for the gripper -->
+    <xacro:if value="${use_internal_bus_gripper_comm}">
+        <joint name="${prefix}finger_joint">
+          <command_interface name="position" />
+          <state_interface name="position"/>
+          <state_interface name="velocity"/>
+        </joint>
+      </xacro:if>
+  </xacro:macro>
   </xacro:macro>
 </robot>

File: kortex_description/grippers/robotiq_2f_85/urdf/robotiq_2f_85_macro.xacro (robot description, xacro)
@@ -10,5 +10,5 @@
     isaac_joint_commands:=/isaac_joint_commands
     isaac_joint_states:=/isaac_joint_states
-    use_internal_bus_gripper_comm:=true">
+    use_internal_bus_gripper_comm:=false">
     <xacro:include filename="$(find robotiq_description)/urdf/robotiq_2f_85_macro.urdf.xacro" />
     <!-- Hardware talks directly to the gripper so we don't need ros2_control unless we are simulating -->
@@ -30,4 +30,12 @@
         <origin xyz="0 0 0" rpy="0 0 0" />
     </xacro:robotiq_gripper>
+    <!-- When running hardware we need to set the ros2_control command and state interfaces for the gripper -->
+    <xacro:if value="${use_internal_bus_gripper_comm}">
+        <joint name="${prefix}robotiq_85_left_knuckle_joint">
+          <command_interface name="position" />
+          <state_interface name="position"/>
+          <state_interface name="velocity"/>
+        </joint>
+      </xacro:if>
   </xacro:macro>
 </robot>

File: kortex_description/robots/kortex_robot.xacro (robot description, xacro)
@@ -81,5 +81,6 @@
         sim_isaac="${sim_isaac}"
         isaac_joint_commands="${isaac_joint_commands}"
-        isaac_joint_states="${isaac_joint_states}"/>
+        isaac_joint_states="${isaac_joint_states}"
+        use_internal_bus_gripper_comm="${use_internal_bus_gripper_comm}"/>
     </xacro:unless>
   </xacro:macro>

Commit message: revert gripper joint in arm ros2_control.xacro

File: kortex_description/arms/gen3/7dof/urdf/kortex.ros2_control.xacro (robot description, xacro)
@@ -135,4 +135,11 @@
         <state_interface name="effort"/>
       </joint>
+      <xacro:if value="${use_internal_bus_gripper_comm}">
+        <joint name="${prefix}${gripper_joint_name}">
+          <command_interface name="position" />
+          <state_interface name="position"/>
+          <state_interface name="velocity"/>
+        </joint>
+      </xacro:if>
     </ros2_control>
   </xacro:macro>

File: kortex_description/grippers/robotiq_2f_140/urdf/robotiq_2f_140_macro.xacro (robot description, xacro)
@@ -30,12 +30,4 @@
         <origin xyz="0 0 0" rpy="0 0 0" />
     </xacro:robotiq_gripper>
-    <!-- When running hardware we need to set the ros2_control command and state interfaces for the gripper -->
-    <xacro:if value="${use_internal_bus_gripper_comm}">
-        <joint name="${prefix}finger_joint">
-          <command_interface name="position" />
-          <state_interface name="position"/>
-          <state_interface name="velocity"/>
-        </joint>
-      </xacro:if>
   </xacro:macro>
 </robot>

File: kortex_description/grippers/robotiq_2f_85/urdf/robotiq_2f_85_macro.xacro (robot description, xacro)
@@ -30,12 +30,4 @@
         <origin xyz="0 0 0" rpy="0 0 0" />
     </xacro:robotiq_gripper>
-    <!-- When running hardware we need to set the ros2_control command and state interfaces for the gripper -->
-    <xacro:if value="${use_internal_bus_gripper_comm}">
-        <joint name="${prefix}robotiq_85_left_knuckle_joint">
-          <command_interface name="position" />
-          <state_interface name="position"/>
-          <state_interface name="velocity"/>
-        </joint>
-      </xacro:if>
   </xacro:macro>
 </robot>

Commit message: Add additional guards if user sets use_fake_hardware and use_internal_bus_gripper_comm true

File: kortex_description/arms/gen3/7dof/urdf/kortex.ros2_control.xacro (robot description, xacro)
@@ -135,11 +135,13 @@
         <state_interface name="effort"/>
       </joint>
-      <xacro:if value="${use_internal_bus_gripper_comm}">
-        <joint name="${prefix}${gripper_joint_name}">
-          <command_interface name="position" />
-          <state_interface name="position"/>
-          <state_interface name="velocity"/>
-        </joint>
-      </xacro:if>
+      <xacro:unless value="${use_fake_hardware or sim_gazebo or sim_ignition or sim_isaac}">
+        <xacro:if value="${use_internal_bus_gripper_comm}">
+          <joint name="${prefix}${gripper_joint_name}">
+            <command_interface name="position" />
+            <state_interface name="position"/>
+            <state_interface name="velocity"/>
+          </joint>
+        </xacro:if>
+      </xacro:unless>
     </ros2_control>
   </xacro:macro>

File: kortex_description/arms/gen3_lite/6dof/urdf/kortex.ros2_control.xacro (robot description, xacro)
@@ -124,11 +124,13 @@
         <state_interface name="effort"/>
       </joint>
-      <xacro:if value="${use_internal_bus_gripper_comm}">
-      <joint name="${prefix}right_finger_bottom_joint">
-        <command_interface name="position"/>
-        <state_interface name="position"/>
-        <state_interface name="velocity"/>
-      </joint>
-      </xacro:if>
+      <xacro:unless value="${use_fake_hardware or sim_gazebo or sim_ignition or sim_isaac}">
+        <xacro:if value="${use_internal_bus_gripper_comm}">
+          <joint name="${prefix}right_finger_bottom_joint">
+            <command_interface name="position"/>
+            <state_interface name="position"/>
+            <state_interface name="velocity"/>
+          </joint>
+        </xacro:if>
+      </xacro:unless>
     </ros2_control>
   </xacro:macro>
