Commit message: Merged in pr-update_urdf (pull request #1)
Update URDF

* enable parent argument for gen3

Approved-by: Andy Zelenak

File: kortex_description/arms/gen3/7dof/urdf/gen3_macro.xacro (robot description, xacro)
@@ -3,5 +3,10 @@
   <!-- Propagate last link name information because it is the gripper's parent link -->
   <xacro:property name="last_arm_link" value="end_effector_link"/>
-  <xacro:macro name="load_arm" params="parent:='' dof vision prefix *origin">
+  <xacro:macro name="load_arm" params="parent dof vision prefix *origin">
+      <joint name="${prefix}base_joint" type="fixed">
+        <xacro:insert_block name="origin" />
+        <parent link="${parent}"/>
+        <child link="${prefix}base_link" />
+      </joint>
       <link name="${prefix}base_link">
         <inertial>

File: kortex_description/robots/gen3.xacro (robot description, xacro)
@@ -9,4 +9,5 @@
     <xacro:arg name="prefix" default="" />
     <xacro:include filename="$(find kortex_description)/robots/kortex_robot.xacro" />
-    <xacro:load_robot arm="$(arg arm)" gripper="$(arg gripper)" dof="$(arg dof)" vision="$(arg vision)" sim="$(arg sim)" prefix="$(arg prefix)" />
+    <link name="world" />
+    <xacro:load_robot parent="world" arm="$(arg arm)" gripper="$(arg gripper)" dof="$(arg dof)" vision="$(arg vision)" sim="$(arg sim)" prefix="$(arg prefix)" />
 </robot>

File: kortex_description/robots/kortex_robot.xacro (robot description, xacro)
@@ -1,5 +1,5 @@
 <?xml version="1.0"?>
 <robot xmlns:xacro="http://ros.org/wiki/xacro">
-    <xacro:macro name="load_robot" params="arm gripper dof vision sim prefix">
+    <xacro:macro name="load_robot" params="parent arm gripper dof vision sim prefix">
         <!-- Files to include -->
         <xacro:include filename="$(find kortex_description)/arms/${arm}/${dof}dof/urdf/${arm}_macro.xacro" />
@@ -16,15 +16,6 @@
         </xacro:if>
         <!-- Run the macros -->
-        <!-- For gazebo-->
-        <xacro:if value="${sim}">
-            <link name="world" />
-            <joint name="world_to_root" type="fixed">
-                <child link="${prefix}base_link" />
-                <parent link="world" />
-                <origin xyz="0 0 0" rpy="0 0 0" />
-            </joint>
-        </xacro:if>
         <!-- Load the arm -->
-        <xacro:load_arm parent="" dof="${dof}" vision="${vision}" prefix="${prefix}">
+        <xacro:load_arm parent="${parent}" dof="${dof}" vision="${vision}" prefix="${prefix}">
             <origin xyz="0 0 0" rpy="0 0 0"/>
         </xacro:load_arm>

Commit message: Add ros2_control hardware interface Approved-by: Andy Zelenak

File: kortex_description/arms/gen3/7dof/urdf/gen3_macro.xacro (robot description, xacro)
@@ -3,7 +3,12 @@
   <!-- Propagate last link name information because it is the gripper's parent link -->
   <xacro:property name="last_arm_link" value="end_effector_link"/>
-  <xacro:macro name="load_arm" params="parent dof vision prefix *origin">
-      <xacro:arg name="use_fake_hardware" default="true"/>
-      <xacro:arg name="fake_sensor_commands" default="true"/>
+  <xacro:macro name="load_arm" params="
+    parent
+    dof
+    vision
+    prefix
+    *origin
+    use_fake_hardware:=false
+    fake_sensor_commands:=false">
       <!-- ros2 control include -->
       <xacro:include filename="$(find kortex_description)/arms/gen3/${dof}dof/urdf/kortex.ros2_control.xacro" />

Commit message: Merged in pr-fix_ip_address (pull request #7)
Add ip_address argument to all gen3 xacros

* add ip_address argument to all gen3 xacros

* revert hardware_interface changes


Approved-by: Andy Zelenak

File: kortex_description/arms/gen3/7dof/urdf/gen3_macro.xacro (robot description, xacro)
@@ -9,4 +9,5 @@
     prefix
     *origin
+    robot_ip
     use_fake_hardware:=false
     fake_sensor_commands:=false">

File: kortex_description/robots/gen3.xacro (robot description, xacro)
@@ -5,4 +5,5 @@
     <xacro:arg name="dof" default="7" />
     <xacro:arg name="vision" default="true" />
+    <xacro:arg name="robot_ip" default="yyy.yyy.yyy.yyy" />
     <xacro:arg name="gripper" default="" />
     <xacro:arg name="sim" default="false" />
@@ -10,4 +11,4 @@
     <xacro:include filename="$(find kortex_description)/robots/kortex_robot.xacro" />
     <link name="world" />
-    <xacro:load_robot parent="world" arm="$(arg arm)" gripper="$(arg gripper)" dof="$(arg dof)" vision="$(arg vision)" sim="$(arg sim)" prefix="$(arg prefix)" />
+    <xacro:load_robot parent="world" arm="$(arg arm)" gripper="$(arg gripper)" dof="$(arg dof)" vision="$(arg vision)" robot_ip="$(arg robot_ip)" sim="$(arg sim)" prefix="$(arg prefix)" />
 </robot>

File: kortex_description/robots/kortex_robot.xacro (robot description, xacro)
@@ -1,5 +1,5 @@
 <?xml version="1.0"?>
 <robot xmlns:xacro="http://ros.org/wiki/xacro">
-    <xacro:macro name="load_robot" params="parent arm gripper dof vision sim prefix">
+    <xacro:macro name="load_robot" params="parent arm gripper dof vision robot_ip sim prefix">
         <!-- Files to include -->
         <xacro:include filename="$(find kortex_description)/arms/${arm}/${dof}dof/urdf/${arm}_macro.xacro" />
@@ -17,5 +17,5 @@
         <!-- Run the macros -->
         <!-- Load the arm -->
-        <xacro:load_arm parent="${parent}" dof="${dof}" vision="${vision}" prefix="${prefix}">
+        <xacro:load_arm parent="${parent}" dof="${dof}" vision="${vision}" robot_ip="${robot_ip}" prefix="${prefix}">
             <origin xyz="0 0 0" rpy="0 0 0"/>
         </xacro:load_arm>

Commit message: Fix arg parsing (again)

File: kortex_description/arms/gen3/7dof/urdf/gen3_macro.xacro (robot description, xacro)
@@ -10,6 +10,6 @@
     *origin
     robot_ip
-    use_fake_hardware:=false
-    fake_sensor_commands:=false">
+    use_fake_hardware
+    fake_sensor_commands">
       <!-- ros2 control include -->
       <xacro:include filename="$(find kortex_description)/arms/gen3/${dof}dof/urdf/kortex.ros2_control.xacro" />

File: kortex_description/robots/gen3.xacro (robot description, xacro)
@@ -9,6 +9,8 @@
     <xacro:arg name="sim" default="false" />
     <xacro:arg name="prefix" default="" />
+    <xacro:arg name="use_fake_hardware" default="true" />
+    <xacro:arg name="fake_sensor_commands" default="true" />
     <xacro:include filename="$(find kortex_description)/robots/kortex_robot.xacro" />
     <link name="world" />
-    <xacro:load_robot parent="world" arm="$(arg arm)" gripper="$(arg gripper)" dof="$(arg dof)" vision="$(arg vision)" robot_ip="$(arg robot_ip)" sim="$(arg sim)" prefix="$(arg prefix)" />
+    <xacro:load_robot parent="world" arm="$(arg arm)" gripper="$(arg gripper)" dof="$(arg dof)" vision="$(arg vision)" robot_ip="$(arg robot_ip)" sim="$(arg sim)" prefix="$(arg prefix)" use_fake_hardware="$(arg use_fake_hardware)" fake_sensor_commands="$(arg fake_sensor_commands)" />
 </robot>

File: kortex_description/robots/kortex_robot.xacro (robot description, xacro)
@@ -1,5 +1,5 @@
 <?xml version="1.0"?>
 <robot xmlns:xacro="http://ros.org/wiki/xacro">
-    <xacro:macro name="load_robot" params="parent arm gripper dof vision robot_ip sim prefix">
+    <xacro:macro name="load_robot" params="parent arm gripper dof vision robot_ip sim prefix use_fake_hardware fake_sensor_commands">
         <!-- Files to include -->
         <xacro:include filename="$(find kortex_description)/arms/${arm}/${dof}dof/urdf/${arm}_macro.xacro" />
@@ -17,5 +17,5 @@
         <!-- Run the macros -->
         <!-- Load the arm -->
-        <xacro:load_arm parent="${parent}" dof="${dof}" vision="${vision}" robot_ip="${robot_ip}" prefix="${prefix}">
+        <xacro:load_arm parent="${parent}" dof="${dof}" vision="${vision}" robot_ip="${robot_ip}" prefix="${prefix}" use_fake_hardware="${use_fake_hardware}" fake_sensor_commands="${fake_sensor_commands}">
             <origin xyz="0 0 0" rpy="0 0 0"/>
         </xacro:load_arm>

Commit message: limited shoulder from +-2.41 to +-1.3

File: kortex_description/arms/gen3/7dof/urdf/gen3_macro.xacro (robot description, xacro)
@@ -115,5 +115,5 @@
       <axis
         xyz="0 0 1" />
-      <limit lower="-2.41" upper="2.41" effort="39" velocity="1.3963" />
+      <limit lower="-1.3" upper="1.3" effort="39" velocity="1.3963" />
     </joint>
     <link name="${prefix}half_arm_2_link">

Commit message: increase range to +-1.4 rad

File: kortex_description/arms/gen3/7dof/urdf/gen3_macro.xacro (robot description, xacro)
@@ -115,5 +115,5 @@
       <axis
         xyz="0 0 1" />
-      <limit lower="-1.3" upper="1.3" effort="39" velocity="1.3963" />
+      <limit lower="-1.4" upper="1.4" effort="39" velocity="1.3963" />
     </joint>
     <link name="${prefix}half_arm_2_link">

Commit message: Limited shoulder to keep elbow up (#22)
* limited shoulder from +-2.41 to +-1.3

* increase range to +-1.4 rad

File: kortex_description/arms/gen3/7dof/urdf/gen3_macro.xacro (robot description, xacro)
@@ -115,5 +115,5 @@
       <axis
         xyz="0 0 1" />
-      <limit lower="-2.41" upper="2.41" effort="39" velocity="1.3963" />
+      <limit lower="-1.4" upper="1.4" effort="39" velocity="1.3963" />
     </joint>
     <link name="${prefix}half_arm_2_link">

Commit message: Add xacro arg for velocity scaling

File: kortex_description/arms/gen3/7dof/urdf/gen3_macro.xacro (robot description, xacro)
@@ -11,5 +11,6 @@
     robot_ip
     use_fake_hardware
-    fake_sensor_commands">
+    fake_sensor_commands
+    max_velocity_scaling_factor">
       <!-- ros2 control include -->
       <xacro:include filename="$(find kortex_description)/arms/gen3/${dof}dof/urdf/kortex.ros2_control.xacro" />
@@ -81,5 +82,5 @@
       <limit
         effort="39"
-        velocity="1.3963" />
+        velocity="${max_velocity_scaling_factor * 1.3963}" />
     </joint>
     <link name="${prefix}half_arm_1_link">
@@ -115,5 +116,5 @@
       <axis
         xyz="0 0 1" />
-      <limit lower="-1.4" upper="1.4" effort="39" velocity="1.3963" />
+      <limit lower="-1.4" upper="1.4" effort="39" velocity="${max_velocity_scaling_factor * 1.3963}" />
     </joint>
     <link name="${prefix}half_arm_2_link">
@@ -151,5 +152,5 @@
       <limit
         effort="39"
-        velocity="1.3963" />
+        velocity="${max_velocity_scaling_factor * 1.3963}" />
     </joint>
     <link name="${prefix}forearm_link">
@@ -185,5 +186,5 @@
       <axis
         xyz="0 0 1" />
-      <limit lower="-2.66" upper="2.66" effort="39" velocity="1.3963" />
+      <limit lower="-2.66" upper="2.66" effort="39" velocity="${max_velocity_scaling_factor * 1.3963}" />
     </joint>
     <link name="${prefix}spherical_wrist_1_link">
@@ -221,5 +222,5 @@
       <limit
         effort="9"
-        velocity="1.2218" />
+        velocity="${max_velocity_scaling_factor * 1.2218}" />
     </joint>
     <link name="${prefix}spherical_wrist_2_link">
@@ -255,5 +256,5 @@
       <axis
         xyz="0 0 1" />
-      <limit lower="-2.23" upper="2.23" effort="9" velocity="1.2218" />
+      <limit lower="-2.23" upper="2.23" effort="9" velocity="${max_velocity_scaling_factor * 1.2218}" />
     </joint>
     <xacro:if value="${vision}">
@@ -317,5 +318,5 @@
       <limit
         effort="9"
-        velocity="1.2218" />
+        velocity="${max_velocity_scaling_factor * 1.2218}" />
     </joint>
     <link name="${prefix}end_effector_link" />

File: kortex_description/robots/gen3.xacro (robot description, xacro)
@@ -11,4 +11,5 @@
     <xacro:arg name="use_fake_hardware" default="true" />
     <xacro:arg name="fake_sensor_commands" default="true" />
+    <xacro:arg name="max_velocity_scaling_factor" default="1.0" />
     <xacro:include filename="$(find kortex_description)/robots/kortex_robot.xacro" />
     <link name="world" />

Commit message: Propagate parameters through urdfs.

File: kortex_description/arms/gen3/7dof/urdf/gen3_macro.xacro (robot description, xacro)
@@ -10,4 +10,10 @@
     *origin
     robot_ip
+    username
+    password
+    port
+    port_realtime
+    session_inactivity_timeout_ms
+    connection_inactivity_timeout_ms
     use_fake_hardware
     fake_sensor_commands
@@ -21,4 +27,10 @@
         tf_prefix=""
         robot_ip="${robot_ip}"
+        username="${username}"
+        password="${password}"
+        port="${port}"
+        port_realtime="${port_realtime}"
+        session_inactivity_timeout_ms="${session_inactivity_timeout_ms}"
+        connection_inactivity_timeout_ms="${connection_inactivity_timeout_ms}"
         use_internal_bus_gripper_comm="${use_internal_bus_gripper_comm}"/>
       <joint name="${prefix}base_joint" type="fixed">

File: kortex_description/arms/gen3/7dof/urdf/kortex.ros2_control.xacro (robot description, xacro)
@@ -15,4 +15,10 @@
           <plugin>kortex2_driver/KortexMultiInterfaceHardware</plugin>
           <param name="robot_ip">${robot_ip}</param>
+          <param name="username">${username}</param>
+          <param name="password">${password}</param>
+          <param name="port">${port}</param>
+          <param name="port_realtime">${port_realtime}</param>
+          <param name="session_inactivity_timeout_ms">${session_inactivity_timeout_ms}</param>
+          <param name="connection_inactivity_timeout_ms">${connection_inactivity_timeout_ms}</param>
           <param name="tf_prefix">"${tf_prefix}"</param>
           <param name="use_internal_bus_gripper_comm">${use_internal_bus_gripper_comm}</param>

File: kortex_description/robots/gen3.xacro (robot description, xacro)
@@ -5,5 +5,11 @@
     <xacro:arg name="dof" default="7" />
     <xacro:arg name="vision" default="true" />
-    <xacro:arg name="robot_ip" default="yyy.yyy.yyy.yyy" />
+    <xacro:arg name="robot_ip" default="192.168.11.11" />
+    <xacro:arg name="username" default="admin" />
+    <xacro:arg name="password" default="admin" />
+    <xacro:arg name="port" default="10000" />
+    <xacro:arg name="port_realtime" default="10001" />
+    <xacro:arg name="session_inactivity_timeout_ms" default="60000" />
+    <xacro:arg name="connection_inactivity_timeout_ms" default="2000" />
     <xacro:arg name="gripper" default="" />
     <xacro:arg name="sim" default="false" />
@@ -14,4 +20,20 @@
     <xacro:include filename="$(find kortex_description)/robots/kortex_robot.xacro" />
     <link name="world" />
-    <xacro:load_robot parent="world" arm="$(arg arm)" gripper="$(arg gripper)" dof="$(arg dof)" vision="$(arg vision)" robot_ip="$(arg robot_ip)" sim="$(arg sim)" prefix="$(arg prefix)" use_fake_hardware="$(arg use_fake_hardware)" fake_sensor_commands="$(arg fake_sensor_commands)" use_internal_bus_gripper_comm="$(arg use_internal_bus_gripper_comm)" />
+    <xacro:load_robot parent="world"
+                      arm="$(arg arm)"
+                      gripper="$(arg gripper)"
+                      dof="$(arg dof)"
+                      vision="$(arg vision)"
+                      robot_ip="$(arg robot_ip)"
+                      username="$(arg username)"
+                      password="$(arg password)"
+                      port="$(arg port)"
+                      port_realtime="$(arg port_realtime)"
+                      session_inactivity_timeout_ms="$(arg session_inactivity_timeout_ms)"
+                      connection_inactivity_timeout_ms="$(arg connection_inactivity_timeout_ms)"
+                      sim="$(arg sim)"
+                      prefix="$(arg prefix)"
+                      use_fake_hardware="$(arg use_fake_hardware)"
+                      fake_sensor_commands="$(arg fake_sensor_commands)"
+                      use_internal_bus_gripper_comm="$(arg use_internal_bus_gripper_comm)" />
 </robot>

File: kortex_description/robots/kortex_robot.xacro (robot description, xacro)
@@ -1,5 +1,7 @@
 <?xml version="1.0"?>
 <robot xmlns:xacro="http://ros.org/wiki/xacro">
-    <xacro:macro name="load_robot" params="parent arm gripper dof vision robot_ip sim prefix use_fake_hardware fake_sensor_commands use_internal_bus_gripper_comm:=false">
+    <xacro:macro name="load_robot" params="parent arm gripper dof vision
+    robot_ip username password port port_realtime session_inactivity_timeout_ms connection_inactivity_timeout_ms
+    sim prefix use_fake_hardware fake_sensor_commands use_internal_bus_gripper_comm:=false">
         <!-- Files to include -->
         <xacro:include filename="$(find kortex_description)/arms/${arm}/${dof}dof/urdf/${arm}_macro.xacro" />
@@ -17,5 +19,9 @@
         <!-- Run the macros -->
         <!-- Load the arm -->
-        <xacro:load_arm parent="${parent}" dof="${dof}" vision="${vision}" robot_ip="${robot_ip}" prefix="${prefix}" use_fake_hardware="${use_fake_hardware}" fake_sensor_commands="${fake_sensor_commands}" use_internal_bus_gripper_comm="${use_internal_bus_gripper_comm}">
+        <xacro:load_arm parent="${parent}" dof="${dof}" vision="${vision}"
+                        robot_ip="${robot_ip}" username="${username}" password="${password}" port="${port}" port_realtime="${port_realtime}"
+                        session_inactivity_timeout_ms="${session_inactivity_timeout_ms}" connection_inactivity_timeout_ms="${connection_inactivity_timeout_ms}"
+                        prefix="${prefix}" use_fake_hardware="${use_fake_hardware}" fake_sensor_commands="${fake_sensor_commands}"
+                        use_internal_bus_gripper_comm="${use_internal_bus_gripper_comm}">
             <origin xyz="0 0 0" rpy="0 0 0"/>
         </xacro:load_arm>
