Commit message: Adjust URDF and launch files for Gazebo and Ignition simulations.

File: kortex_description/arms/gen3/7dof/urdf/gen3_macro.xacro (robot description, xacro)
@@ -16,48 +16,52 @@
     session_inactivity_timeout_ms:=6000
     connection_inactivity_timeout_ms:=2000
-    use_fake_hardware
-    fake_sensor_commands
-    use_internal_bus_gripper_comm:=false">
-      <!-- ros2 control include -->
-      <xacro:include filename="$(find kortex_description)/arms/gen3/${dof}dof/urdf/kortex.ros2_control.xacro" />
-      <xacro:kortex_ros2_control
-        name="KortexMultiInterfaceHardware" prefix="${prefix}"
-        use_fake_hardware="${use_fake_hardware}"
-        fake_sensor_commands="${fake_sensor_commands}"
-        tf_prefix=""
-        robot_ip="${robot_ip}"
-        username="${username}"
-        password="${password}"
-        port="${port}"
-        port_realtime="${port_realtime}"
-        session_inactivity_timeout_ms="${session_inactivity_timeout_ms}"
-        connection_inactivity_timeout_ms="${connection_inactivity_timeout_ms}"
-        use_internal_bus_gripper_comm="${use_internal_bus_gripper_comm}"/>
-      <joint name="${prefix}base_joint" type="fixed">
-        <xacro:insert_block name="origin" />
-        <parent link="${parent}"/>
-        <child link="${prefix}base_link" />
-      </joint>
-      <link name="${prefix}base_link">
-        <inertial>
-          <origin xyz="-0.000648 -0.000166 0.084487" rpy="0 0 0" />
-          <mass value="1.697" />
-          <inertia ixx="0.004622" ixy="9E-06" ixz="6E-05" iyy="0.004495" iyz="9E-06" izz="0.002079" />
-        </inertial>
-        <visual>
-          <origin xyz="0 0 0" rpy="0 0 0" />
-          <geometry>
-            <mesh filename="package://kortex_description/arms/gen3/${dof}dof/meshes/base_link.STL" />
-          </geometry>
-          <material name="">
-            <color rgba="0.75294 0.75294 0.75294 1" />
-          </material>
-        </visual>
-        <collision>
-          <origin xyz="0 0 0" rpy="0 0 0" />
-          <geometry>
-            <mesh filename="package://kortex_description/arms/gen3/${dof}dof/meshes/base_link.STL" />
-          </geometry>
-        </collision>
+    use_internal_bus_gripper_comm:=false
+    use_fake_hardware:=false
+    fake_sensor_commands:=false
+    gazebo_sim:=false
+    ignition_sim:=false" >
+    <!-- ros2 control include -->
+    <xacro:include filename="$(find kortex_description)/arms/gen3/${dof}dof/urdf/kortex.ros2_control.xacro" />
+    <xacro:kortex_ros2_control
+      name="${prefix}KortexMultiInterfaceHardware" prefix="${prefix}"
+      use_fake_hardware="${use_fake_hardware}"
+      fake_sensor_commands="${fake_sensor_commands}"
+      gazebo_sim="${gazebo_sim}"
+      ignition_sim="${ignition_sim}"
+      tf_prefix=""
+      robot_ip="${robot_ip}"
+      username="${username}"
+      password="${password}"
+      port="${port}"
+      port_realtime="${port_realtime}"
+      session_inactivity_timeout_ms="${session_inactivity_timeout_ms}"
+      connection_inactivity_timeout_ms="${connection_inactivity_timeout_ms}"
+      use_internal_bus_gripper_comm="${use_internal_bus_gripper_comm}" />
+    <joint name="${prefix}base_joint" type="fixed">
+      <xacro:insert_block name="origin" />
+      <parent link="${parent}"/>
+      <child link="${prefix}base_link" />
+    </joint>
+    <link name="${prefix}base_link">
+      <inertial>
+        <origin xyz="-0.000648 -0.000166 0.084487" rpy="0 0 0" />
+        <mass value="1.697" />
+        <inertia ixx="0.004622" ixy="9E-06" ixz="6E-05" iyy="0.004495" iyz="9E-06" izz="0.002079" />
+      </inertial>
+      <visual>
+        <origin xyz="0 0 0" rpy="0 0 0" />
+        <geometry>
+          <mesh filename="file://$(find kortex_description)/arms/gen3/${dof}dof/meshes/base_link.STL" />
+        </geometry>
+        <material name="">
+          <color rgba="0.75294 0.75294 0.75294 1" />
+        </material>
+      </visual>
+      <collision>
+        <origin xyz="0 0 0" rpy="0 0 0" />
+        <geometry>
+          <mesh filename="file://$(find kortex_description)/arms/gen3/${dof}dof/meshes/base_link.STL" />
+        </geometry>
+      </collision>
     </link>
     <link name="${prefix}shoulder_link">
@@ -70,14 +74,14 @@
         <origin xyz="0 0 0" rpy="0 0 0" />
         <geometry>
-          <mesh filename="package://kortex_description/arms/gen3/${dof}dof/meshes/shoulder_link.STL" />
-        </geometry>
-        <material name="">
-          <color rgba="0.75294 0.75294 0.75294 1" />
-        </material>
-      </visual>
-      <collision>
-        <origin xyz="0 0 0" rpy="0 0 0" />
-        <geometry>
-          <mesh filename="package://kortex_description/arms/gen3/${dof}dof/meshes/shoulder_link.STL" />
+          <mesh filename="file://$(find kortex_description)/arms/gen3/${dof}dof/meshes/shoulder_link.STL" />
+        </geometry>
+        <material name="">
+          <color rgba="0.75294 0.75294 0.75294 1" />
+        </material>
+      </visual>
+      <collision>
+        <origin xyz="0 0 0" rpy="0 0 0" />
+        <geometry>
+          <mesh filename="file://$(find kortex_description)/arms/gen3/${dof}dof/meshes/shoulder_link.STL" />
         </geometry>
       </collision>
@@ -106,14 +110,14 @@
         <origin xyz="0 0 0" rpy="0 0 0" />
         <geometry>
-          <mesh filename="package://kortex_description/arms/gen3/${dof}dof/meshes/half_arm_1_link.STL" />
-        </geometry>
-        <material name="">
-          <color rgba="0.75294 0.75294 0.75294 1" />
-        </material>
-      </visual>
-      <collision>
-        <origin xyz="0 0 0" rpy="0 0 0" />
-        <geometry>
-          <mesh filename="package://kortex_description/arms/gen3/${dof}dof/meshes/half_arm_1_link.STL" />
+          <mesh filename="file://$(find kortex_description)/arms/gen3/${dof}dof/meshes/half_arm_1_link.STL" />
+        </geometry>
+        <material name="">
+          <color rgba="0.75294 0.75294 0.75294 1" />
+        </material>
+      </visual>
+      <collision>
+        <origin xyz="0 0 0" rpy="0 0 0" />
+        <geometry>
+          <mesh filename="file://$(find kortex_description)/arms/gen3/${dof}dof/meshes/half_arm_1_link.STL" />
         </geometry>
       </collision>
@@ -140,14 +144,14 @@
         <origin xyz="0 0 0" rpy="0 0 0" />
         <geometry>
-          <mesh filename="package://kortex_description/arms/gen3/${dof}dof/meshes/half_arm_2_link.STL" />
-        </geometry>
-        <material name="">
-          <color rgba="0.75294 0.75294 0.75294 1" />
-        </material>
-      </visual>
-      <collision>
-        <origin xyz="0 0 0" rpy="0 0 0" />
-        <geometry>
-          <mesh filename="package://kortex_description/arms/gen3/${dof}dof/meshes/half_arm_2_link.STL" />
+          <mesh filename="file://$(find kortex_description)/arms/gen3/${dof}dof/meshes/half_arm_2_link.STL" />
+        </geometry>
+        <material name="">
+          <color rgba="0.75294 0.75294 0.75294 1" />
+        </material>
+      </visual>
+      <collision>
+        <origin xyz="0 0 0" rpy="0 0 0" />
+        <geometry>
+          <mesh filename="file://$(find kortex_description)/arms/gen3/${dof}dof/meshes/half_arm_2_link.STL" />
         </geometry>
       </collision>
@@ -176,14 +180,14 @@
         <origin xyz="0 0 0" rpy="0 0 0" />
         <geometry>
-          <mesh filename="package://kortex_description/arms/gen3/${dof}dof/meshes/forearm_link.STL" />
-        </geometry>
-        <material name="">
-          <color rgba="0.75294 0.75294 0.75294 1" />
-        </material>
-      </visual>
-      <collision>
-        <origin xyz="0 0 0" rpy="0 0 0" />
-        <geometry>
-          <mesh filename="package://kortex_description/arms/gen3/${dof}dof/meshes/forearm_link.STL" />
+          <mesh filename="file://$(find kortex_description)/arms/gen3/${dof}dof/meshes/forearm_link.STL" />
+        </geometry>
+        <material name="">
+          <color rgba="0.75294 0.75294 0.75294 1" />
+        </material>
+      </visual>
+      <collision>
+        <origin xyz="0 0 0" rpy="0 0 0" />
+        <geometry>
+          <mesh filename="file://$(find kortex_description)/arms/gen3/${dof}dof/meshes/forearm_link.STL" />
         </geometry>
       </collision>
@@ -210,14 +214,14 @@
         <origin xyz="0 0 0" rpy="0 0 0" />
         <geometry>
-          <mesh filename="package://kortex_description/arms/gen3/${dof}dof/meshes/spherical_wrist_1_link.STL" />
-        </geometry>
-        <material name="">
-          <color rgba="0.75294 0.75294 0.75294 1" />
-        </material>
-      </visual>
-      <collision>
-        <origin xyz="0 0 0" rpy="0 0 0" />
-        <geometry>
-          <mesh filename="package://kortex_description/arms/gen3/${dof}dof/meshes/spherical_wrist_1_link.STL" />
+          <mesh filename="file://$(find kortex_description)/arms/gen3/${dof}dof/meshes/spherical_wrist_1_link.STL" />
+        </geometry>
+        <material name="">
+          <color rgba="0.75294 0.75294 0.75294 1" />
+        </material>
+      </visual>
+      <collision>
+        <origin xyz="0 0 0" rpy="0 0 0" />
+        <geometry>
+          <mesh filename="file://$(find kortex_description)/arms/gen3/${dof}dof/meshes/spherical_wrist_1_link.STL" />
         </geometry>
       </collision>
@@ -246,14 +250,14 @@
         <origin xyz="0 0 0" rpy="0 0 0" />
         <geometry>
-          <mesh filename="package://kortex_description/arms/gen3/${dof}dof/meshes/spherical_wrist_2_link.STL" />
-        </geometry>
-        <material name="">
-          <color rgba="0.75294 0.75294 0.75294 1" />
-        </material>
-      </visual>
-      <collision>
-        <origin xyz="0 0 0" rpy="0 0 0" />
-        <geometry>
-          <mesh filename="package://kortex_description/arms/gen3/${dof}dof/meshes/spherical_wrist_2_link.STL" />
+          <mesh filename="file://$(find kortex_description)/arms/gen3/${dof}dof/meshes/spherical_wrist_2_link.STL" />
+        </geometry>
+        <material name="">
+          <color rgba="0.75294 0.75294 0.75294 1" />
+        </material>
+      </visual>
+      <collision>
+        <origin xyz="0 0 0" rpy="0 0 0" />
+        <geometry>
+          <mesh filename="file://$(find kortex_description)/arms/gen3/${dof}dof/meshes/spherical_wrist_2_link.STL" />
         </geometry>
       </collision>
@@ -281,14 +285,14 @@
         <origin xyz="0 0 0" rpy="0 0 0" />
         <geometry>
-          <mesh filename="package://kortex_description/arms/gen3/${dof}dof/meshes/bracelet_with_vision_link.STL" />
-        </geometry>
-        <material name="">
-          <color rgba="0.75294 0.75294 0.75294 1" />
-        </material>
-      </visual>
-      <collision>
-        <origin xyz="0 0 0" rpy="0 0 0" />
-        <geometry>
-          <mesh filename="package://kortex_description/arms/gen3/${dof}dof/meshes/bracelet_with_vision_link.STL" />
+          <mesh filename="file://$(find kortex_description)/arms/gen3/${dof}dof/meshes/bracelet_with_vision_link.STL" />
+        </geometry>
+        <material name="">
+          <color rgba="0.75294 0.75294 0.75294 1" />
+        </material>
+      </visual>
+      <collision>
+        <origin xyz="0 0 0" rpy="0 0 0" />
+        <geometry>
+          <mesh filename="file://$(find kortex_description)/arms/gen3/${dof}dof/meshes/bracelet_with_vision_link.STL" />
         </geometry>
       </collision>
@@ -305,14 +309,14 @@
         <origin xyz="0 0 0" rpy="0 0 0" />
         <geometry>
-          <mesh filename="package://kortex_description/arms/gen3/${dof}dof/meshes/bracelet_no_vision_link.STL" />
-        </geometry>
-        <material name="">
-          <color rgba="0.75294 0.75294 0.75294 1" />
-        </material>
-      </visual>
-      <collision>
-        <origin xyz="0 0 0" rpy="0 0 0" />
-        <geometry>
-          <mesh filename="package://kortex_description/arms/gen3/${dof}dof/meshes/bracelet_no_vision_link.STL" />
+          <mesh filename="file://$(find kortex_description)/arms/gen3/${dof}dof/meshes/bracelet_no_vision_link.STL" />
+        </geometry>
+        <material name="">
+          <color rgba="0.75294 0.75294 0.75294 1" />
+        </material>
+      </visual>
+      <collision>
+        <origin xyz="0 0 0" rpy="0 0 0" />
+        <geometry>
+          <mesh filename="file://$(find kortex_description)/arms/gen3/${dof}dof/meshes/bracelet_no_vision_link.STL" />
         </geometry>
       </collision>

File: kortex_description/arms/gen3/7dof/urdf/kortex.ros2_control.xacro (robot description, xacro)
@@ -1,10 +1,28 @@
 <?xml version="1.0"?>
 <robot xmlns:xacro="http://www.ros.org/wiki/xacro">
-  <xacro:macro name="kortex_ros2_control" params="name prefix
-    use_fake_hardware:=false fake_sensor_commands:=false
-    use_internal_bus_gripper_comm:=false tf_prefix
-    robot_ip username password port port_realtime session_inactivity_timeout_ms connection_inactivity_timeout_ms">
+  <xacro:macro name="kortex_ros2_control" params="
+    name
+    prefix
+    use_fake_hardware:=false
+    fake_sensor_commands:=false
+    gazebo_sim:=false
+    ignition_sim:=false
+    use_internal_bus_gripper_comm:=false
+    tf_prefix
+    robot_ip
+    username
+    password
+    port
+    port_realtime
+    session_inactivity_timeout_ms
+    connection_inactivity_timeout_ms">
     <ros2_control name="${name}" type="system">
       <hardware>
+        <xacro:if value="${gazebo_sim}">
+          <plugin>gazebo_ros2_control/GazeboSystem</plugin>
+        </xacro:if>
+        <xacro:if value="${ignition_sim}">
+          <plugin>ignition_ros2_control/IgnitionSystem</plugin>
+        </xacro:if>
         <xacro:if value="${use_fake_hardware}">
           <plugin>fake_components/GenericSystem</plugin>
@@ -12,5 +30,5 @@
           <param name="state_following_offset">0.0</param>
         </xacro:if>
-        <xacro:unless value="${use_fake_hardware}">
+        <xacro:unless value="${use_fake_hardware or gazebo_sim or ignition_sim}">
           <plugin>kortex2_driver/KortexMultiInterfaceHardware</plugin>
           <param name="robot_ip">${robot_ip}</param>
@@ -117,5 +135,4 @@
         <state_interface name="effort"/>
       </joint>
-      <!-- TODO(andyz) - make this optional -->
       <xacro:if value="${use_internal_bus_gripper_comm}">
       <joint name="${prefix}finger_joint">

File: kortex_description/robots/kortex_robot.xacro (robot description, xacro)
@@ -1,56 +1,73 @@
 <?xml version="1.0"?>
 <robot xmlns:xacro="http://ros.org/wiki/xacro">
-    <xacro:macro name="load_robot" params="parent arm gripper dof vision
-    robot_ip username password port port_realtime session_inactivity_timeout_ms connection_inactivity_timeout_ms
-    sim prefix use_fake_hardware fake_sensor_commands use_internal_bus_gripper_comm:=false">
-        <!-- Files to include -->
-        <xacro:include filename="$(find kortex_description)/arms/${arm}/${dof}dof/urdf/${arm}_macro.xacro" />
-        <xacro:unless value="${not gripper}">
-            <xacro:include filename="$(find kortex_description)/grippers/${gripper}/urdf/${gripper}_macro.xacro" />
-        </xacro:unless>
-        <xacro:if value="${sim}">
-            <!-- Arm transmission elements-->
-            <xacro:include filename="$(find kortex_description)/arms/${arm}/${dof}dof/urdf/${arm}_transmission_macro.xacro" />
-            <!-- Gripper transmission elements if there is a gripper-->
-            <xacro:unless value="${not gripper}">
-                <xacro:include filename="$(find kortex_description)/grippers/${gripper}/urdf/${gripper}_transmission_macro.xacro" />
-            </xacro:unless>
-        </xacro:if>
-        <!-- Run the macros -->
-        <!-- Load the arm -->
-        <xacro:load_arm parent="${parent}" dof="${dof}" vision="${vision}"
-                        robot_ip="${robot_ip}" username="${username}" password="${password}" port="${port}" port_realtime="${port_realtime}"
-                        session_inactivity_timeout_ms="${session_inactivity_timeout_ms}" connection_inactivity_timeout_ms="${connection_inactivity_timeout_ms}"
-                        prefix="${prefix}" use_fake_hardware="${use_fake_hardware}" fake_sensor_commands="${fake_sensor_commands}"
-                        use_internal_bus_gripper_comm="${use_internal_bus_gripper_comm}">
-            <origin xyz="0 0 0" rpy="0 0 0"/>
-        </xacro:load_arm>
-        <!-- Load the gripper -->
-        <xacro:unless value="${not gripper}">
-            <!-- last_arm_link is defined in "$(find kortex_description)/arms/${arm}/urdf/${arm}_macro.xacro" -->
-            <xacro:load_gripper parent="${prefix}${last_arm_link}"  prefix="${prefix}"/>
-        </xacro:unless>
-        <!-- If no gripper, define tool frame here -->
-        <xacro:if value="${not gripper}">
-            <link name="${prefix}tool_frame"/>
-            <joint name="${prefix}tool_frame_joint" type="fixed">
-                <origin xyz="0 0 0" rpy="0 0 0" />
-                <parent link="${prefix}${last_arm_link}" />
-                <child link="${prefix}tool_frame" />
-                <axis xyz="0 0 0" />
-            </joint>
-        </xacro:if>
-        <!-- Load the Gazebo transmissions and gazebo_ros_control plugin -->
-        <xacro:if value="${sim}">
-            <xacro:load_gazebo_arm_transmissions prefix="${prefix}"/>
-            <xacro:unless value="${not gripper}">
-                <xacro:load_gazebo_gripper_transmissions prefix="${prefix}"/>
-            </xacro:unless>
-            <gazebo>
-                <plugin name="gazebo_ros_control" filename="libgazebo_ros_control.so">
-                    <legacyModeNS>true</legacyModeNS>
-                </plugin>
-            </gazebo>
-        </xacro:if>
-    </xacro:macro>
+  <xacro:macro name="load_robot" params="
+    parent
+    *origin
+    prefix
+    arm
+    gripper
+    dof
+    vision
+    robot_ip
+    username
+    password
+    port
+    port_realtime
+    session_inactivity_timeout_ms
+    connection_inactivity_timeout_ms
+    use_internal_bus_gripper_comm:=false
+    use_fake_hardware:=false
+    fake_sensor_commands:=false
+    gazebo_sim:=false
+    ignition_sim:=false" >
+    <!-- Include and load arm macro files -->
+    <xacro:include filename="$(find kortex_description)/arms/${arm}/${dof}dof/urdf/${arm}_macro.xacro" />
+    <!-- Load the arm -->
+    <xacro:load_arm
+      parent="${parent}"
+      dof="${dof}"
+      vision="${vision}"
+      robot_ip="${robot_ip}"
+      username="${username}"
+      password="${password}"
+      port="${port}"
+      port_realtime="${port_realtime}"
+      session_inactivity_timeout_ms="${session_inactivity_timeout_ms}"
+      connection_inactivity_timeout_ms="${connection_inactivity_timeout_ms}"
+      prefix="${prefix}"
+      use_internal_bus_gripper_comm="${use_internal_bus_gripper_comm}"
+      use_fake_hardware="${use_fake_hardware}"
+      fake_sensor_commands="${fake_sensor_commands}"
+      gazebo_sim="${gazebo_sim}"
+      ignition_sim="${ignition_sim}" >
+      <xacro:insert_block name="origin" />
+    </xacro:load_arm>
+    <!-- If no gripper, define tool frame here -->
+    <xacro:if value="${not gripper}">
+      <link name="${prefix}tool_frame"/>
+      <joint name="${prefix}tool_frame_joint" type="fixed">
+        <origin xyz="0 0 0" rpy="0 0 0" />
+        <parent link="${prefix}${last_arm_link}" />
+        <child link="${prefix}tool_frame" />
+        <axis xyz="0 0 0" />
+      </joint>
+    </xacro:if>
+    <!-- Include and load the gripper if defined -->
+    <xacro:unless value="${not gripper}">
+      <xacro:include filename="$(find kortex_description)/grippers/${gripper}/urdf/${gripper}_macro.xacro" />
+      <!-- last_arm_link is defined in "$(find kortex_description)/arms/${arm}/urdf/${arm}_macro.xacro" -->
+      <xacro:load_gripper parent="${prefix}${last_arm_link}"  prefix="${prefix}"/>
+    </xacro:unless>
+    <!-- Load the Gazebo transmissions and gazebo_ros_control plugin -->
+    <xacro:if value="${gazebo_sim or ignition_sim}">
+      <!-- Arm transmission elements-->
+      <xacro:include filename="$(find kortex_description)/arms/${arm}/${dof}dof/urdf/${arm}_transmission_macro.xacro" />
+      <xacro:load_gazebo_arm_transmissions prefix="${prefix}"/>
+      <!-- Gripper transmission elements if there is a gripper-->
+      <xacro:unless value="${not gripper}">
+        <xacro:include filename="$(find kortex_description)/grippers/${gripper}/urdf/${gripper}_transmission_macro.xacro" />
+        <xacro:load_gazebo_gripper_transmissions prefix="${prefix}"/>
+      </xacro:unless>
+    </xacro:if>
+  </xacro:macro>
 </robot>
