Commit message: Updated to work again and updated simulation parameters.

File: kortex_description/arms/gen3/7dof/urdf/gen3_macro.xacro (robot description, xacro)
@@ -19,7 +19,7 @@
     use_fake_hardware:=false
     fake_sensor_commands:=false
-    gazebo_sim:=false
-    ignition_sim:=false
-    initial_positions:=${dict(joint_1=0.0,joint_2=0.0,joint_3=0.0,joint_4=0.0,joint_5=0.0,joint_6=0.0)}" >
+    sim_gazebo:=false
+    sim_ignition:=false
+    initial_positions:=${dict(joint_1=0.0,joint_2=0.0,joint_3=0.0,joint_4=0.0,joint_5=0.0,joint_6=0.0,joint_7=0.0)}" >
     <!-- ros2 control include -->
     <xacro:include filename="$(find kortex_description)/arms/gen3/${dof}dof/urdf/kortex.ros2_control.xacro" />
@@ -28,6 +28,6 @@
       use_fake_hardware="${use_fake_hardware}"
       fake_sensor_commands="${fake_sensor_commands}"
-      gazebo_sim="${gazebo_sim}"
-      ignition_sim="${ignition_sim}"
+      sim_gazebo="${sim_gazebo}"
+      sim_ignition="${sim_ignition}"
       tf_prefix=""
       initial_positions="${initial_positions}"
@@ -352,5 +352,5 @@
     </joint>
     <!-- TODO(destogl) this probably collides with camera URDF -->
-<!--    <xacro:if value="${vision}">
+    <xacro:if value="${vision}">
       <link name="${prefix}camera_link" />
       <joint name="${prefix}camera_module" type="fixed">
@@ -371,5 +371,5 @@
         <child  link="${prefix}camera_color_frame" />
       </joint>
-    </xacro:if>-->
+    </xacro:if>
   </xacro:macro>
 </robot>

File: kortex_description/arms/gen3/7dof/urdf/kortex.ros2_control.xacro (robot description, xacro)
@@ -6,6 +6,6 @@
     use_fake_hardware:=false
     fake_sensor_commands:=false
-    gazebo_sim:=false
-    ignition_sim:=false
+    sim_gazebo:=false
+    sim_ignition:=false
     use_internal_bus_gripper_comm:=false
     tf_prefix
@@ -20,8 +20,8 @@
     <ros2_control name="${name}" type="system">
       <hardware>
-        <xacro:if value="${gazebo_sim}">
+        <xacro:if value="${sim_gazebo}">
           <plugin>gazebo_ros2_control/GazeboSystem</plugin>
         </xacro:if>
-        <xacro:if value="${ignition_sim}">
+        <xacro:if value="${sim_ignition}">
           <plugin>ign_ros2_control/IgnitionSystem</plugin>
         </xacro:if>
@@ -31,5 +31,5 @@
           <param name="state_following_offset">0.0</param>
         </xacro:if>
-        <xacro:unless value="${use_fake_hardware or gazebo_sim or ignition_sim}">
+        <xacro:unless value="${use_fake_hardware or sim_gazebo or sim_ignition}">
           <plugin>kortex2_driver/KortexMultiInterfaceHardware</plugin>
           <param name="robot_ip">${robot_ip}</param>

File: kortex_description/robots/kinova.urdf.xacro (robot description, xacro)
@@ -19,6 +19,6 @@
   <xacro:arg name="use_fake_hardware" default="true" />
   <xacro:arg name="fake_sensor_commands" default="true" />
-  <xacro:arg name="gazebo_sim" default="false" />
-  <xacro:arg name="ignition_sim" default="false" />
+  <xacro:arg name="sim_gazebo" default="false" />
+  <xacro:arg name="sim_ignition" default="false" />
   <xacro:arg name="simulation_controllers" default="$(find kortex2_bringup)/config/kortex_controllers.yaml" />
   <!-- import main macro -->
@@ -43,9 +43,9 @@
     use_fake_hardware="$(arg use_fake_hardware)"
     fake_sensor_commands="$(arg fake_sensor_commands)"
-    gazebo_sim="$(arg gazebo_sim)"
-    ignition_sim="$(arg ignition_sim)" >
+    sim_gazebo="$(arg sim_gazebo)"
+    sim_ignition="$(arg sim_ignition)" >
     <origin xyz="0 0 0" rpy="0 0 0" />          <!-- position robot in the world -->
   </xacro:load_robot>
-  <xacro:if value="$(arg gazebo_sim)">
+  <xacro:if value="$(arg sim_gazebo)">
     <!-- Gazebo plugins -->
     <gazebo reference="world">
@@ -57,5 +57,5 @@
     </gazebo>
   </xacro:if>
-  <xacro:if value="$(arg ignition_sim)">
+  <xacro:if value="$(arg sim_ignition)">
     <!-- Gazebo plugins -->
     <gazebo reference="world">

File: kortex_description/robots/kortex_robot.xacro (robot description, xacro)
@@ -19,6 +19,6 @@
     use_fake_hardware:=false
     fake_sensor_commands:=false
-    gazebo_sim:=false
-    ignition_sim:=false" >
+    sim_gazebo:=false
+    sim_ignition:=false" >
     <!-- Include and load arm macro files -->
     <xacro:include filename="$(find kortex_description)/arms/${arm}/${dof}dof/urdf/${arm}_macro.xacro" />
@@ -39,6 +39,6 @@
       use_fake_hardware="${use_fake_hardware}"
       fake_sensor_commands="${fake_sensor_commands}"
-      gazebo_sim="${gazebo_sim}"
-      ignition_sim="${ignition_sim}" >
+      sim_gazebo="${sim_gazebo}"
+      sim_ignition="${sim_ignition}" >
       <xacro:insert_block name="origin" />
     </xacro:load_arm>
@@ -60,5 +60,5 @@
     </xacro:unless>
     <!-- Load the Gazebo transmissions and gazebo_ros_control plugin -->
-    <xacro:if value="${gazebo_sim or ignition_sim}">
+    <xacro:if value="${sim_gazebo or sim_ignition}">
       <!-- Arm transmission elements-->
       <xacro:include filename="$(find kortex_description)/arms/${arm}/${dof}dof/urdf/${arm}_transmission_macro.xacro" />

File: kortex_move_it_config/gen3_move_it_config/config/7dof/gen3.srdf.xacro (robot description, xacro)
@@ -14,6 +14,6 @@
     <!--CHAINS - When a chain is specified, all the links along the chain (including endpoints) are included in the group. Additionally, all the joints that are parents to included links are also included. This means that joints along the chain and the parent joint of the base link are included in the group-->
     <!--SUBGROUPS - Groups can also be formed by referencing to already defined group names-->
-    <group name="$(arg prefix)$(arg name)">
-        <joint name="$(arg prefix)joint_1" />
+    <group name="$(arg name)">
+<!--        <joint name="$(arg prefix)joint_1" />
         <joint name="$(arg prefix)joint_2" />
         <joint name="$(arg prefix)joint_3" />
@@ -23,5 +23,6 @@
         <joint name="$(arg prefix)joint_7" />
         <joint name="$(arg prefix)end_effector" />
-        <joint name="$(arg prefix)tool_frame_joint" />
+        <joint name="$(arg prefix)tool_frame_joint" />-->
+        <chain base_link="$(arg prefix)base_link" tip_link="$(arg prefix)end_effector_link" />
     </group>
     <!--GROUP STATES - Purpose - Define a named state for a particular group, in terms of joint values. This is useful to define states like 'folded arms'-->
