Commit message: Kortex simulations (#64)
* Adjust URDF and launch files for Gazebo and Ignition simulations.

* Add simulation dependecies until released.

* Correct name of controllers URDF argument.

* Fix repos lines.

* Using gen3 per default in launch files and do not use any gripper. Kinematics file was adjusted because it results somehow in the wrong type.

* Add ros_ign in .repos file.

* Add delay before starting rviz to avoid warning that joint-values are not available.

* Use sustitutions for kinematics_yaml instead of file parsing to have correct parameter types.

* fix ign_ros2_control to working hash.

* Fixup rviz default rviz configuration when moveit is not used.

* Do not add camera links because they are and should be added by camera URDF itself.

* Add updated for the simulation.

* Update simulation repositories.

* Add rezilient setup here as workarround.

* Updated to work again and updated simulation parameters.

* remove temp rezilinet file.

* Update urls and versions. (#67)

* Correct Ignition plugin name for ros2_control support.

* Correct joint names for testing node.

* Fix pre-commit.

* Update docs for simulation purposes.

Co-authored-by: Lovro <lovro.ivanov@gmail.com>

File: kortex_description/robots/kortex_robot.xacro (robot description, xacro)
@@ -1,56 +1,73 @@
 <?xml version="1.0"?>
 <robot xmlns:xacro="http://ros.org/wiki/xacro">
-    <xacro:macro name="load_robot" params="parent arm gripper dof vision
-    robot_ip username password port port_realtime session_inactivity_timeout_ms connection_inactivity_timeout_ms
-    sim prefix use_fake_hardware fake_sensor_commands use_internal_bus_gripper_comm:=false">
-        <!-- Files to include -->
-        <xacro:include filename="$(find kortex_description)/arms/${arm}/${dof}dof/urdf/${arm}_macro.xacro" />
-        <xacro:unless value="${not gripper}">
-            <xacro:include filename="$(find kortex_description)/grippers/${gripper}/urdf/${gripper}_macro.xacro" />
-        </xacro:unless>
-        <xacro:if value="${sim}">
-            <!-- Arm transmission elements-->
-            <xacro:include filename="$(find kortex_description)/arms/${arm}/${dof}dof/urdf/${arm}_transmission_macro.xacro" />
-            <!-- Gripper transmission elements if there is a gripper-->
-            <xacro:unless value="${not gripper}">
-                <xacro:include filename="$(find kortex_description)/grippers/${gripper}/urdf/${gripper}_transmission_macro.xacro" />
-            </xacro:unless>
-        </xacro:if>
-        <!-- Run the macros -->
-        <!-- Load the arm -->
-        <xacro:load_arm parent="${parent}" dof="${dof}" vision="${vision}"
-                        robot_ip="${robot_ip}" username="${username}" password="${password}" port="${port}" port_realtime="${port_realtime}"
-                        session_inactivity_timeout_ms="${session_inactivity_timeout_ms}" connection_inactivity_timeout_ms="${connection_inactivity_timeout_ms}"
-                        prefix="${prefix}" use_fake_hardware="${use_fake_hardware}" fake_sensor_commands="${fake_sensor_commands}"
-                        use_internal_bus_gripper_comm="${use_internal_bus_gripper_comm}">
-            <origin xyz="0 0 0" rpy="0 0 0"/>
-        </xacro:load_arm>
-        <!-- Load the gripper -->
-        <xacro:unless value="${not gripper}">
-            <!-- last_arm_link is defined in "$(find kortex_description)/arms/${arm}/urdf/${arm}_macro.xacro" -->
-            <xacro:load_gripper parent="${prefix}${last_arm_link}"  prefix="${prefix}"/>
-        </xacro:unless>
-        <!-- If no gripper, define tool frame here -->
-        <xacro:if value="${not gripper}">
-            <link name="${prefix}tool_frame"/>
-            <joint name="${prefix}tool_frame_joint" type="fixed">
-                <origin xyz="0 0 0" rpy="0 0 0" />
-                <parent link="${prefix}${last_arm_link}" />
-                <child link="${prefix}tool_frame" />
-                <axis xyz="0 0 0" />
-            </joint>
-        </xacro:if>
-        <!-- Load the Gazebo transmissions and gazebo_ros_control plugin -->
-        <xacro:if value="${sim}">
-            <xacro:load_gazebo_arm_transmissions prefix="${prefix}"/>
-            <xacro:unless value="${not gripper}">
-                <xacro:load_gazebo_gripper_transmissions prefix="${prefix}"/>
-            </xacro:unless>
-            <gazebo>
-                <plugin name="gazebo_ros_control" filename="libgazebo_ros_control.so">
-                    <legacyModeNS>true</legacyModeNS>
-                </plugin>
-            </gazebo>
-        </xacro:if>
-    </xacro:macro>
+  <xacro:macro name="load_robot" params="
+    parent
+    *origin
+    prefix
+    arm
+    gripper
+    dof
+    vision
+    robot_ip
+    username
+    password
+    port
+    port_realtime
+    session_inactivity_timeout_ms
+    connection_inactivity_timeout_ms
+    use_internal_bus_gripper_comm:=false
+    use_fake_hardware:=false
+    fake_sensor_commands:=false
+    sim_gazebo:=false
+    sim_ignition:=false" >
+    <!-- Include and load arm macro files -->
+    <xacro:include filename="$(find kortex_description)/arms/${arm}/${dof}dof/urdf/${arm}_macro.xacro" />
+    <!-- Load the arm -->
+    <xacro:load_arm
+      parent="${parent}"
+      dof="${dof}"
+      vision="${vision}"
+      robot_ip="${robot_ip}"
+      username="${username}"
+      password="${password}"
+      port="${port}"
+      port_realtime="${port_realtime}"
+      session_inactivity_timeout_ms="${session_inactivity_timeout_ms}"
+      connection_inactivity_timeout_ms="${connection_inactivity_timeout_ms}"
+      prefix="${prefix}"
+      use_internal_bus_gripper_comm="${use_internal_bus_gripper_comm}"
+      use_fake_hardware="${use_fake_hardware}"
+      fake_sensor_commands="${fake_sensor_commands}"
+      sim_gazebo="${sim_gazebo}"
+      sim_ignition="${sim_ignition}" >
+      <xacro:insert_block name="origin" />
+    </xacro:load_arm>
+    <!-- If no gripper, define tool frame here -->
+    <xacro:if value="${not gripper}">
+      <link name="${prefix}tool_frame"/>
+      <joint name="${prefix}tool_frame_joint" type="fixed">
+        <origin xyz="0 0 0" rpy="0 0 0" />
+        <parent link="${prefix}${last_arm_link}" />
+        <child link="${prefix}tool_frame" />
+        <axis xyz="0 0 0" />
+      </joint>
+    </xacro:if>
+    <!-- Include and load the gripper if defined -->
+    <xacro:unless value="${not gripper}">
+      <xacro:include filename="$(find kortex_description)/grippers/${gripper}/urdf/${gripper}_macro.xacro" />
+      <!-- last_arm_link is defined in "$(find kortex_description)/arms/${arm}/urdf/${arm}_macro.xacro" -->
+      <xacro:load_gripper parent="${prefix}${last_arm_link}"  prefix="${prefix}"/>
+    </xacro:unless>
+    <!-- Load the Gazebo transmissions and gazebo_ros_control plugin -->
+    <xacro:if value="${sim_gazebo or sim_ignition}">
+      <!-- Arm transmission elements-->
+      <xacro:include filename="$(find kortex_description)/arms/${arm}/${dof}dof/urdf/${arm}_transmission_macro.xacro" />
+      <xacro:load_gazebo_arm_transmissions prefix="${prefix}"/>
+      <!-- Gripper transmission elements if there is a gripper-->
+      <xacro:unless value="${not gripper}">
+        <xacro:include filename="$(find kortex_description)/grippers/${gripper}/urdf/${gripper}_transmission_macro.xacro" />
+        <xacro:load_gazebo_gripper_transmissions prefix="${prefix}"/>
+      </xacro:unless>
+    </xacro:if>
+  </xacro:macro>
 </robot>

File: kortex_move_it_config/gen3_move_it_config/config/7dof/gen3.srdf.xacro (robot description, xacro)
@@ -4,5 +4,8 @@
     A URDF file must exist for this robot as well, where the joints and the links that are referenced are defined
 -->
-<robot name="gen3" xmlns:xacro="http://www.ros.org/wiki/xacro">
+<robot xmlns:xacro="http://www.ros.org/wiki/xacro" name="$(arg name)">
+    <!-- robot name parameter -->
+    <xacro:arg name="name" default="arm"/>
+    <!-- parameters -->
     <xacro:arg name="prefix" default="" />
     <!--GROUPS - Representation of a set of joints and links. This can be useful for specifying DOF to plan for, defining arms, end effectors, etc-->
@@ -11,6 +14,6 @@
     <!--CHAINS - When a chain is specified, all the links along the chain (including endpoints) are included in the group. Additionally, all the joints that are parents to included links are also included. This means that joints along the chain and the parent joint of the base link are included in the group-->
     <!--SUBGROUPS - Groups can also be formed by referencing to already defined group names-->
-    <group name="arm">
-        <joint name="$(arg prefix)joint_1" />
+    <group name="$(arg name)">
+<!--        <joint name="$(arg prefix)joint_1" />
         <joint name="$(arg prefix)joint_2" />
         <joint name="$(arg prefix)joint_3" />
@@ -20,8 +23,9 @@
         <joint name="$(arg prefix)joint_7" />
         <joint name="$(arg prefix)end_effector" />
-        <joint name="$(arg prefix)tool_frame_joint" />
+        <joint name="$(arg prefix)tool_frame_joint" />-->
+        <chain base_link="$(arg prefix)base_link" tip_link="$(arg prefix)end_effector_link" />
     </group>
     <!--GROUP STATES - Purpose - Define a named state for a particular group, in terms of joint values. This is useful to define states like 'folded arms'-->
-    <group_state name="home" group="arm">
+    <group_state name="$(arg prefix)home" group="$(arg name)">
         <joint name="$(arg prefix)joint_1" value="0" />
         <joint name="$(arg prefix)joint_2" value="0.26" />
@@ -32,5 +36,5 @@
         <joint name="$(arg prefix)joint_7" value="1.57" />
     </group_state>
-    <group_state name="retract" group="arm">
+    <group_state name="$(arg prefix)retract" group="$(arg name)">
         <joint name="$(arg prefix)joint_1" value="0" />
         <joint name="$(arg prefix)joint_2" value="-0.35" />
@@ -41,5 +45,5 @@
         <joint name="$(arg prefix)joint_7" value="1.57" />
     </group_state>
-    <group_state name="vertical" group="arm">
+    <group_state name="$(arg prefix)vertical" group="$(arg name)">
         <joint name="$(arg prefix)joint_1" value="0" />
         <joint name="$(arg prefix)joint_2" value="0" />

Commit message: Revert joint2 limit to factory values

File: kortex_description/arms/gen3/7dof/urdf/gen3_macro.xacro (robot description, xacro)
@@ -135,5 +135,5 @@
       <axis
         xyz="0 0 1" />
-      <limit lower="-1.4" upper="1.4" effort="39" velocity="1.3963" />
+      <limit lower="-2.41" upper="2.41" effort="39" velocity="1.3963" />
     </joint>
     <link name="${prefix}half_arm_2_link">

Commit message: Update gen3 URDF mesh path

File: kortex_description/arms/gen3/7dof/urdf/gen3_macro.xacro (robot description, xacro)
@@ -54,14 +54,14 @@
         <origin xyz="0 0 0" rpy="0 0 0" />
         <geometry>
-          <mesh filename="file://$(find kortex_description)/arms/gen3/${dof}dof/meshes/base_link.STL" />
-        </geometry>
-        <material name="">
-          <color rgba="0.75294 0.75294 0.75294 1" />
-        </material>
-      </visual>
-      <collision>
-        <origin xyz="0 0 0" rpy="0 0 0" />
-        <geometry>
-          <mesh filename="file://$(find kortex_description)/arms/gen3/${dof}dof/meshes/base_link.STL" />
+          <mesh filename="package://kortex_description/arms/gen3/${dof}dof/meshes/base_link.STL" />
+        </geometry>
+        <material name="">
+          <color rgba="0.75294 0.75294 0.75294 1" />
+        </material>
+      </visual>
+      <collision>
+        <origin xyz="0 0 0" rpy="0 0 0" />
+        <geometry>
+          <mesh filename="package://kortex_description/arms/gen3/${dof}dof/meshes/base_link.STL" />
         </geometry>
       </collision>
@@ -76,14 +76,14 @@
         <origin xyz="0 0 0" rpy="0 0 0" />
         <geometry>
-          <mesh filename="file://$(find kortex_description)/arms/gen3/${dof}dof/meshes/shoulder_link.STL" />
-        </geometry>
-        <material name="">
-          <color rgba="0.75294 0.75294 0.75294 1" />
-        </material>
-      </visual>
-      <collision>
-        <origin xyz="0 0 0" rpy="0 0 0" />
-        <geometry>
-          <mesh filename="file://$(find kortex_description)/arms/gen3/${dof}dof/meshes/shoulder_link.STL" />
+          <mesh filename="package://kortex_description/arms/gen3/${dof}dof/meshes/shoulder_link.STL" />
+        </geometry>
+        <material name="">
+          <color rgba="0.75294 0.75294 0.75294 1" />
+        </material>
+      </visual>
+      <collision>
+        <origin xyz="0 0 0" rpy="0 0 0" />
+        <geometry>
+          <mesh filename="package://kortex_description/arms/gen3/${dof}dof/meshes/shoulder_link.STL" />
         </geometry>
       </collision>
@@ -112,14 +112,14 @@
         <origin xyz="0 0 0" rpy="0 0 0" />
         <geometry>
-          <mesh filename="file://$(find kortex_description)/arms/gen3/${dof}dof/meshes/half_arm_1_link.STL" />
-        </geometry>
-        <material name="">
-          <color rgba="0.75294 0.75294 0.75294 1" />
-        </material>
-      </visual>
-      <collision>
-        <origin xyz="0 0 0" rpy="0 0 0" />
-        <geometry>
-          <mesh filename="file://$(find kortex_description)/arms/gen3/${dof}dof/meshes/half_arm_1_link.STL" />
+          <mesh filename="package://kortex_description/arms/gen3/${dof}dof/meshes/half_arm_1_link.STL" />
+        </geometry>
+        <material name="">
+          <color rgba="0.75294 0.75294 0.75294 1" />
+        </material>
+      </visual>
+      <collision>
+        <origin xyz="0 0 0" rpy="0 0 0" />
+        <geometry>
+          <mesh filename="package://kortex_description/arms/gen3/${dof}dof/meshes/half_arm_1_link.STL" />
         </geometry>
       </collision>
@@ -146,14 +146,14 @@
         <origin xyz="0 0 0" rpy="0 0 0" />
         <geometry>
-          <mesh filename="file://$(find kortex_description)/arms/gen3/${dof}dof/meshes/half_arm_2_link.STL" />
-        </geometry>
-        <material name="">
-          <color rgba="0.75294 0.75294 0.75294 1" />
-        </material>
-      </visual>
-      <collision>
-        <origin xyz="0 0 0" rpy="0 0 0" />
-        <geometry>
-          <mesh filename="file://$(find kortex_description)/arms/gen3/${dof}dof/meshes/half_arm_2_link.STL" />
+          <mesh filename="package://kortex_description/arms/gen3/${dof}dof/meshes/half_arm_2_link.STL" />
+        </geometry>
+        <material name="">
+          <color rgba="0.75294 0.75294 0.75294 1" />
+        </material>
+      </visual>
+      <collision>
+        <origin xyz="0 0 0" rpy="0 0 0" />
+        <geometry>
+          <mesh filename="package://kortex_description/arms/gen3/${dof}dof/meshes/half_arm_2_link.STL" />
         </geometry>
       </collision>
@@ -182,14 +182,14 @@
         <origin xyz="0 0 0" rpy="0 0 0" />
         <geometry>
-          <mesh filename="file://$(find kortex_description)/arms/gen3/${dof}dof/meshes/forearm_link.STL" />
-        </geometry>
-        <material name="">
-          <color rgba="0.75294 0.75294 0.75294 1" />
-        </material>
-      </visual>
-      <collision>
-        <origin xyz="0 0 0" rpy="0 0 0" />
-        <geometry>
-          <mesh filename="file://$(find kortex_description)/arms/gen3/${dof}dof/meshes/forearm_link.STL" />
+          <mesh filename="package://kortex_description/arms/gen3/${dof}dof/meshes/forearm_link.STL" />
+        </geometry>
+        <material name="">
+          <color rgba="0.75294 0.75294 0.75294 1" />
+        </material>
+      </visual>
+      <collision>
+        <origin xyz="0 0 0" rpy="0 0 0" />
+        <geometry>
+          <mesh filename="package://kortex_description/arms/gen3/${dof}dof/meshes/forearm_link.STL" />
         </geometry>
       </collision>
@@ -216,14 +216,14 @@
         <origin xyz="0 0 0" rpy="0 0 0" />
         <geometry>
-          <mesh filename="file://$(find kortex_description)/arms/gen3/${dof}dof/meshes/spherical_wrist_1_link.STL" />
-        </geometry>
-        <material name="">
-          <color rgba="0.75294 0.75294 0.75294 1" />
-        </material>
-      </visual>
-      <collision>
-        <origin xyz="0 0 0" rpy="0 0 0" />
-        <geometry>
-          <mesh filename="file://$(find kortex_description)/arms/gen3/${dof}dof/meshes/spherical_wrist_1_link.STL" />
+          <mesh filename="package://kortex_description/arms/gen3/${dof}dof/meshes/spherical_wrist_1_link.STL" />
+        </geometry>
+        <material name="">
+          <color rgba="0.75294 0.75294 0.75294 1" />
+        </material>
+      </visual>
+      <collision>
+        <origin xyz="0 0 0" rpy="0 0 0" />
+        <geometry>
+          <mesh filename="package://kortex_description/arms/gen3/${dof}dof/meshes/spherical_wrist_1_link.STL" />
         </geometry>
       </collision>
@@ -252,14 +252,14 @@
         <origin xyz="0 0 0" rpy="0 0 0" />
         <geometry>
-          <mesh filename="file://$(find kortex_description)/arms/gen3/${dof}dof/meshes/spherical_wrist_2_link.STL" />
-        </geometry>
-        <material name="">
-          <color rgba="0.75294 0.75294 0.75294 1" />
-        </material>
-      </visual>
-      <collision>
-        <origin xyz="0 0 0" rpy="0 0 0" />
-        <geometry>
-          <mesh filename="file://$(find kortex_description)/arms/gen3/${dof}dof/meshes/spherical_wrist_2_link.STL" />
+          <mesh filename="package://kortex_description/arms/gen3/${dof}dof/meshes/spherical_wrist_2_link.STL" />
+        </geometry>
+        <material name="">
+          <color rgba="0.75294 0.75294 0.75294 1" />
+        </material>
+      </visual>
+      <collision>
+        <origin xyz="0 0 0" rpy="0 0 0" />
+        <geometry>
+          <mesh filename="package://kortex_description/arms/gen3/${dof}dof/meshes/spherical_wrist_2_link.STL" />
         </geometry>
       </collision>
@@ -287,14 +287,14 @@
         <origin xyz="0 0 0" rpy="0 0 0" />
         <geometry>
-          <mesh filename="file://$(find kortex_description)/arms/gen3/${dof}dof/meshes/bracelet_with_vision_link.STL" />
-        </geometry>
-        <material name="">
-          <color rgba="0.75294 0.75294 0.75294 1" />
-        </material>
-      </visual>
-      <collision>
-        <origin xyz="0 0 0" rpy="0 0 0" />
-        <geometry>
-          <mesh filename="file://$(find kortex_description)/arms/gen3/${dof}dof/meshes/bracelet_with_vision_link.STL" />
+          <mesh filename="package://kortex_description/arms/gen3/${dof}dof/meshes/bracelet_with_vision_link.STL" />
+        </geometry>
+        <material name="">
+          <color rgba="0.75294 0.75294 0.75294 1" />
+        </material>
+      </visual>
+      <collision>
+        <origin xyz="0 0 0" rpy="0 0 0" />
+        <geometry>
+          <mesh filename="package://kortex_description/arms/gen3/${dof}dof/meshes/bracelet_with_vision_link.STL" />
         </geometry>
       </collision>
@@ -311,14 +311,14 @@
         <origin xyz="0 0 0" rpy="0 0 0" />
         <geometry>
-          <mesh filename="file://$(find kortex_description)/arms/gen3/${dof}dof/meshes/bracelet_no_vision_link.STL" />
-        </geometry>
-        <material name="">
-          <color rgba="0.75294 0.75294 0.75294 1" />
-        </material>
-      </visual>
-      <collision>
-        <origin xyz="0 0 0" rpy="0 0 0" />
-        <geometry>
-          <mesh filename="file://$(find kortex_description)/arms/gen3/${dof}dof/meshes/bracelet_no_vision_link.STL" />
+          <mesh filename="package://kortex_description/arms/gen3/${dof}dof/meshes/bracelet_no_vision_link.STL" />
+        </geometry>
+        <material name="">
+          <color rgba="0.75294 0.75294 0.75294 1" />
+        </material>
+      </visual>
+      <collision>
+        <origin xyz="0 0 0" rpy="0 0 0" />
+        <geometry>
+          <mesh filename="package://kortex_description/arms/gen3/${dof}dof/meshes/bracelet_no_vision_link.STL" />
         </geometry>
       </collision>
