Commit message: Add gazebo plugins to enable sim camera

File: kortex_description/arms/gen3/7dof/urdf/gen3_macro.xacro (robot description, xacro)
@@ -292,5 +292,5 @@
         </geometry>
         <material name="">
-          <color rgba="0.75294 0.75294 0.75294 1" />
+          <color rgba="0.75294 0 0 1" />
         </material>
       </visual>
@@ -357,5 +357,5 @@
       <link name="${prefix}camera_link" />
       <joint name="${prefix}camera_module" type="fixed">
-        <origin xyz="0 0.05639 -0.00305" rpy="3.14159265358979 3.14159265358979 0" />
+        <origin xyz="0 0.05639 0.01305" rpy="0 -1.570796326794897 -1.570796326794897" />
         <parent link="${prefix}end_effector_link" />
         <child  link="${prefix}camera_link" />
@@ -363,5 +363,5 @@
       <link name="${prefix}camera_depth_frame" />
       <joint name="${prefix}depth_module" type="fixed">
-        <origin xyz="0.0275 0.066 -0.00305" rpy="3.14159265358979 3.14159265358979 0" />
+        <origin xyz="0.0275 0.066 0.01305" rpy="0 -1.570796326794897 -1.570796326794897" />
         <parent link="${prefix}end_effector_link" />
         <child  link="${prefix}camera_depth_frame" />
@@ -369,5 +369,5 @@
       <link name="${prefix}camera_color_frame" />
       <joint name="${prefix}color_module" type="fixed">
-        <origin xyz="0 0.05639 -0.00305" rpy="3.14159265358979 3.14159265358979 0" />
+        <origin xyz="0 0.05639 0.01305" rpy="0 -1.570796326794897 -1.570796326794897" />
         <parent link="${prefix}end_effector_link" />
         <child  link="${prefix}camera_color_frame" />

File: kortex_description/robots/kinova.urdf.xacro (robot description, xacro)
@@ -22,4 +22,7 @@
   <xacro:arg name="sim_ignition" default="false" />
   <xacro:arg name="sim_isaac" default="false" />
+  <xacro:arg name="gazebo_renderer" default="ogre"/>
+  <xacro:arg name="gazebo_camera_fps" default="6"/>
+  <xacro:arg name="simulate_depth" default="true"/>
   <xacro:arg name="simulation_controllers" default="$(find kortex_description)/arm/$(arg arm)/$(arg dof)dof/config/ros2_controllers.yaml" />
   <!-- import main macro -->
@@ -60,4 +63,11 @@
   </xacro:if>
   <xacro:if value="$(arg sim_ignition)">
+    <!-- Configure simulated camera -->
+    <xacro:if value="$(arg simulate_depth)">
+      <xacro:property name="sim_sensor_type" value="rgbd_camera" />
+    </xacro:if>
+    <xacro:unless value="$(arg simulate_depth)">
+      <xacro:property name="sim_sensor_type" value="camera" />
+    </xacro:unless>
     <!-- Gazebo plugins -->
     <gazebo reference="world">
@@ -68,4 +78,70 @@
         <controller_manager_node_name>$(arg prefix)controller_manager</controller_manager_node_name>
       </plugin>
+      <plugin filename="libignition-gazebo-sensors-system.so" name="ignition::gazebo::systems::Sensors">
+        <render_engine>$(arg gazebo_renderer)</render_engine>
+      </plugin>
+    </gazebo>
+    <gazebo reference="camera_color_frame">
+      <sensor name="camera_sensor" type="${sim_sensor_type}">
+        <camera>
+          <horizontal_fov>1.047</horizontal_fov>
+          <image>
+            <width>640</width>
+            <height>480</height>
+            <format>RGB_INT8</format>
+          </image>
+          <clip>
+            <near>0.1</near>
+            <far>5</far>
+          </clip>
+          <distortion>
+            <k1>0.0</k1>
+            <k2>0.0</k2>
+            <k3>0.0</k3>
+            <p1>0.0</p1>
+            <p2>0.0</p2>
+            <center>0.5 0.5</center>
+          </distortion>
+          <lens>
+            <intrinsics>
+              <fx>554.25469</fx>
+              <fy>554.25469</fy>
+              <cx>320.5</cx>
+              <cy>240.5</cy>
+              <s>0</s>
+            </intrinsics>
+            <!-- These need to match the intrinsics above or
+            Ignition will default to different default values -->
+            <projection>
+              <p_fx>554.25469</p_fx>
+              <p_fy>554.25469</p_fy>
+              <p_cx>320.5</p_cx>
+              <p_cy>240.5</p_cy>
+              <tx>0</tx>
+              <ty>0</ty>
+            </projection>
+          </lens>
+          <noise>
+            <type>gaussian</type>
+            <mean>0</mean>
+            <stddev>0.00</stddev>
+          </noise>
+          <xacro:if value="$(arg simulate_depth)">
+            <depth_camera>
+              <clip>
+                <near>0.25</near>
+                <far>5</far>
+              </clip>
+            </depth_camera>
+          </xacro:if>
+          <optical_frame_id>color_optical_frame</optical_frame_id>
+        </camera>
+        <ignition_frame_id>camera_color_frame</ignition_frame_id>
+        <always_on>1</always_on>
+        <update_rate>$(arg gazebo_camera_fps)</update_rate>
+        <visualize>true</visualize>
+        <topic>wrist_mounted_camera</topic>
+        <enable_metrics>false</enable_metrics>
+      </sensor>
     </gazebo>
   </xacro:if>

Commit message: update parameters

File: kortex_description/arms/gen3/7dof/urdf/gen3_macro.xacro (robot description, xacro)
@@ -355,22 +355,45 @@
     <!-- TODO(destogl) this probably collides with camera URDF -->
     <xacro:if value="${vision}">
-      <link name="${prefix}camera_link" />
-      <joint name="${prefix}camera_module" type="fixed">
-        <origin xyz="0 0.05639 0.01305" rpy="0 -1.570796326794897 -1.570796326794897" />
-        <parent link="${prefix}end_effector_link" />
-        <child  link="${prefix}camera_link" />
-      </joint>
-      <link name="${prefix}camera_depth_frame" />
-      <joint name="${prefix}depth_module" type="fixed">
-        <origin xyz="0.0275 0.066 0.01305" rpy="0 -1.570796326794897 -1.570796326794897" />
-        <parent link="${prefix}end_effector_link" />
-        <child  link="${prefix}camera_depth_frame" />
-      </joint>
-      <link name="${prefix}camera_color_frame" />
-      <joint name="${prefix}color_module" type="fixed">
-        <origin xyz="0 0.05639 0.01305" rpy="0 -1.570796326794897 -1.570796326794897" />
-        <parent link="${prefix}end_effector_link" />
-        <child  link="${prefix}camera_color_frame" />
-      </joint>
+      <!-- sim camera needs to be rotated which might not apply to built in vision module -->
+      <xacro:if value="${sim_ignition}">
+        <link name="${prefix}camera_link" />
+        <joint name="${prefix}camera_module" type="fixed">
+          <origin xyz="0 0.05639 0.01305" rpy="0 -1.570796326794897 -1.570796326794897" />
+          <parent link="${prefix}end_effector_link" />
+          <child  link="${prefix}camera_link" />
+        </joint>
+        <link name="${prefix}camera_depth_frame" />
+        <joint name="${prefix}depth_module" type="fixed">
+          <origin xyz="0.0275 0.066 0.01305" rpy="0 -1.570796326794897 -1.570796326794897" />
+          <parent link="${prefix}end_effector_link" />
+          <child  link="${prefix}camera_depth_frame" />
+        </joint>
+        <link name="${prefix}camera_color_frame" />
+        <joint name="${prefix}color_module" type="fixed">
+          <origin xyz="0 0.05639 0.01305" rpy="0 -1.570796326794897 -1.570796326794897" />
+          <parent link="${prefix}end_effector_link" />
+          <child  link="${prefix}camera_color_frame" />
+        </joint>
+      </xacro:if>
+      <xacro:unless value="${sim_ignition}">
+        <link name="${prefix}camera_link" />
+        <joint name="${prefix}camera_module" type="fixed">
+          <origin xyz="0 0.05639 0.01305" rpy="0 -1.570796326794897 -1.570796326794897" />
+          <parent link="${prefix}end_effector_link" />
+          <child  link="${prefix}camera_link" />
+        </joint>
+        <link name="${prefix}camera_depth_frame" />
+        <joint name="${prefix}depth_module" type="fixed">
+          <origin xyz="0.0275 0.066 0.01305" rpy="0 -1.570796326794897 -1.570796326794897" />
+          <parent link="${prefix}end_effector_link" />
+          <child  link="${prefix}camera_depth_frame" />
+        </joint>
+        <link name="${prefix}camera_color_frame" />
+        <joint name="${prefix}color_module" type="fixed">
+          <origin xyz="0 0.05639 0.01305" rpy="0 -1.570796326794897 -1.570796326794897" />
+          <parent link="${prefix}end_effector_link" />
+          <child  link="${prefix}camera_color_frame" />
+        </joint>
+      </xacro:unless>
     </xacro:if>
   </xacro:macro>

File: kortex_description/robots/kinova.urdf.xacro (robot description, xacro)
@@ -23,6 +23,7 @@
   <xacro:arg name="sim_isaac" default="false" />
   <xacro:arg name="gazebo_renderer" default="ogre"/>
-  <xacro:arg name="gazebo_camera_fps" default="6"/>
-  <xacro:arg name="simulate_depth" default="true"/>
+  <xacro:arg name="camera_width" default="640"/>
+  <xacro:arg name="camera_height" default="480"/>
+  <xacro:arg name="camera_fps" default="6"/>
   <xacro:arg name="simulation_controllers" default="$(find kortex_description)/arm/$(arg arm)/$(arg dof)dof/config/ros2_controllers.yaml" />
   <!-- import main macro -->
@@ -63,11 +64,4 @@
   </xacro:if>
   <xacro:if value="$(arg sim_ignition)">
-    <!-- Configure simulated camera -->
-    <xacro:if value="$(arg simulate_depth)">
-      <xacro:property name="sim_sensor_type" value="rgbd_camera" />
-    </xacro:if>
-    <xacro:unless value="$(arg simulate_depth)">
-      <xacro:property name="sim_sensor_type" value="camera" />
-    </xacro:unless>
     <!-- Gazebo plugins -->
     <gazebo reference="world">
@@ -83,10 +77,10 @@
     </gazebo>
     <gazebo reference="camera_color_frame">
-      <sensor name="camera_sensor" type="${sim_sensor_type}">
+      <sensor name="camera_sensor" type="rgbd_camera">
         <camera>
           <horizontal_fov>1.047</horizontal_fov>
           <image>
-            <width>640</width>
-            <height>480</height>
+            <width>$(arg camera_width)</width>
+            <height>$(arg camera_height)</height>
             <format>RGB_INT8</format>
           </image>
@@ -127,17 +121,15 @@
             <stddev>0.00</stddev>
           </noise>
-          <xacro:if value="$(arg simulate_depth)">
-            <depth_camera>
-              <clip>
-                <near>0.25</near>
-                <far>5</far>
-              </clip>
-            </depth_camera>
-          </xacro:if>
+          <depth_camera>
+            <clip>
+              <near>0.25</near>
+              <far>5</far>
+            </clip>
+          </depth_camera>
           <optical_frame_id>color_optical_frame</optical_frame_id>
         </camera>
         <ignition_frame_id>camera_color_frame</ignition_frame_id>
         <always_on>1</always_on>
-        <update_rate>$(arg gazebo_camera_fps)</update_rate>
+        <update_rate>$(arg camera_fps)</update_rate>
         <visualize>true</visualize>
         <topic>wrist_mounted_camera</topic>

Commit message: Use PI variable

File: kortex_description/arms/gen3/7dof/urdf/gen3_macro.xacro (robot description, xacro)
@@ -3,4 +3,5 @@
   <!-- Propagate last link name information because it is the gripper's parent link -->
   <xacro:property name="last_arm_link" value="end_effector_link"/>
+  <xacro:property name="PI" value="3.1415926535897931"/>
   <xacro:macro name="load_arm" params="
     parent
@@ -359,5 +360,5 @@
         <link name="${prefix}camera_link" />
         <joint name="${prefix}camera_module" type="fixed">
-          <origin xyz="0 0.05639 0.01305" rpy="0 -1.570796326794897 -1.570796326794897" />
+          <origin xyz="0 0.05639 0.01305" rpy="0 ${-PI/2} ${-PI/2}" />
           <parent link="${prefix}end_effector_link" />
           <child  link="${prefix}camera_link" />
@@ -365,5 +366,5 @@
         <link name="${prefix}camera_depth_frame" />
         <joint name="${prefix}depth_module" type="fixed">
-          <origin xyz="0.0275 0.066 0.01305" rpy="0 -1.570796326794897 -1.570796326794897" />
+          <origin xyz="0.0275 0.066 0.01305" rpy="0 ${-PI/2} ${-PI/2}" />
           <parent link="${prefix}end_effector_link" />
           <child  link="${prefix}camera_depth_frame" />
@@ -371,5 +372,5 @@
         <link name="${prefix}camera_color_frame" />
         <joint name="${prefix}color_module" type="fixed">
-          <origin xyz="0 0.05639 0.01305" rpy="0 -1.570796326794897 -1.570796326794897" />
+          <origin xyz="0 0.05639 0.01305" rpy="0 ${-PI/2} ${-PI/2}" />
           <parent link="${prefix}end_effector_link" />
           <child  link="${prefix}camera_color_frame" />
@@ -379,5 +380,5 @@
         <link name="${prefix}camera_link" />
         <joint name="${prefix}camera_module" type="fixed">
-          <origin xyz="0 0.05639 0.01305" rpy="0 -1.570796326794897 -1.570796326794897" />
+          <origin xyz="0 0.05639 -0.00305" rpy="${PI} ${PI} 0" />
           <parent link="${prefix}end_effector_link" />
           <child  link="${prefix}camera_link" />
@@ -385,5 +386,5 @@
         <link name="${prefix}camera_depth_frame" />
         <joint name="${prefix}depth_module" type="fixed">
-          <origin xyz="0.0275 0.066 0.01305" rpy="0 -1.570796326794897 -1.570796326794897" />
+          <origin xyz="0.0275 0.066 -0.00305" rpy="${PI} ${PI} 0" />
           <parent link="${prefix}end_effector_link" />
           <child  link="${prefix}camera_depth_frame" />
@@ -391,5 +392,5 @@
         <link name="${prefix}camera_color_frame" />
         <joint name="${prefix}color_module" type="fixed">
-          <origin xyz="0 0.05639 0.01305" rpy="0 -1.570796326794897 -1.570796326794897" />
+          <origin xyz="0 0.05639 -0.00305" rpy="${PI} ${PI} 0" />
           <parent link="${prefix}end_effector_link" />
           <child  link="${prefix}camera_color_frame" />

Commit message: Add camera to 7dof gen3 ignition sim (#141)
* Add gazebo plugins to enable sim camera

* cleanup

* update parameters

* Use PI variable

* Update kortex_moveit_config/kinova_gen3_7dof_robotiq_2f_85_moveit_config/launch/sim.launch.py

---------

Co-authored-by: Alex Moriarty <alex.moriarty@picknik.ai>

File: kortex_description/arms/gen3/7dof/urdf/gen3_macro.xacro (robot description, xacro)
@@ -3,4 +3,5 @@
   <!-- Propagate last link name information because it is the gripper's parent link -->
   <xacro:property name="last_arm_link" value="end_effector_link"/>
+  <xacro:property name="PI" value="3.1415926535897931"/>
   <xacro:macro name="load_arm" params="
     parent
@@ -355,22 +356,45 @@
     <!-- TODO(destogl) this probably collides with camera URDF -->
     <xacro:if value="${vision}">
-      <link name="${prefix}camera_link" />
-      <joint name="${prefix}camera_module" type="fixed">
-        <origin xyz="0 0.05639 -0.00305" rpy="3.14159265358979 3.14159265358979 0" />
-        <parent link="${prefix}end_effector_link" />
-        <child  link="${prefix}camera_link" />
-      </joint>
-      <link name="${prefix}camera_depth_frame" />
-      <joint name="${prefix}depth_module" type="fixed">
-        <origin xyz="0.0275 0.066 -0.00305" rpy="3.14159265358979 3.14159265358979 0" />
-        <parent link="${prefix}end_effector_link" />
-        <child  link="${prefix}camera_depth_frame" />
-      </joint>
-      <link name="${prefix}camera_color_frame" />
-      <joint name="${prefix}color_module" type="fixed">
-        <origin xyz="0 0.05639 -0.00305" rpy="3.14159265358979 3.14159265358979 0" />
-        <parent link="${prefix}end_effector_link" />
-        <child  link="${prefix}camera_color_frame" />
-      </joint>
+      <!-- sim camera needs to be rotated which might not apply to built in vision module -->
+      <xacro:if value="${sim_ignition}">
+        <link name="${prefix}camera_link" />
+        <joint name="${prefix}camera_module" type="fixed">
+          <origin xyz="0 0.05639 0.01305" rpy="0 ${-PI/2} ${-PI/2}" />
+          <parent link="${prefix}end_effector_link" />
+          <child  link="${prefix}camera_link" />
+        </joint>
+        <link name="${prefix}camera_depth_frame" />
+        <joint name="${prefix}depth_module" type="fixed">
+          <origin xyz="0.0275 0.066 0.01305" rpy="0 ${-PI/2} ${-PI/2}" />
+          <parent link="${prefix}end_effector_link" />
+          <child  link="${prefix}camera_depth_frame" />
+        </joint>
+        <link name="${prefix}camera_color_frame" />
+        <joint name="${prefix}color_module" type="fixed">
+          <origin xyz="0 0.05639 0.01305" rpy="0 ${-PI/2} ${-PI/2}" />
+          <parent link="${prefix}end_effector_link" />
+          <child  link="${prefix}camera_color_frame" />
+        </joint>
+      </xacro:if>
+      <xacro:unless value="${sim_ignition}">
+        <link name="${prefix}camera_link" />
+        <joint name="${prefix}camera_module" type="fixed">
+          <origin xyz="0 0.05639 -0.00305" rpy="${PI} ${PI} 0" />
+          <parent link="${prefix}end_effector_link" />
+          <child  link="${prefix}camera_link" />
+        </joint>
+        <link name="${prefix}camera_depth_frame" />
+        <joint name="${prefix}depth_module" type="fixed">
+          <origin xyz="0.0275 0.066 -0.00305" rpy="${PI} ${PI} 0" />
+          <parent link="${prefix}end_effector_link" />
+          <child  link="${prefix}camera_depth_frame" />
+        </joint>
+        <link name="${prefix}camera_color_frame" />
+        <joint name="${prefix}color_module" type="fixed">
+          <origin xyz="0 0.05639 -0.00305" rpy="${PI} ${PI} 0" />
+          <parent link="${prefix}end_effector_link" />
+          <child  link="${prefix}camera_color_frame" />
+        </joint>
+      </xacro:unless>
     </xacro:if>
   </xacro:macro>

File: kortex_description/robots/kinova.urdf.xacro (robot description, xacro)
@@ -22,4 +22,8 @@
   <xacro:arg name="sim_ignition" default="false" />
   <xacro:arg name="sim_isaac" default="false" />
+  <xacro:arg name="gazebo_renderer" default="ogre"/>
+  <xacro:arg name="camera_width" default="640"/>
+  <xacro:arg name="camera_height" default="480"/>
+  <xacro:arg name="camera_fps" default="6"/>
   <xacro:arg name="simulation_controllers" default="$(find kortex_description)/arm/$(arg arm)/$(arg dof)dof/config/ros2_controllers.yaml" />
   <!-- import main macro -->
@@ -68,4 +72,68 @@
         <controller_manager_node_name>$(arg prefix)controller_manager</controller_manager_node_name>
       </plugin>
+      <plugin filename="libignition-gazebo-sensors-system.so" name="ignition::gazebo::systems::Sensors">
+        <render_engine>$(arg gazebo_renderer)</render_engine>
+      </plugin>
+    </gazebo>
+    <gazebo reference="camera_color_frame">
+      <sensor name="camera_sensor" type="rgbd_camera">
+        <camera>
+          <horizontal_fov>1.047</horizontal_fov>
+          <image>
+            <width>$(arg camera_width)</width>
+            <height>$(arg camera_height)</height>
+            <format>RGB_INT8</format>
+          </image>
+          <clip>
+            <near>0.1</near>
+            <far>5</far>
+          </clip>
+          <distortion>
+            <k1>0.0</k1>
+            <k2>0.0</k2>
+            <k3>0.0</k3>
+            <p1>0.0</p1>
+            <p2>0.0</p2>
+            <center>0.5 0.5</center>
+          </distortion>
+          <lens>
+            <intrinsics>
+              <fx>554.25469</fx>
+              <fy>554.25469</fy>
+              <cx>320.5</cx>
+              <cy>240.5</cy>
+              <s>0</s>
+            </intrinsics>
+            <!-- These need to match the intrinsics above or
+            Ignition will default to different default values -->
+            <projection>
+              <p_fx>554.25469</p_fx>
+              <p_fy>554.25469</p_fy>
+              <p_cx>320.5</p_cx>
+              <p_cy>240.5</p_cy>
+              <tx>0</tx>
+              <ty>0</ty>
+            </projection>
+          </lens>
+          <noise>
+            <type>gaussian</type>
+            <mean>0</mean>
+            <stddev>0.00</stddev>
+          </noise>
+          <depth_camera>
+            <clip>
+              <near>0.25</near>
+              <far>5</far>
+            </clip>
+          </depth_camera>
+          <optical_frame_id>color_optical_frame</optical_frame_id>
+        </camera>
+        <ignition_frame_id>camera_color_frame</ignition_frame_id>
+        <always_on>1</always_on>
+        <update_rate>$(arg camera_fps)</update_rate>
+        <visualize>true</visualize>
+        <topic>wrist_mounted_camera</topic>
+        <enable_metrics>false</enable_metrics>
+      </sensor>
     </gazebo>
   </xacro:if>
