Commit message: adding missing command interface

File: kortex_description/arms/gen3/7dof/urdf/gen3_macro.xacro (robot description, xacro)
@@ -17,5 +17,8 @@
     session_inactivity_timeout_ms:=6000
     connection_inactivity_timeout_ms:=2000
-    use_internal_bus_gripper_comm:=false
+    use_internal_bus_gripper_comm:=true
+    gripper_joint_name
+    gripper_max_velocity:=100.0
+    gripper_max_force:=100.0
     use_fake_hardware:=false
     fake_sensor_commands:=false
@@ -42,5 +45,8 @@
       session_inactivity_timeout_ms="${session_inactivity_timeout_ms}"
       connection_inactivity_timeout_ms="${connection_inactivity_timeout_ms}"
-      use_internal_bus_gripper_comm="${use_internal_bus_gripper_comm}" />
+      use_internal_bus_gripper_comm="${use_internal_bus_gripper_comm}"
+      gripper_max_velocity="${gripper_max_velocity}"
+      gripper_max_force="${gripper_max_force}"
+      gripper_joint_name="${gripper_joint_name}"/>
     <joint name="${prefix}base_joint" type="fixed">
       <xacro:insert_block name="origin" />

File: kortex_description/arms/gen3/7dof/urdf/kortex.ros2_control.xacro (robot description, xacro)
@@ -19,4 +19,5 @@
     session_inactivity_timeout_ms
     connection_inactivity_timeout_ms
+    gripper_joint_name:=finger_joint
     gripper_max_velocity:=100.0
     gripper_max_force:=100.0">
@@ -50,5 +51,5 @@
           <param name="tf_prefix">"${tf_prefix}"</param>
           <param name="use_internal_bus_gripper_comm">${use_internal_bus_gripper_comm}</param>
-          <param name="gripper_joint_name">finger_joint</param>
+          <param name="gripper_joint_name">${gripper_joint_name}</param>
           <param name="gripper_max_velocity">${gripper_max_velocity}</param>
           <param name="gripper_max_force">${gripper_max_force}</param>
@@ -160,4 +161,19 @@
         <state_interface name="effort"/>
       </joint>
+      <joint name="${prefix}${gripper_joint_name}">
+        <command_interface name="position">
+          <param name="min">{-2*pi}</param>
+          <param name="max">{2*pi}</param>
+        </command_interface>
+        <command_interface name="velocity">
+          <param name="min">-3.2</param>
+          <param name="max">3.2</param>
+        </command_interface>
+        <state_interface name="position">
+          <param name="initial_value">${initial_positions['joint_7']}</param>
+        </state_interface>
+        <state_interface name="velocity"/>
+        <state_interface name="effort"/>
+      </joint>
     </ros2_control>
   </xacro:macro>

File: kortex_description/grippers/robotiq_2f_85/urdf/robotiq_2f_85_macro.xacro (robot description, xacro)
@@ -4,4 +4,5 @@
     parent
     prefix
+    gripper_joint_name:=finger_joint
     use_fake_hardware:=false
     fake_sensor_commands:=false
@@ -25,4 +26,13 @@
         <origin xyz="0 0 0" rpy="0 0 0" />
     </xacro:robotiq_gripper>
+    <xacro:if value="${not sim_ignition or sim_isaac or use_fake_hardware}">
+      <joint name="${prefix}$(gripper_joint_name)">
+        <command_interface name="position" />
+        <state_interface name="position">
+            <param name="initial_value">0.7929</param>
+        </state_interface>
+        <state_interface name="velocity"/>
+      </joint>
+    </xacro:if>
   </xacro:macro>
 </robot>

File: kortex_description/robots/gen3.xacro (robot description, xacro)
@@ -13,4 +13,5 @@
     <xacro:arg name="connection_inactivity_timeout_ms" default="2000" />
     <xacro:arg name="gripper" default="robotiq_2f_85" />
+    <xacro:arg name="gripper_joint_name" default="finger_joint" />
     <xacro:arg name="gripper_max_velocity" default="100.0" />
     <xacro:arg name="gripper_max_force" default="100.0" />
@@ -28,4 +29,5 @@
         arm="$(arg arm)"
         gripper="$(arg gripper)"
+        gripper_joint_name="$(arg gripper_joint_name)"
         gripper_max_velocity="$(arg gripper_max_velocity)"
         gripper_max_force="$(arg gripper_max_force)"

File: kortex_description/robots/kinova.urdf.xacro (robot description, xacro)
@@ -16,4 +16,7 @@
   <xacro:arg name="connection_inactivity_timeout_ms" default="2000" />
   <xacro:arg name="gripper" default="robotiq_2f_85" />
+  <xacro:arg name="gripper_joint_name" default="finger_joint" />
+  <xacro:arg name="gripper_max_velocity" default="100.0" />
+  <xacro:arg name="gripper_max_force" default="100.0" />
   <xacro:arg name="use_internal_bus_gripper_comm" default="false" />
   <xacro:arg name="use_fake_hardware" default="false" />
@@ -35,4 +38,7 @@
     arm="$(arg arm)"
     gripper="$(arg gripper)"
+    gripper_joint_name="$(arg gripper_joint_name)"
+    gripper_max_velocity="$(arg gripper_max_velocity)"
+    gripper_max_force="$(arg gripper_max_force)"
     dof="$(arg dof)"
     vision="$(arg vision)"

File: kortex_description/robots/kortex_robot.xacro (robot description, xacro)
@@ -7,4 +7,5 @@
     arm
     gripper
+    gripper_joint_name
     dof
     vision
@@ -45,4 +46,5 @@
       sim_ignition="${sim_ignition}"
       sim_isaac="${sim_isaac}"
+      gripper_joint_name="${gripper_joint_name}"
       gripper_max_velocity="${gripper_max_velocity}"
       gripper_max_force="${gripper_max_force}">
@@ -66,4 +68,5 @@
         parent="${prefix}${last_arm_link}"
         prefix="${prefix}"
+        gripper_joint_name="${gripper_joint_name}"
         use_fake_hardware="${use_fake_hardware}"
         fake_sensor_commands="${fake_sensor_commands}"

Commit message: [wip] fixing up xacros

File: kortex_description/arms/gen3/7dof/urdf/gen3_macro.xacro (robot description, xacro)
@@ -360,5 +360,4 @@
         xyz="0 0 0" />
     </joint>
-    <!-- TODO(destogl) this probably collides with camera URDF -->
     <xacro:if value="${vision}">
       <!-- sim camera needs to be rotated which might not apply to built in vision module -->

File: kortex_description/arms/gen3/7dof/urdf/kortex.ros2_control.xacro (robot description, xacro)
@@ -19,5 +19,5 @@
     session_inactivity_timeout_ms
     connection_inactivity_timeout_ms
-    gripper_joint_name:=finger_joint
+    gripper_joint_name
     gripper_max_velocity:=100.0
     gripper_max_force:=100.0">
@@ -161,19 +161,4 @@
         <state_interface name="effort"/>
       </joint>
-      <joint name="${prefix}${gripper_joint_name}">
-        <command_interface name="position">
-          <param name="min">{-2*pi}</param>
-          <param name="max">{2*pi}</param>
-        </command_interface>
-        <command_interface name="velocity">
-          <param name="min">-3.2</param>
-          <param name="max">3.2</param>
-        </command_interface>
-        <state_interface name="position">
-          <param name="initial_value">${initial_positions['joint_7']}</param>
-        </state_interface>
-        <state_interface name="velocity"/>
-        <state_interface name="effort"/>
-      </joint>
     </ros2_control>
   </xacro:macro>

File: kortex_description/grippers/robotiq_2f_85/urdf/robotiq_2f_85_macro.xacro (robot description, xacro)
@@ -4,9 +4,9 @@
     parent
     prefix
-    gripper_joint_name:=finger_joint
     use_fake_hardware:=false
     fake_sensor_commands:=false
     sim_ignition:=false
-    sim_isaac:=false">
+    sim_isaac:=false
+    use_internal_bus_gripper_comm:=true">
     <xacro:include filename="$(find robotiq_description)/urdf/robotiq_2f_85_macro.urdf.xacro" />
     <!-- Hardware talks directly to the gripper so we don't need ros2_control unless we are simulating -->
@@ -26,12 +26,14 @@
         <origin xyz="0 0 0" rpy="0 0 0" />
     </xacro:robotiq_gripper>
-    <xacro:if value="${not sim_ignition or sim_isaac or use_fake_hardware}">
-      <joint name="${prefix}$(gripper_joint_name)">
-        <command_interface name="position" />
-        <state_interface name="position">
+    <xacro:if value="${use_internal_bus_gripper_comm}">
+      <xacro:if value="${not include_ros2_control}">
+        <joint name="${prefix}robotiq_85_left_knuckle_joint">
+          <command_interface name="position" />
+          <state_interface name="position">
             <param name="initial_value">0.7929</param>
-        </state_interface>
-        <state_interface name="velocity"/>
-      </joint>
+          </state_interface>
+          <state_interface name="velocity"/>
+        </joint>
+      </xacro:if>
     </xacro:if>
   </xacro:macro>

Commit message: update 7dof urdf

File: kortex_description/arms/gen3/7dof/urdf/gen3_macro.xacro (robot description, xacro)
@@ -26,4 +26,5 @@
     sim_ignition:=false
     sim_isaac:=false
+    use_external_cable:=false
     initial_positions:=${dict(joint_1=0.0,joint_2=0.0,joint_3=0.0,joint_4=0.0,joint_5=0.0,joint_6=0.0,joint_7=0.0)}" >
     <!-- ros2 control include -->
@@ -98,18 +99,38 @@
       </collision>
     </link>
-    <joint
+    <xacro:if value="${use_external_cable}">
+      <joint
       name="${prefix}joint_1"
-      type="continuous">
-      <origin xyz="0 0 0.15643" rpy="3.1416 2.7629E-18 -4.9305E-36" />
-      <parent
-        link="${prefix}base_link" />
-      <child
-        link="${prefix}shoulder_link" />
-      <axis
-        xyz="0 0 1" />
-      <limit
-        effort="39"
-        velocity="1.3963" />
-    </joint>
+      type="revolute">
+        <origin xyz="0 0 0.15643" rpy="3.1416 2.7629E-18 -4.9305E-36" />
+        <parent
+          link="${prefix}base_link" />
+        <child
+          link="${prefix}shoulder_link" />
+        <axis
+          xyz="0 0 1" />
+        <limit
+          lower="${-2*PI}"
+          upper="${2*PI}"
+          effort="39"
+          velocity="1.3963" />
+      </joint>
+    </xacro:if>
+    <xacro:unless value="${use_external_cable}">
+      <joint
+        name="${prefix}joint_1"
+        type="continuous">
+        <origin xyz="0 0 0.15643" rpy="3.1416 2.7629E-18 -4.9305E-36" />
+        <parent
+          link="${prefix}base_link" />
+        <child
+          link="${prefix}shoulder_link" />
+        <axis
+          xyz="0 0 1" />
+        <limit
+          effort="39"
+          velocity="1.3963" />
+      </joint>
+    </xacro:unless>
     <link name="${prefix}half_arm_1_link">
       <inertial>
@@ -168,18 +189,38 @@
       </collision>
     </link>
-    <joint
-      name="${prefix}joint_3"
-      type="continuous">
-      <origin xyz="0 -0.21038 -0.006375" rpy="-1.5708 1.2326E-32 -2.9122E-16" />
-      <parent
-        link="${prefix}half_arm_1_link" />
-      <child
-        link="${prefix}half_arm_2_link" />
-      <axis
-        xyz="0 0 1" />
-      <limit
-        effort="39"
-        velocity="1.3963" />
-    </joint>
+    <xacro:if value="${use_external_cable}">
+      <joint
+        name="${prefix}joint_3"
+        type="revolute">
+        <origin xyz="0 -0.21038 -0.006375" rpy="-1.5708 1.2326E-32 -2.9122E-16" />
+        <parent
+          link="${prefix}half_arm_1_link" />
+        <child
+          link="${prefix}half_arm_2_link" />
+        <axis
+          xyz="0 0 1" />
+        <limit
+          lower="${-2*PI}"
+          upper="${2*PI}"
+          effort="39"
+          velocity="1.3963" />
+      </joint>
+    </xacro:if>
+    <xacro:unless value="${use_external_cable}">
+      <joint
+        name="${prefix}joint_3"
+        type="continuous">
+        <origin xyz="0 -0.21038 -0.006375" rpy="-1.5708 1.2326E-32 -2.9122E-16" />
+        <parent
+          link="${prefix}half_arm_1_link" />
+        <child
+          link="${prefix}half_arm_2_link" />
+        <axis
+          xyz="0 0 1" />
+        <limit
+          effort="39"
+          velocity="1.3963" />
+      </joint>
+    </xacro:unless>
     <link name="${prefix}forearm_link">
       <inertial>
@@ -238,18 +279,38 @@
       </collision>
     </link>
-    <joint
-      name="${prefix}joint_5"
-      type="continuous">
-      <origin xyz="0 -0.20843 -0.006375" rpy="-1.5708 2.2204E-16 -6.373E-17" />
-      <parent
-        link="${prefix}forearm_link" />
-      <child
-        link="${prefix}spherical_wrist_1_link" />
-      <axis
-        xyz="0 0 1" />
-      <limit
-        effort="9"
-        velocity="1.2218" />
-    </joint>
+    <xacro:if value="${use_external_cable}">
+      <joint
+        name="${prefix}joint_5"
+        type="revolute">
+        <origin xyz="0 -0.20843 -0.006375" rpy="-1.5708 2.2204E-16 -6.373E-17" />
+        <parent
+          link="${prefix}forearm_link" />
+        <child
+          link="${prefix}spherical_wrist_1_link" />
+        <axis
+          xyz="0 0 1" />
+        <limit
+          lower="${-2*PI}"
+          upper="${2*PI}"
+          effort="9"
+          velocity="1.2218" />
+      </joint>
+    </xacro:if>
+    <xacro:unless value="${use_external_cable">
+      <joint
+        name="${prefix}joint_5"
+        type="continuous">
+        <origin xyz="0 -0.20843 -0.006375" rpy="-1.5708 2.2204E-16 -6.373E-17" />
+        <parent
+          link="${prefix}forearm_link" />
+        <child
+          link="${prefix}spherical_wrist_1_link" />
+        <axis
+          xyz="0 0 1" />
+        <limit
+          effort="9"
+          velocity="1.2218" />
+      </joint>
+    </xacro:unless>
     <link name="${prefix}spherical_wrist_2_link">
       <inertial>
@@ -334,18 +395,38 @@
     </link>
     </xacro:unless>
-    <joint
-      name="${prefix}joint_7"
-      type="continuous">
-      <origin xyz="0 -0.10593 -0.00017505" rpy="-1.5708 -5.5511E-17 9.6396E-17" />
-      <parent
-        link="${prefix}spherical_wrist_2_link" />
-      <child
-        link="${prefix}bracelet_link" />
-      <axis
-        xyz="0 0 1" />
-      <limit
-        effort="9"
-        velocity="1.2218" />
-    </joint>
+    <xacro:if value="${use_external_cable">
+      <joint
+        name="${prefix}joint_7"
+        type="revolute">
+        <origin xyz="0 -0.10593 -0.00017505" rpy="-1.5708 -5.5511E-17 9.6396E-17" />
+        <parent
+          link="${prefix}spherical_wrist_2_link" />
+        <child
+          link="${prefix}bracelet_link" />
+        <axis
+          xyz="0 0 1" />
+        <limit
+          lower="${-2*PI}"
+          upper="${2*PI}"
+          effort="9"
+          velocity="1.2218" />
+      </joint>
+    </xacro:if>
+    <xacro:unless value="${use_external_cable">
+      <joint
+        name="${prefix}joint_7"
+        type="continuous">
+        <origin xyz="0 -0.10593 -0.00017505" rpy="-1.5708 -5.5511E-17 9.6396E-17" />
+        <parent
+          link="${prefix}spherical_wrist_2_link" />
+        <child
+          link="${prefix}bracelet_link" />
+        <axis
+          xyz="0 0 1" />
+        <limit
+          effort="9"
+          velocity="1.2218" />
+      </joint>
+    </xacro:unless>
     <link name="${prefix}end_effector_link" />
     <joint

Commit message: Fix mention of nonexistent STL file
The STL files were replaced with dae files, but one of the old STL files
is pointed to in the gen3_macro.xacro file. Point to the new dae file
version.

File: kortex_description/arms/gen3/7dof/urdf/gen3_macro.xacro (robot description, xacro)
@@ -370,5 +370,5 @@
         <origin xyz="0 0 0" rpy="0 0 0" />
         <geometry>
-          <mesh filename="file://$(find kortex_description)/arms/gen3/${dof}dof/meshes/bracelet_with_vision_link.STL" />
+          <mesh filename="file://$(find kortex_description)/arms/gen3/${dof}dof/meshes/bracelet_with_vision_link.dae" />
         </geometry>
       </collision>

Commit message: Modified the joint limits of Gen3 and Gen3 Lite robots as per the values in the User Guides

File: kortex_description/arms/gen3/7dof/urdf/gen3_macro.xacro (robot description, xacro)
@@ -169,5 +169,5 @@
       <axis
         xyz="0 0 1" />
-      <limit lower="-2.41" upper="2.41" effort="39" velocity="1.3963" />
+      <limit lower="-2.24" upper="2.24" effort="39" velocity="1.3963" />
     </joint>
     <link name="${prefix}half_arm_2_link">
@@ -259,5 +259,5 @@
       <axis
         xyz="0 0 1" />
-      <limit lower="-2.66" upper="2.66" effort="39" velocity="1.3963" />
+      <limit lower="-2.57" upper="2.57" effort="39" velocity="1.3963" />
     </joint>
     <link name="${prefix}spherical_wrist_1_link">
@@ -349,5 +349,5 @@
       <axis
         xyz="0 0 1" />
-      <limit lower="-2.23" upper="2.23" effort="9" velocity="1.2218" />
+      <limit lower="-2.09" upper="2.09" effort="9" velocity="1.2218" />
     </joint>
     <xacro:if value="${vision}">
