Commit message: update 6dof xacros

File: kortex_description/arms/gen3/6dof/urdf/kortex.ros2_control.xacro (robot description, xacro)
@@ -83,10 +83,10 @@
       <joint name="${prefix}joint_3">
         <command_interface name="position">
-          <param name="min">{-2*pi}</param>
-          <param name="max">{2*pi}</param>
+          <param name="min">-2.66</param>
+          <param name="max">2.66</param>
         </command_interface>
         <command_interface name="velocity">
-          <param name="min">-3.15</param>
-          <param name="max">3.15</param>
+          <param name="min">-3.2</param>
+          <param name="max">3.2</param>
         </command_interface>
         <state_interface name="position">
@@ -98,6 +98,6 @@
       <joint name="${prefix}joint_4">
         <command_interface name="position">
-          <param name="min">-2.66</param>
-          <param name="max">2.66</param>
+          <param name="min">{-2*pi}</param>
+          <param name="max">{2*pi}</param>
         </command_interface>
         <command_interface name="velocity">
@@ -113,6 +113,6 @@
       <joint name="${prefix}joint_5">
         <command_interface name="position">
-          <param name="min">{-2*pi}</param>
-          <param name="max">{2*pi}</param>
+          <param name="min">-2.23</param>
+          <param name="max">2.23</param>
         </command_interface>
         <command_interface name="velocity">
@@ -128,6 +128,6 @@
       <joint name="${prefix}joint_6">
         <command_interface name="position">
-          <param name="min">-2.23</param>
-          <param name="max">2.23</param>
+          <param name="min">{-2*pi}</param>
+          <param name="max">{2*pi}</param>
         </command_interface>
         <command_interface name="velocity">
@@ -141,19 +141,4 @@
         <state_interface name="effort"/>
       </joint>
-      <joint name="${prefix}joint_7">
-        <command_interface name="position">
-          <param name="min">{-2*pi}</param>
-          <param name="max">{2*pi}</param>
-        </command_interface>
-        <command_interface name="velocity">
-          <param name="min">-3.2</param>
-          <param name="max">3.2</param>
-        </command_interface>
-        <state_interface name="position">
-          <param name="initial_value">${initial_positions['joint_7']}</param>
-        </state_interface>
-        <state_interface name="velocity"/>
-        <state_interface name="effort"/>
-      </joint>
     </ros2_control>
   </xacro:macro>

Commit message: Update 6dof description

File: kortex_description/arms/gen3/6dof/urdf/kortex.ros2_control.xacro (robot description, xacro)
@@ -19,4 +19,5 @@
     session_inactivity_timeout_ms
     connection_inactivity_timeout_ms
+    gripper_joint_name
     gripper_max_velocity:=100.0
     gripper_max_force:=100.0">
@@ -50,5 +51,5 @@
           <param name="tf_prefix">"${tf_prefix}"</param>
           <param name="use_internal_bus_gripper_comm">${use_internal_bus_gripper_comm}</param>
-          <param name="gripper_joint_name">finger_joint</param>
+          <param name="gripper_joint_name">${gripper_joint_name}</param>
           <param name="gripper_max_velocity">${gripper_max_velocity}</param>
           <param name="gripper_max_force">${gripper_max_force}</param>
@@ -145,4 +146,11 @@
         <state_interface name="effort"/>
       </joint>
+      <xacro:if value="${use_internal_bus_gripper_comm}">
+        <joint name="${prefix}${gripper_joint_name}">
+          <command_interface name="position" />
+          <state_interface name="position"/>
+          <state_interface name="velocity"/>
+        </joint>
+      </xacro:if>
     </ros2_control>
   </xacro:macro>

Commit message: Make Gripper velocity and force configurable through URDF (#137)
* add params for gripper max force and velocity

Previously the gripper force and velocity were hard coded to 100 they now accept a percentage but default to 100

File: kortex_description/arms/gen3/6dof/urdf/kortex.ros2_control.xacro (robot description, xacro)
@@ -18,5 +18,8 @@
     port_realtime
     session_inactivity_timeout_ms
-    connection_inactivity_timeout_ms">
+    connection_inactivity_timeout_ms
+    gripper_joint_name
+    gripper_max_velocity:=100.0
+    gripper_max_force:=100.0">
     <ros2_control name="${name}" type="system">
       <hardware>
@@ -48,5 +51,7 @@
           <param name="tf_prefix">"${tf_prefix}"</param>
           <param name="use_internal_bus_gripper_comm">${use_internal_bus_gripper_comm}</param>
-          <param name="gripper_joint_name">finger_joint</param>
+          <param name="gripper_joint_name">${gripper_joint_name}</param>
+          <param name="gripper_max_velocity">${gripper_max_velocity}</param>
+          <param name="gripper_max_force">${gripper_max_force}</param>
         </xacro:unless>
       </hardware>
@@ -141,4 +146,11 @@
         <state_interface name="effort"/>
       </joint>
+      <xacro:if value="${use_internal_bus_gripper_comm}">
+        <joint name="${prefix}${gripper_joint_name}">
+          <command_interface name="position" />
+          <state_interface name="position"/>
+          <state_interface name="velocity"/>
+        </joint>
+      </xacro:if>
     </ros2_control>
   </xacro:macro>

File: kortex_description/arms/gen3/7dof/urdf/gen3_macro.xacro (robot description, xacro)
@@ -17,5 +17,8 @@
     session_inactivity_timeout_ms:=6000
     connection_inactivity_timeout_ms:=2000
-    use_internal_bus_gripper_comm:=false
+    use_internal_bus_gripper_comm:=true
+    gripper_joint_name
+    gripper_max_velocity:=100.0
+    gripper_max_force:=100.0
     use_fake_hardware:=false
     fake_sensor_commands:=false
@@ -42,5 +45,8 @@
       session_inactivity_timeout_ms="${session_inactivity_timeout_ms}"
       connection_inactivity_timeout_ms="${connection_inactivity_timeout_ms}"
-      use_internal_bus_gripper_comm="${use_internal_bus_gripper_comm}" />
+      use_internal_bus_gripper_comm="${use_internal_bus_gripper_comm}"
+      gripper_max_velocity="${gripper_max_velocity}"
+      gripper_max_force="${gripper_max_force}"
+      gripper_joint_name="${gripper_joint_name}"/>
     <joint name="${prefix}base_joint" type="fixed">
       <xacro:insert_block name="origin" />
@@ -354,5 +360,4 @@
         xyz="0 0 0" />
     </joint>
-    <!-- TODO(destogl) this probably collides with camera URDF -->
     <xacro:if value="${vision}">
       <!-- sim camera needs to be rotated which might not apply to built in vision module -->

File: kortex_description/arms/gen3/7dof/urdf/kortex.ros2_control.xacro (robot description, xacro)
@@ -9,5 +9,5 @@
     sim_ignition:=false
     sim_isaac:=false
-    use_internal_bus_gripper_comm:=false
+    use_internal_bus_gripper_comm:=true
     tf_prefix
     initial_positions:=${dict(joint_1=0.0,joint_2=0.0,joint_3=0.0,joint_4=0.0,joint_5=0.0,joint_6=0.0,joint_7=0.0)}
@@ -18,5 +18,8 @@
     port_realtime
     session_inactivity_timeout_ms
-    connection_inactivity_timeout_ms">
+    connection_inactivity_timeout_ms
+    gripper_joint_name
+    gripper_max_velocity:=100.0
+    gripper_max_force:=100.0">
     <ros2_control name="${name}" type="system">
       <hardware>
@@ -48,5 +51,7 @@
           <param name="tf_prefix">"${tf_prefix}"</param>
           <param name="use_internal_bus_gripper_comm">${use_internal_bus_gripper_comm}</param>
-          <param name="gripper_joint_name">finger_joint</param>
+          <param name="gripper_joint_name">${gripper_joint_name}</param>
+          <param name="gripper_max_velocity">${gripper_max_velocity}</param>
+          <param name="gripper_max_force">${gripper_max_force}</param>
         </xacro:unless>
       </hardware>
@@ -156,4 +161,11 @@
         <state_interface name="effort"/>
       </joint>
+      <xacro:if value="${use_internal_bus_gripper_comm}">
+        <joint name="${prefix}${gripper_joint_name}">
+          <command_interface name="position" />
+          <state_interface name="position"/>
+          <state_interface name="velocity"/>
+        </joint>
+      </xacro:if>
     </ros2_control>
   </xacro:macro>

File: kortex_description/grippers/robotiq_2f_85/urdf/robotiq_2f_85_macro.xacro (robot description, xacro)
@@ -7,5 +7,6 @@
     fake_sensor_commands:=false
     sim_ignition:=false
-    sim_isaac:=false">
+    sim_isaac:=false
+    use_internal_bus_gripper_comm:=true">
     <xacro:include filename="$(find robotiq_description)/urdf/robotiq_2f_85_macro.urdf.xacro" />
     <!-- Hardware talks directly to the gripper so we don't need ros2_control unless we are simulating -->

File: kortex_description/robots/gen3.xacro (robot description, xacro)
@@ -13,4 +13,7 @@
     <xacro:arg name="connection_inactivity_timeout_ms" default="2000" />
     <xacro:arg name="gripper" default="robotiq_2f_85" />
+    <xacro:arg name="gripper_joint_name" default="finger_joint" />
+    <xacro:arg name="gripper_max_velocity" default="100.0" />
+    <xacro:arg name="gripper_max_force" default="100.0" />
     <xacro:arg name="sim_gazebo" default="false" />
     <xacro:arg name="sim_ignition" default="false" />
@@ -26,4 +29,7 @@
         arm="$(arg arm)"
         gripper="$(arg gripper)"
+        gripper_joint_name="$(arg gripper_joint_name)"
+        gripper_max_velocity="$(arg gripper_max_velocity)"
+        gripper_max_force="$(arg gripper_max_force)"
         dof="$(arg dof)"
         vision="$(arg vision)"

File: kortex_description/robots/kortex_robot.xacro (robot description, xacro)
@@ -7,4 +7,5 @@
     arm
     gripper
+    gripper_joint_name
     dof
     vision
@@ -21,5 +22,7 @@
     sim_gazebo:=false
     sim_ignition:=false
-    sim_isaac:=false" >
+    sim_isaac:=false
+    gripper_max_velocity:=100.0
+    gripper_max_force:=100.0">
     <!-- Include and load arm macro files -->
     <xacro:include filename="$(find kortex_description)/arms/${arm}/${dof}dof/urdf/${arm}_macro.xacro" />
@@ -42,5 +45,8 @@
       sim_gazebo="${sim_gazebo}"
       sim_ignition="${sim_ignition}"
-      sim_isaac="${sim_isaac}" >
+      sim_isaac="${sim_isaac}"
+      gripper_joint_name="${gripper_joint_name}"
+      gripper_max_velocity="${gripper_max_velocity}"
+      gripper_max_force="${gripper_max_force}">
       <xacro:insert_block name="origin" />
     </xacro:load_arm>
