Commit message: [wip] updating 6dof xacros

File: kortex_description/arms/gen3/6dof/urdf/gen3_macro.xacro (robot description, xacro)
@@ -3,5 +3,48 @@
   <!-- Propagate last link name information because it is the gripper's parent link -->
   <xacro:property name="last_arm_link" value="end_effector_link"/>
-  <xacro:macro name="load_arm" params="parent:='' dof vision prefix *origin">
+  <xacro:macro name="load_arm" params="
+    parent
+    dof
+    vision
+    prefix
+    *origin
+    robot_ip
+    username:=admin
+    password:=admin
+    port:=10000
+    port_realtime:=10001
+    session_inactivity_timeout_ms:=6000
+    connection_inactivity_timeout_ms:=2000
+    use_internal_bus_gripper_comm:=false
+    use_fake_hardware:=false
+    fake_sensor_commands:=false
+    sim_gazebo:=false
+    sim_ignition:=false
+    sim_isaac:=false
+    initial_positions:=${dict(joint_1=0.0,joint_2=0.0,joint_3=0.0,joint_4=0.0,joint_5=0.0,joint_6=0.0)}" >
+    <!-- ros2 control include -->
+    <xacro:include filename="$(find kortex_description)/arms/gen3/${dof}dof/urdf/kortex.ros2_control.xacro" />
+    <xacro:kortex_ros2_control
+      name="${prefix}KortexMultiInterfaceHardware" prefix="${prefix}"
+      use_fake_hardware="${use_fake_hardware}"
+      fake_sensor_commands="${fake_sensor_commands}"
+      sim_gazebo="${sim_gazebo}"
+      sim_ignition="${sim_ignition}"
+      sim_isaac="${sim_isaac}"
+      tf_prefix=""
+      initial_positions="${initial_positions}"
+      robot_ip="${robot_ip}"
+      username="${username}"
+      password="${password}"
+      port="${port}"
+      port_realtime="${port_realtime}"
+      session_inactivity_timeout_ms="${session_inactivity_timeout_ms}"
+      connection_inactivity_timeout_ms="${connection_inactivity_timeout_ms}"
+      use_internal_bus_gripper_comm="${use_internal_bus_gripper_comm}" />
+    <joint name="${prefix}base_joint" type="fixed">
+      <xacro:insert_block name="origin" />
+      <parent link="${parent}"/>
+      <child link="${prefix}base_link" />
+    </joint>
     <link name="${prefix}base_link">
       <inertial>
@@ -13,14 +56,14 @@
         <origin xyz="0 0 0" rpy="0 0 0" />
         <geometry>
-          <mesh filename="package://kortex_description/arms/gen3/${dof}dof/meshes/base_link.STL" />
-        </geometry>
-        <material name="">
-          <color rgba="0.75294 0.75294 0.75294 1" />
-        </material>
-      </visual>
-      <collision>
-        <origin xyz="0 0 0" rpy="0 0 0" />
-        <geometry>
-          <mesh filename="package://kortex_description/arms/gen3/${dof}dof/meshes/base_link.STL" />
+          <mesh filename="file://$(find kortex_description)/arms/gen3/${dof}dof/meshes/base_link.STL" />
+        </geometry>
+        <material name="">
+          <color rgba="0.75294 0.75294 0.75294 1" />
+        </material>
+      </visual>
+      <collision>
+        <origin xyz="0 0 0" rpy="0 0 0" />
+        <geometry>
+          <mesh filename="file://$(find kortex_description)/arms/gen3/${dof}dof/meshes/base_link.STL" />
         </geometry>
       </collision>
@@ -35,43 +78,61 @@
         <origin xyz="0 0 0" rpy="0 0 0" />
         <geometry>
-          <mesh filename="package://kortex_description/arms/gen3/${dof}dof/meshes/shoulder_link.STL" />
-        </geometry>
-        <material name="">
-          <color rgba="0.75294 0.75294 0.75294 1" />
-        </material>
-      </visual>
-      <collision>
-        <origin xyz="0 0 0" rpy="0 0 0" />
-        <geometry>
-          <mesh filename="package://kortex_description/arms/gen3/${dof}dof/meshes/shoulder_link.STL" />
-        </geometry>
-      </collision>
-    </link>
-    <joint name="${prefix}joint_1" type="continuous">
-      <origin xyz="0 0 0.15643" rpy="-3.1416 0.0 0.0" />
+          <mesh filename="file://$(find kortex_description)/arms/gen3/${dof}dof/meshes/shoulder_link.STL" />
+        </geometry>
+        <material name="">
+          <color rgba="0.75294 0.75294 0.75294 1" />
+        </material>
+      </visual>
+      <collision>
+        <origin xyz="0 0 0" rpy="0 0 0" />
+        <geometry>
+          <mesh filename="file://$(find kortex_description)/arms/gen3/${dof}dof/meshes/shoulder_link.STL" />
+        </geometry>
+      </collision>
+    </link>
+    <joint
+      name="${prefix}joint_1"
+      type="continuous">
+      <origin
+        xyz="0 0 0.15643"
+        rpy="-3.1416 0.0 0.0" />
       <parent link="${prefix}base_link" />
       <child link="${prefix}shoulder_link" />
       <axis xyz="0 0 1" />
-      <limit effort="39" velocity="1.3963" />
+      <limit
+        effort="39"
+        velocity="1.3963" />
     </joint>
     <link name="${prefix}bicep_link">
       <inertial>
-        <origin xyz="3.5E-05 -0.208207 -0.01889" rpy="0 0 0" />
+        <origin
+          xyz="3.5E-05 -0.208207 -0.01889"
+          rpy="0 0 0" />
         <mass value="1.262" />
-        <inertia ixx="0.046752" ixy="-9E-06" ixz="0" iyy="0.00085" iyz="-9.8E-05" izz="0.047188" />
-      </inertial>
-      <visual>
-        <origin xyz="0 0 0" rpy="0 0 0" />
-        <geometry>
-          <mesh filename="package://kortex_description/arms/gen3/${dof}dof/meshes/bicep_link.STL" />
-        </geometry>
-        <material name="">
-          <color rgba="0.75294 0.75294 0.75294 1" />
-        </material>
-      </visual>
-      <collision>
-        <origin xyz="0 0 0" rpy="0 0 0" />
-        <geometry>
-          <mesh filename="package://kortex_description/arms/gen3/${dof}dof/meshes/bicep_link.STL" />
+        <inertia
+          ixx="0.046752"
+          ixy="-9E-06"
+          ixz="0"
+          iyy="0.00085"
+          iyz="-9.8E-05"
+          izz="0.047188" />
+      </inertial>
+      <visual>
+        <origin
+          xyz="0 0 0"
+          rpy="0 0 0" />
+        <geometry>
+          <mesh filename="file://$(find kortex_description)/arms/gen3/${dof}dof/meshes/bicep_link.STL" />
+        </geometry>
+        <material name="">
+          <color rgba="0.75294 0.75294 0.75294 1" />
+        </material>
+      </visual>
+      <collision>
+        <origin
+          xyz="0 0 0"
+          rpy="0 0 0" />
+        <geometry>
+          <mesh filename="file://$(find kortex_description)/arms/gen3/${dof}dof/meshes/bicep_link.STL" />
         </geometry>
       </collision>
@@ -93,14 +154,14 @@
         <origin xyz="0 0 0" rpy="0 0 0" />
         <geometry>
-          <mesh filename="package://kortex_description/arms/gen3/${dof}dof/meshes/forearm_link.STL" />
-        </geometry>
-        <material name="">
-          <color rgba="0.75294 0.75294 0.75294 1" />
-        </material>
-      </visual>
-      <collision>
-        <origin xyz="0 0 0" rpy="0 0 0" />
-        <geometry>
-          <mesh filename="package://kortex_description/arms/gen3/${dof}dof/meshes/forearm_link.STL" />
+          <mesh filename="file://$(find kortex_description)/arms/gen3/${dof}dof/meshes/forearm_link.STL" />
+        </geometry>
+        <material name="">
+          <color rgba="0.75294 0.75294 0.75294 1" />
+        </material>
+      </visual>
+      <collision>
+        <origin xyz="0 0 0" rpy="0 0 0" />
+        <geometry>
+          <mesh filename="file://$(find kortex_description)/arms/gen3/${dof}dof/meshes/forearm_link.STL" />
         </geometry>
       </collision>
@@ -122,14 +183,14 @@
         <origin xyz="0 0 0" rpy="0 0 0" />
         <geometry>
-          <mesh filename="package://kortex_description/arms/gen3/${dof}dof/meshes/spherical_wrist_1_link.STL" />
-        </geometry>
-        <material name="">
-          <color rgba="0.75294 0.75294 0.75294 1" />
-        </material>
-      </visual>
-      <collision>
-        <origin xyz="0 0 0" rpy="0 0 0" />
-        <geometry>
-          <mesh filename="package://kortex_description/arms/gen3/${dof}dof/meshes/spherical_wrist_1_link.STL" />
+          <mesh filename="file://$(find kortex_description)/arms/gen3/${dof}dof/meshes/spherical_wrist_1_link.STL" />
+        </geometry>
+        <material name="">
+          <color rgba="0.75294 0.75294 0.75294 1" />
+        </material>
+      </visual>
+      <collision>
+        <origin xyz="0 0 0" rpy="0 0 0" />
+        <geometry>
+          <mesh filename="file://$(find kortex_description)/arms/gen3/${dof}dof/meshes/spherical_wrist_1_link.STL" />
         </geometry>
       </collision>
@@ -151,14 +212,14 @@
         <origin xyz="0 0 0" rpy="0 0 0" />
         <geometry>
-          <mesh filename="package://kortex_description/arms/gen3/${dof}dof/meshes/spherical_wrist_2_link.STL" />
-        </geometry>
-        <material name="">
-          <color rgba="0.75294 0.75294 0.75294 1" />
-        </material>
-      </visual>
-      <collision>
-        <origin xyz="0 0 0" rpy="0 0 0" />
-        <geometry>
-          <mesh filename="package://kortex_description/arms/gen3/${dof}dof/meshes/spherical_wrist_2_link.STL" />
+          <mesh filename="file://$(find kortex_description)/arms/gen3/${dof}dof/meshes/spherical_wrist_2_link.STL" />
+        </geometry>
+        <material name="">
+          <color rgba="0.75294 0.75294 0.75294 1" />
+        </material>
+      </visual>
+      <collision>
+        <origin xyz="0 0 0" rpy="0 0 0" />
+        <geometry>
+          <mesh filename="file://$(find kortex_description)/arms/gen3/${dof}dof/meshes/spherical_wrist_2_link.STL" />
         </geometry>
       </collision>
@@ -181,14 +242,14 @@
         <origin xyz="0 0 0" rpy="0 0 0" />
         <geometry>
-          <mesh filename="package://kortex_description/arms/gen3/${dof}dof/meshes/bracelet_with_vision_link.STL" />
-        </geometry>
-        <material name="">
-          <color rgba="0.75294 0.75294 0.75294 1" />
-        </material>
-      </visual>
-      <collision>
-        <origin xyz="0 0 0" rpy="0 0 0" />
-        <geometry>
-          <mesh filename="package://kortex_description/arms/gen3/${dof}dof/meshes/bracelet_with_vision_link.STL" />
+          <mesh filename="file://$(find kortex_description)/arms/gen3/${dof}dof/meshes/bracelet_with_vision_link.STL" />
+        </geometry>
+        <material name="">
+          <color rgba="0.75294 0.75294 0.75294 1" />
+        </material>
+      </visual>
+      <collision>
+        <origin xyz="0 0 0" rpy="0 0 0" />
+        <geometry>
+          <mesh filename="file://$(find kortex_description)/arms/gen3/${dof}dof/meshes/bracelet_with_vision_link.STL" />
         </geometry>
       </collision>
@@ -205,14 +266,14 @@
         <origin xyz="0 0 0" rpy="0 0 0" />
         <geometry>
-          <mesh filename="package://kortex_description/arms/gen3/${dof}dof/meshes/bracelet_no_vision_link.STL" />
-        </geometry>
-        <material name="">
-          <color rgba="0.75294 0.75294 0.75294 1" />
-        </material>
-      </visual>
-      <collision>
-        <origin xyz="0 0 0" rpy="0 0 0" />
-        <geometry>
-          <mesh filename="package://kortex_description/arms/gen3/${dof}dof/meshes/bracelet_no_vision_link.STL" />
+          <mesh filename="file://$(find kortex_description)/arms/gen3/${dof}dof/meshes/bracelet_no_vision_link.STL" />
+        </geometry>
+        <material name="">
+          <color rgba="0.75294 0.75294 0.75294 1" />
+        </material>
+      </visual>
+      <collision>
+        <origin xyz="0 0 0" rpy="0 0 0" />
+        <geometry>
+          <mesh filename="file://$(find kortex_description)/arms/gen3/${dof}dof/meshes/bracelet_no_vision_link.STL" />
         </geometry>
       </collision>
@@ -238,4 +299,25 @@
         xyz="0 0 0" />
     </joint>
+    <!-- TODO(destogl) this probably collides with camera URDF -->
+    <xacro:if value="${vision}">
+      <link name="${prefix}camera_link" />
+      <joint name="${prefix}camera_module" type="fixed">
+        <origin xyz="0 0.05639 -0.00305" rpy="3.14159265358979 3.14159265358979 0" />
+        <parent link="${prefix}end_effector_link" />
+        <child  link="${prefix}camera_link" />
+      </joint>
+      <link name="${prefix}camera_depth_frame" />
+      <joint name="${prefix}depth_module" type="fixed">
+        <origin xyz="0.0275 0.066 -0.00305" rpy="3.14159265358979 3.14159265358979 0" />
+        <parent link="${prefix}end_effector_link" />
+        <child  link="${prefix}camera_depth_frame" />
+      </joint>
+      <link name="${prefix}camera_color_frame" />
+      <joint name="${prefix}color_module" type="fixed">
+        <origin xyz="0 0.05639 -0.00305" rpy="3.14159265358979 3.14159265358979 0" />
+        <parent link="${prefix}end_effector_link" />
+        <child  link="${prefix}camera_color_frame" />
+      </joint>
+    </xacro:if>
   </xacro:macro>
 </robot>

Commit message: update 6 dof

File: kortex_description/arms/gen3/6dof/urdf/gen3_macro.xacro (robot description, xacro)
@@ -3,4 +3,5 @@
   <!-- Propagate last link name information because it is the gripper's parent link -->
   <xacro:property name="last_arm_link" value="end_effector_link"/>
+  <xacro:property name="PI" value="3.1415926535897931"/>
   <xacro:macro name="load_arm" params="
     parent
@@ -22,4 +23,5 @@
     sim_ignition:=false
     sim_isaac:=false
+    use_external_cable:=false
     initial_positions:=${dict(joint_1=0.0,joint_2=0.0,joint_3=0.0,joint_4=0.0,joint_5=0.0,joint_6=0.0)}" >
     <!-- ros2 control include -->
@@ -91,17 +93,36 @@
       </collision>
     </link>
-    <joint
-      name="${prefix}joint_1"
-      type="continuous">
-      <origin
-        xyz="0 0 0.15643"
-        rpy="-3.1416 0.0 0.0" />
-      <parent link="${prefix}base_link" />
-      <child link="${prefix}shoulder_link" />
-      <axis xyz="0 0 1" />
-      <limit
-        effort="39"
-        velocity="1.3963" />
-    </joint>
+    <xacro:if value="${use_external_cable}">
+      <joint
+        name="${prefix}joint_1"
+        type="revolute">
+        <origin
+          xyz="0 0 0.15643"
+          rpy="-3.1416 0.0 0.0" />
+        <parent link="${prefix}base_link" />
+        <child link="${prefix}shoulder_link" />
+        <axis xyz="0 0 1" />
+        <limit
+          lower="${-2*PI}"
+          upper="${2*PI}"
+          effort="39"
+          velocity="1.3963" />
+      </joint>
+    </xacro:if>
+    <xacro:unless value="${use_external_cable}">
+      <joint
+        name="${prefix}joint_1"
+        type="continuous">
+        <origin
+          xyz="0 0 0.15643"
+          rpy="-3.1416 0.0 0.0" />
+        <parent link="${prefix}base_link" />
+        <child link="${prefix}shoulder_link" />
+        <axis xyz="0 0 1" />
+        <limit
+          effort="39"
+          velocity="1.3963" />
+      </joint>
+    </xacro:unless>
     <link name="${prefix}bicep_link">
       <inertial>
@@ -196,11 +217,22 @@
       </collision>
     </link>
-    <joint name="${prefix}joint_4" type="continuous">
-      <origin xyz="0 0.20843 -0.006375" rpy="1.5708 0.0 0.0" />
-      <parent link="${prefix}forearm_link" />
-      <child link="${prefix}spherical_wrist_1_link" />
-      <axis xyz="0 0 1" />
-      <limit effort="9" velocity="1.2218" />
-    </joint>
+    <xacro:if value="${use_external_cable}">
+      <joint name="${prefix}joint_4" type="revolute">
+        <origin xyz="0 0.20843 -0.006375" rpy="1.5708 0.0 0.0" />
+        <parent link="${prefix}forearm_link" />
+        <child link="${prefix}spherical_wrist_1_link" />
+        <axis xyz="0 0 1" />
+        <limit lower="${-2*PI}" upper="${2*PI}" effort="9" velocity="1.2218" />
+      </joint>
+    </xacro:if>
+    <xacro:unless value="${use_external_cable}">
+      <joint name="${prefix}joint_4" type="continuous">
+        <origin xyz="0 0.20843 -0.006375" rpy="1.5708 0.0 0.0" />
+        <parent link="${prefix}forearm_link" />
+        <child link="${prefix}spherical_wrist_1_link" />
+        <axis xyz="0 0 1" />
+        <limit effort="9" velocity="1.2218" />
+      </joint>
+    </xacro:unless>
     <link name="${prefix}spherical_wrist_2_link">
       <inertial>
@@ -280,11 +312,22 @@
     </link>
     </xacro:unless>
-    <joint name="${prefix}joint_6" type="continuous">
-      <origin xyz="0 0.10593 -0.00017505" rpy="1.5708 0.0 0.0" />
-      <parent link="${prefix}spherical_wrist_2_link" />
-      <child link="${prefix}bracelet_link" />
-      <axis xyz="0 0 1" />
-      <limit effort="9" velocity="1.2218" />
-    </joint>
+    <xacro:if value="${use_external_cable">
+      <joint name="${prefix}joint_6" type="revolute">
+        <origin xyz="0 0.10593 -0.00017505" rpy="1.5708 0.0 0.0" />
+        <parent link="${prefix}spherical_wrist_2_link" />
+        <child link="${prefix}bracelet_link" />
+        <axis xyz="0 0 1" />
+        <limit lower="${-2*PI}" upper="${2*PI}" effort="9" velocity="1.2218" />
+      </joint>
+    </xacro:if>
+    <xacro:unless value="${use_external_cable">
+      <joint name="${prefix}joint_6" type="continuous">
+        <origin xyz="0 0.10593 -0.00017505" rpy="1.5708 0.0 0.0" />
+        <parent link="${prefix}spherical_wrist_2_link" />
+        <child link="${prefix}bracelet_link" />
+        <axis xyz="0 0 1" />
+        <limit effort="9" velocity="1.2218" />
+      </joint>
+    </xacro:unless>
     <link name="${prefix}end_effector_link" />
     <joint

Commit message: Add use_external_cable parameter to URDF (#155)

File: kortex_description/arms/gen3/6dof/urdf/gen3_macro.xacro (robot description, xacro)
@@ -3,4 +3,5 @@
   <!-- Propagate last link name information because it is the gripper's parent link -->
   <xacro:property name="last_arm_link" value="end_effector_link"/>
+  <xacro:property name="PI" value="3.1415926535897931"/>
   <xacro:macro name="load_arm" params="
     parent
@@ -22,4 +23,5 @@
     sim_ignition:=false
     sim_isaac:=false
+    use_external_cable:=false
     initial_positions:=${dict(joint_1=0.0,joint_2=0.0,joint_3=0.0,joint_4=0.0,joint_5=0.0,joint_6=0.0)}" >
     <!-- ros2 control include -->
@@ -91,17 +93,36 @@
       </collision>
     </link>
-    <joint
-      name="${prefix}joint_1"
-      type="continuous">
-      <origin
-        xyz="0 0 0.15643"
-        rpy="-3.1416 0.0 0.0" />
-      <parent link="${prefix}base_link" />
-      <child link="${prefix}shoulder_link" />
-      <axis xyz="0 0 1" />
-      <limit
-        effort="39"
-        velocity="1.3963" />
-    </joint>
+    <xacro:if value="${use_external_cable}">
+      <joint
+        name="${prefix}joint_1"
+        type="revolute">
+        <origin
+          xyz="0 0 0.15643"
+          rpy="-3.1416 0.0 0.0" />
+        <parent link="${prefix}base_link" />
+        <child link="${prefix}shoulder_link" />
+        <axis xyz="0 0 1" />
+        <limit
+          lower="${-2*PI}"
+          upper="${2*PI}"
+          effort="39"
+          velocity="1.3963" />
+      </joint>
+    </xacro:if>
+    <xacro:unless value="${use_external_cable}">
+      <joint
+        name="${prefix}joint_1"
+        type="continuous">
+        <origin
+          xyz="0 0 0.15643"
+          rpy="-3.1416 0.0 0.0" />
+        <parent link="${prefix}base_link" />
+        <child link="${prefix}shoulder_link" />
+        <axis xyz="0 0 1" />
+        <limit
+          effort="39"
+          velocity="1.3963" />
+      </joint>
+    </xacro:unless>
     <link name="${prefix}bicep_link">
       <inertial>
@@ -196,11 +217,22 @@
       </collision>
     </link>
-    <joint name="${prefix}joint_4" type="continuous">
-      <origin xyz="0 0.20843 -0.006375" rpy="1.5708 0.0 0.0" />
-      <parent link="${prefix}forearm_link" />
-      <child link="${prefix}spherical_wrist_1_link" />
-      <axis xyz="0 0 1" />
-      <limit effort="9" velocity="1.2218" />
-    </joint>
+    <xacro:if value="${use_external_cable}">
+      <joint name="${prefix}joint_4" type="revolute">
+        <origin xyz="0 0.20843 -0.006375" rpy="1.5708 0.0 0.0" />
+        <parent link="${prefix}forearm_link" />
+        <child link="${prefix}spherical_wrist_1_link" />
+        <axis xyz="0 0 1" />
+        <limit lower="${-2*PI}" upper="${2*PI}" effort="9" velocity="1.2218" />
+      </joint>
+    </xacro:if>
+    <xacro:unless value="${use_external_cable}">
+      <joint name="${prefix}joint_4" type="continuous">
+        <origin xyz="0 0.20843 -0.006375" rpy="1.5708 0.0 0.0" />
+        <parent link="${prefix}forearm_link" />
+        <child link="${prefix}spherical_wrist_1_link" />
+        <axis xyz="0 0 1" />
+        <limit effort="9" velocity="1.2218" />
+      </joint>
+    </xacro:unless>
     <link name="${prefix}spherical_wrist_2_link">
       <inertial>
@@ -280,11 +312,22 @@
     </link>
     </xacro:unless>
-    <joint name="${prefix}joint_6" type="continuous">
-      <origin xyz="0 0.10593 -0.00017505" rpy="1.5708 0.0 0.0" />
-      <parent link="${prefix}spherical_wrist_2_link" />
-      <child link="${prefix}bracelet_link" />
-      <axis xyz="0 0 1" />
-      <limit effort="9" velocity="1.2218" />
-    </joint>
+    <xacro:if value="${use_external_cable}">
+      <joint name="${prefix}joint_6" type="revolute">
+        <origin xyz="0 0.10593 -0.00017505" rpy="1.5708 0.0 0.0" />
+        <parent link="${prefix}spherical_wrist_2_link" />
+        <child link="${prefix}bracelet_link" />
+        <axis xyz="0 0 1" />
+        <limit lower="${-2*PI}" upper="${2*PI}" effort="9" velocity="1.2218" />
+      </joint>
+    </xacro:if>
+    <xacro:unless value="${use_external_cable}">
+      <joint name="${prefix}joint_6" type="continuous">
+        <origin xyz="0 0.10593 -0.00017505" rpy="1.5708 0.0 0.0" />
+        <parent link="${prefix}spherical_wrist_2_link" />
+        <child link="${prefix}bracelet_link" />
+        <axis xyz="0 0 1" />
+        <limit effort="9" velocity="1.2218" />
+      </joint>
+    </xacro:unless>
     <link name="${prefix}end_effector_link" />
     <joint
