Commit message: fix: automated fix attempt for issue #213

File: kortex_description/arms/gen3/6dof/urdf/gen3_macro.xacro (robot description, xacro)
@@ -24,4 +24,5 @@
     fake_sensor_commands:=false
     sim_gazebo:=false
+    sim_ignition:=false
     sim_isaac:=false
     isaac_joint_commands:=/isaac_joint_commands
@@ -37,4 +38,5 @@
       fake_sensor_commands="${fake_sensor_commands}"
       sim_gazebo="${sim_gazebo}"
+      sim_ignition="${sim_ignition}"
       sim_isaac="${sim_isaac}"
       isaac_joint_commands="${isaac_joint_commands}"

File: kortex_description/arms/gen3/6dof/urdf/kortex.ros2_control.xacro (robot description, xacro)
@@ -7,4 +7,5 @@
     fake_sensor_commands:=false
     sim_gazebo:=false
+    sim_ignition:=false
     sim_isaac:=false
     isaac_joint_commands:=/isaac_joint_commands
@@ -30,4 +31,7 @@
           <plugin>gz_ros2_control/GazeboSimSystem</plugin>
         </xacro:if>
+        <xacro:if value="${sim_ignition}">
+          <plugin>ign_ros2_control/IgnitionSystem</plugin>
+        </xacro:if>
         <xacro:if value="${sim_isaac}">
           <plugin>topic_based_ros2_control/TopicBasedSystem</plugin>
@@ -40,5 +44,5 @@
           <param name="state_following_offset">0.0</param>
         </xacro:if>
-        <xacro:unless value="${use_fake_hardware or sim_gazebo or sim_isaac}">
+        <xacro:unless value="${use_fake_hardware or sim_gazebo or sim_ignition or sim_isaac}">
           <plugin>kortex_driver/KortexMultiInterfaceHardware</plugin>
           <param name="robot_ip">${robot_ip}</param>

File: kortex_description/arms/gen3/7dof/urdf/gen3_macro.xacro (robot description, xacro)
@@ -24,4 +24,5 @@
     fake_sensor_commands:=false
     sim_gazebo:=false
+    sim_ignition:=false
     sim_isaac:=false
     isaac_joint_commands:=/isaac_joint_commands
@@ -37,4 +38,5 @@
       fake_sensor_commands="${fake_sensor_commands}"
       sim_gazebo="${sim_gazebo}"
+      sim_ignition="${sim_ignition}"
       sim_isaac="${sim_isaac}"
       isaac_joint_commands="${isaac_joint_commands}"

File: kortex_description/arms/gen3/7dof/urdf/kortex.ros2_control.xacro (robot description, xacro)
@@ -7,4 +7,5 @@
     fake_sensor_commands:=false
     sim_gazebo:=false
+    sim_ignition:=false
     sim_isaac:=false
     isaac_joint_commands:=/isaac_joint_commands
@@ -30,4 +31,7 @@
           <plugin>gz_ros2_control/GazeboSimSystem</plugin>
         </xacro:if>
+        <xacro:if value="${sim_ignition}">
+          <plugin>ign_ros2_control/IgnitionSystem</plugin>
+        </xacro:if>
         <xacro:if value="${sim_isaac}">
           <plugin>topic_based_ros2_control/TopicBasedSystem</plugin>
@@ -40,5 +44,5 @@
           <param name="state_following_offset">0.0</param>
         </xacro:if>
-        <xacro:unless value="${use_fake_hardware or sim_gazebo or sim_isaac}">
+        <xacro:unless value="${use_fake_hardware or sim_gazebo or sim_ignition or sim_isaac}">
           <plugin>kortex_driver/KortexMultiInterfaceHardware</plugin>
           <param name="robot_ip">${robot_ip}</param>

File: kortex_description/arms/gen3_lite/6dof/urdf/gen3_lite_macro.xacro (robot description, xacro)
@@ -23,4 +23,5 @@
     fake_sensor_commands:=false
     sim_gazebo:=false
+    sim_ignition:=false
     sim_isaac:=false
     isaac_joint_commands:=/isaac_joint_commands
@@ -36,4 +37,9 @@
       </xacro:unless>
     </xacro:if>
+    <xacro:if value="${sim_ignition}">
+      <xacro:unless value="${moveit_active}">
+        <xacro:property name="ros2_control_name" value="IgnitionSystem"/>
+      </xacro:unless>
+    </xacro:if>
      <xacro:if value="${use_fake_hardware}">
       <xacro:unless value="${moveit_active}">
@@ -41,5 +47,5 @@
       </xacro:unless>
     </xacro:if>
-    <xacro:unless value="${use_fake_hardware or sim_gazebo}">
+    <xacro:unless value="${use_fake_hardware or sim_gazebo or sim_ignition}">
       <xacro:unless value="${moveit_active}">
         <xacro:property name="ros2_control_name" value="${prefix}KortexMultiInterfaceHardware"/>
@@ -54,4 +60,5 @@
       fake_sensor_commands="${fake_sensor_commands}"
       sim_gazebo="${sim_gazebo}"
+      sim_ignition="${sim_ignition}"
       sim_isaac="${sim_isaac}"
       isaac_joint_commands="${isaac_joint_commands}"

File: kortex_description/arms/gen3_lite/6dof/urdf/kortex.ros2_control.xacro (robot description, xacro)
@@ -7,4 +7,5 @@
     fake_sensor_commands:=false
     sim_gazebo:=false
+    sim_ignition:=false
     sim_isaac:=false
     isaac_joint_commands:=/isaac_joint_commands
@@ -31,4 +32,9 @@
           </xacro:unless>
         </xacro:if>
+        <xacro:if value="${sim_ignition}">
+          <xacro:unless value="${moveit_active}">
+            <plugin>ign_ros2_control/IgnitionSystem</plugin>
+          </xacro:unless>
+        </xacro:if>
         <xacro:if value="${sim_isaac}">
           <xacro:unless value="${moveit_active}">
@@ -45,5 +51,5 @@
           </xacro:unless>
         </xacro:if>
-        <xacro:unless value="${use_fake_hardware or sim_gazebo or sim_isaac}">
+        <xacro:unless value="${use_fake_hardware or sim_gazebo or sim_ignition or sim_isaac}">
           <xacro:unless value="${moveit_active}">
             <plugin>kortex_driver/KortexMultiInterfaceHardware</plugin>

File: kortex_description/grippers/gen3_lite_2f/urdf/gen3_lite_2f.ros2_control.xacro (robot description, xacro)
@@ -6,4 +6,5 @@
         fake_sensor_commands:=false
         sim_gazebo:=false
+        sim_ignition:=false
         sim_isaac:=false
         isaac_joint_commands:=/isaac_joint_commands
@@ -32,4 +33,7 @@
                     <plugin>gz_ros2_control/GzSimSystem</plugin>
                 </xacro:if>
+                <xacro:if value="${sim_ignition}">
+                    <plugin>ign_ros2_control/IgnitionSystem</plugin>
+                </xacro:if>
                 <xacro:if value="${use_fake_hardware}">
                     <plugin>mock_components/GenericSystem</plugin>
@@ -37,5 +41,5 @@
                     <param name="state_following_offset">0.0</param>
                 </xacro:if>
-                <xacro:unless value="${sim_isaac or sim_gazebo or use_fake_hardware}">
+                <xacro:unless value="${sim_isaac or sim_gazebo or sim_ignition or use_fake_hardware}">
                     <plugin>kortex_driver/KortexMultiInterfaceHardware</plugin>
                     <param name="robot_ip">${robot_ip}</param>

File: kortex_description/grippers/gen3_lite_2f/urdf/gen3_lite_2f_macro.xacro (robot description, xacro)
@@ -8,4 +8,5 @@
     fake_sensor_commands:=false
     sim_gazebo:=false
+    sim_ignition:=false
     sim_isaac:=false
     isaac_joint_commands:=/isaac_joint_commands
@@ -13,5 +14,5 @@
     use_internal_bus_gripper_comm:=true
     moveit_active:=false">
-  <xacro:if value="${use_fake_hardware or sim_isaac or sim_gazebo}">
+  <xacro:if value="${use_fake_hardware or sim_isaac or sim_gazebo or sim_ignition}">
     <xacro:unless value="${moveit_active}">
     <!-- ros2 control include -->
@@ -20,8 +21,11 @@
         <xacro:property name="ros2_control_name" value="GazeboSimSystem"/>
       </xacro:if>
+      <xacro:if value="${sim_ignition}">
+        <xacro:property name="ros2_control_name" value="IgnitionSystem"/>
+      </xacro:if>
       <xacro:if value="${use_fake_hardware}">
         <xacro:property name="ros2_control_name" value="GenericSystem"/>
       </xacro:if>
-      <xacro:unless value="${use_fake_hardware or sim_gazebo}">
+      <xacro:unless value="${use_fake_hardware or sim_gazebo or sim_ignition}">
         <xacro:property name="ros2_control_name" value="${prefix}KortexMultiInterfaceHardware"/>
       </xacro:unless>
@@ -31,4 +35,5 @@
         fake_sensor_commands="${fake_sensor_commands}"
         sim_gazebo="${sim_gazebo}"
+        sim_ignition="${sim_ignition}"
         sim_isaac="${sim_isaac}"
         isaac_joint_commands="${isaac_joint_commands}"

File: kortex_description/robots/gen3.xacro (robot description, xacro)
@@ -17,4 +17,5 @@
     <xacro:arg name="gripper_max_force" default="100.0" />
     <xacro:arg name="sim_gazebo" default="false" />
+    <xacro:arg name="sim_ignition" default="false" />
     <xacro:arg name="sim_isaac" default="false" />
     <xacro:arg name="prefix" default="" />
@@ -50,4 +51,5 @@
         fake_sensor_commands="$(arg fake_sensor_commands)"
         sim_gazebo="$(arg sim_gazebo)"
+        sim_ignition="$(arg sim_ignition)"
         sim_isaac="$(arg sim_isaac)"
         use_external_cable="$(arg use_external_cable)"

File: kortex_description/robots/gen3_lite_gen3_lite_2f.xacro (robot description, xacro)
@@ -17,4 +17,5 @@
     <xacro:arg name="gripper_max_force" default="100.0" />
     <xacro:arg name="sim_gazebo" default="false" />
+    <xacro:arg name="sim_ignition" default="false" />
     <xacro:arg name="sim_isaac" default="false" />
     <xacro:arg name="prefix" default="" />
@@ -47,4 +48,5 @@
         fake_sensor_commands="$(arg fake_sensor_commands)"
         sim_gazebo="$(arg sim_gazebo)"
+        sim_ignition="$(arg sim_ignition)"
         sim_isaac="$(arg sim_isaac)"
         use_external_cable="$(arg use_external_cable)"

File: kortex_description/robots/kinova.urdf.xacro (robot description, xacro)
@@ -23,4 +23,5 @@
   <xacro:arg name="fake_sensor_commands" default="false" />
   <xacro:arg name="sim_gazebo" default="false" />
+  <xacro:arg name="sim_ignition" default="false" />
   <xacro:arg name="sim_isaac" default="false" />
   <xacro:arg name="gazebo_renderer" default="ogre"/>
@@ -59,4 +60,5 @@
     fake_sensor_commands="$(arg fake_sensor_commands)"
     sim_gazebo="$(arg sim_gazebo)"
+    sim_ignition="$(arg sim_ignition)"
     sim_isaac="$(arg sim_isaac)"
     initial_positions="${xacro.load_yaml(initial_positions_file)}"
@@ -77,4 +79,20 @@
       </plugin>
     </gazebo>
+  </xacro:if>
+  <xacro:if value="$(arg sim_ignition)">
+    <!-- Ignition Gazebo plugins -->
+    <gazebo reference="world">
+    </gazebo>
+    <gazebo>
+      <plugin filename="ign_ros2_control-system" name="ign_ros2_control::IgnitionROS2ControlPlugin">
+        <parameters>$(arg simulation_controllers)</parameters>
+        <controller_manager_node_name>$(arg prefix)controller_manager</controller_manager_node_name>
+      </plugin>
+      <plugin filename="ignition-gazebo-sensors-system" name="ignition::gazebo::systems::Sensors">
+        <render_engine>$(arg gazebo_renderer)</render_engine>
+      </plugin>
+    </gazebo>
+  </xacro:if>
+  <xacro:if value="$(arg sim_gazebo)">
     <gazebo reference="camera_color_frame">
       <sensor name="camera_sensor" type="rgbd_camera">

File: kortex_description/robots/kortex_robot.xacro (robot description, xacro)
@@ -21,4 +21,5 @@
     fake_sensor_commands:=false
     sim_gazebo:=false
+    sim_ignition:=false
     sim_isaac:=false
     isaac_joint_commands:=/isaac_joint_commands
@@ -49,4 +50,5 @@
       fake_sensor_commands="${fake_sensor_commands}"
       sim_gazebo="${sim_gazebo}"
+      sim_ignition="${sim_ignition}"
       sim_isaac="${sim_isaac}"
       isaac_joint_commands="${isaac_joint_commands}"
@@ -81,4 +83,5 @@
         fake_sensor_commands="${fake_sensor_commands}"
         sim_gazebo="${sim_gazebo}"
+        sim_ignition="${sim_ignition}"
         sim_isaac="${sim_isaac}"
         isaac_joint_commands="${isaac_joint_commands}"
