Commit message: Comm frequency up to 1kHz for each arm + surrouding walls

File: kortex_description/arms/gen3/6dof/urdf/gen3_macro.xacro (robot description, xacro)
@@ -29,5 +29,8 @@
     use_external_cable:=false
     initial_positions:=${dict(joint_1=0.0,joint_2=0.0,joint_3=0.0,joint_4=0.0,joint_5=0.0,joint_6=0.0)}
-    moveit_active:=false">
+    moveit_active:=false
+    hw_is_async:=false
+    hw_async_cores:=[]
+    hw_async_priority:=80">
     <!-- ros2 control include -->
     <xacro:include filename="$(find kortex_description)/arms/gen3/${dof}dof/urdf/kortex.ros2_control.xacro" />
@@ -53,5 +56,8 @@
       gripper_max_force="${gripper_max_force}"
       gripper_joint_name="${gripper_joint_name}"
-      gripper="${gripper}"/>
+      gripper="${gripper}"
+      hw_is_async="${hw_is_async}"
+      hw_async_cores="${hw_async_cores}"
+      hw_async_priority="${hw_async_priority}"/>
     <joint name="${prefix}base_joint" type="fixed">
       <xacro:insert_block name="origin" />

File: kortex_description/arms/gen3/6dof/urdf/kortex.ros2_control.xacro (robot description, xacro)
@@ -24,6 +24,9 @@
     gripper_max_velocity:=100.0
     gripper_max_force:=100.0
-    moveit_active:=false">
-    <ros2_control name="${name}" type="system">
+    moveit_active:=false
+    hw_is_async:=false
+    hw_async_cores:=[]
+    hw_async_priority:=80">
+    <ros2_control name="${name}" type="system" is_async="${hw_is_async}">
       <hardware>
         <xacro:if value="${sim_gazebo}">
@@ -57,4 +60,12 @@
         </xacro:unless>
       </hardware>
+      <xacro:if value="${hw_is_async}">
+        <properties>
+          <async affinity="${hw_async_cores}"
+                 scheduling_policy="synchronized"
+                 thread_priority="${hw_async_priority}"
+                 print_warnings="false"/>
+        </properties>
+      </xacro:if>
       <joint name="${prefix}joint_1">
         <command_interface name="position">

File: kortex_description/arms/gen3/7dof/urdf/gen3_macro.xacro (robot description, xacro)
@@ -29,5 +29,8 @@
     use_external_cable:=false
     initial_positions:=${dict(joint_1=0.0,joint_2=0.0,joint_3=0.0,joint_4=0.0,joint_5=0.0,joint_6=0.0,joint_7=0.0)}
-    moveit_active:=false">
+    moveit_active:=false
+    hw_is_async:=false
+    hw_async_cores:=[]
+    hw_async_priority:=80">
     <!-- ros2 control include -->
     <xacro:include filename="$(find kortex_description)/arms/gen3/${dof}dof/urdf/kortex.ros2_control.xacro" />
@@ -53,5 +56,8 @@
       gripper_max_force="${gripper_max_force}"
       gripper_joint_name="${gripper_joint_name}"
-      gripper="${gripper}"/>
+      gripper="${gripper}"
+      hw_is_async="${hw_is_async}"
+      hw_async_cores="${hw_async_cores}"
+      hw_async_priority="${hw_async_priority}"/>
     <joint name="${prefix}base_joint" type="fixed">
       <xacro:insert_block name="origin" />

File: kortex_description/arms/gen3/7dof/urdf/kortex.ros2_control.xacro (robot description, xacro)
@@ -24,6 +24,9 @@
     gripper_max_velocity:=100.0
     gripper_max_force:=100.0
-    moveit_active:=false">
-    <ros2_control name="${name}" type="system">
+    moveit_active:=false
+    hw_is_async:=false
+    hw_async_cores:=[]
+    hw_async_priority:=80">
+    <ros2_control name="${name}" type="system" is_async="${hw_is_async}">
       <hardware>
         <xacro:if value="${sim_gazebo}">
@@ -57,4 +60,15 @@
         </xacro:unless>
       </hardware>
+      <!-- Run this component's read()+write() on its own thread, so a blocking
+           BaseCyclic::Refresh() does not serialise against other arms in the
+           same controller_manager. See CLAUDE.md "Two arms". -->
+      <xacro:if value="${hw_is_async}">
+        <properties>
+          <async affinity="${hw_async_cores}"
+                 scheduling_policy="synchronized"
+                 thread_priority="${hw_async_priority}"
+                 print_warnings="false"/>
+        </properties>
+      </xacro:if>
       <joint name="${prefix}joint_1">
         <command_interface name="position">

File: kortex_description/arms/gen3_lite/6dof/urdf/gen3_lite_macro.xacro (robot description, xacro)
@@ -29,5 +29,8 @@
     use_external_cable:=false
     initial_positions:=${dict(joint_1=0.0,joint_2=0.0,joint_3=0.0,joint_4=0.0,joint_5=0.0,joint_6=0.0)}
-    moveit_active:=false" >
+    moveit_active:=false
+    hw_is_async:=false
+    hw_async_cores:=[]
+    hw_async_priority:=80" >
     <!-- ros2 control include -->
     <xacro:include filename="$(find kortex_description)/arms/gen3_lite/${dof}dof/urdf/kortex.ros2_control.xacro" />
@@ -71,5 +74,8 @@
       gripper_max_force="${gripper_max_force}"
       gripper_joint_name="${gripper_joint_name}"
-      moveit_active="${moveit_active}"/>
+      moveit_active="${moveit_active}"
+      hw_is_async="${hw_is_async}"
+      hw_async_cores="${hw_async_cores}"
+      hw_async_priority="${hw_async_priority}"/>
     <joint name="${prefix}base_joint" type="fixed">
       <xacro:insert_block name="origin" />

File: kortex_description/arms/gen3_lite/6dof/urdf/kortex.ros2_control.xacro (robot description, xacro)
@@ -23,6 +23,9 @@
     gripper_max_velocity:=100.0
     gripper_max_force:=100.0
-    moveit_active:=false">
-    <ros2_control name="${name}" type="system">
+    moveit_active:=false
+    hw_is_async:=false
+    hw_async_cores:=[]
+    hw_async_priority:=80">
+    <ros2_control name="${name}" type="system" is_async="${hw_is_async}">
       <hardware>
         <xacro:if value="${sim_gazebo}">
@@ -79,4 +82,12 @@
         </xacro:if>
       </hardware>
+      <xacro:if value="${hw_is_async}">
+        <properties>
+          <async affinity="${hw_async_cores}"
+                 scheduling_policy="synchronized"
+                 thread_priority="${hw_async_priority}"
+                 print_warnings="false"/>
+        </properties>
+      </xacro:if>
       <joint name="${prefix}joint_1">
         <command_interface name="position">

File: kortex_description/multiple_robots/dual_arm_structure.xacro (robot description, xacro)
@@ -3,7 +3,12 @@
   <!-- Macro: load_dual_arm_structure
        Creates a parametric box body (visual + collision) fixed to 'parent'.
-       Arm bases attach to ${name}_link at +/-(length/2) on the X axis.
+       NOTE: kortex_dual_robots.xacro always passes length/width/height
+       explicitly, so the defaults below are NEVER used. To resize the plate,
+       edit the plate_length / plate_width / plate_thickness args in
+       kortex_dual_robots.xacro — changing the defaults here does nothing.
+       Arm bases attach to ${name}_link at +/-(base_separation/2) on the Y
+       axis, on the top face (z = +height/2).
        Params: parent, *origin, name (default: dual_arm_structure),
-               length/width/height in metres (defaults: 0.30 / 0.20 / 0.40). -->
+               length (X) / width (Y) / height (Z) in metres. -->
   <xacro:macro name="load_dual_arm_structure" params="
       parent
@@ -12,5 +17,5 @@
       length:=0.30
       width:=0.20
-      height:=0.40">
+      height:=0.05">
     <link name="${name}_link">
       <visual>

File: kortex_description/multiple_robots/kortex_dual_robots.xacro (robot description, xacro)
@@ -10,5 +10,5 @@
     <xacro:arg name="left_vision" default="false"/>
     <xacro:arg name="left_prefix" default="left_"/>
-    <xacro:arg name="left_robot_ip" default="192.168.1.10"/>
+    <xacro:arg name="left_robot_ip" default="192.168.2.10"/>
     <xacro:arg name="left_username" default="admin"/>
     <xacro:arg name="left_password" default="admin"/>
@@ -17,6 +17,7 @@
     <xacro:arg name="left_session_inactivity_timeout_ms" default="60000"/>
     <xacro:arg name="left_connection_inactivity_timeout_ms" default="2000"/>
-    <xacro:arg name="left_xyz" default="0.0565 0 0.1395"/>
-    <xacro:arg name="left_rpy" default="1.5708 0  1.5708"/>
+    <!-- Base pose is derived from base_separation below; rpy stays overridable
+         so the arms can be yawed inward later without editing the plate maths. -->
+    <xacro:arg name="left_rpy" default="0 0 0"/>
     <!-- ============================================================== -->
     <!-- RIGHT ARM arguments                                             -->
@@ -28,5 +29,5 @@
     <xacro:arg name="right_vision" default="false"/>
     <xacro:arg name="right_prefix" default="right_"/>
-    <xacro:arg name="right_robot_ip" default="192.168.1.11"/>
+    <xacro:arg name="right_robot_ip" default="192.168.1.10"/>
     <xacro:arg name="right_username" default="admin"/>
     <xacro:arg name="right_password" default="admin"/>
@@ -35,6 +36,5 @@
     <xacro:arg name="right_session_inactivity_timeout_ms" default="60000"/>
     <xacro:arg name="right_connection_inactivity_timeout_ms" default="2000"/>
-    <xacro:arg name="right_xyz" default="-0.0565 0 0.1395"/>
-    <xacro:arg name="right_rpy" default="-1.5708 0 1.5708"/>
+    <xacro:arg name="right_rpy" default="0 0 0"/>
     <!-- ============================================================== -->
     <!-- Shared arguments                                                -->
@@ -49,12 +49,54 @@
     <xacro:arg name="gripper_max_force" default="100.0"/>
     <!-- ============================================================== -->
-    <!-- Structure arguments                                            -->
-    <!-- ============================================================== -->
-    <xacro:arg name="struct_name"   default="dual_arm_structure"/>
-    <xacro:arg name="struct_length" default="0.113"/>
-    <xacro:arg name="struct_width"  default="0.225"/>
-    <xacro:arg name="struct_height" default="0.585"/>
-    <xacro:arg name="struct_xyz"    default="0 0 0.2925"/>
-    <xacro:arg name="struct_rpy"    default="0 0 0"/>
+    <!-- Mounting geometry                                              -->
+    <!-- Both arms stand vertically (base +Z = world +Z) on a horizontal -->
+    <!-- plate, spaced base_separation apart along Y: left at +Y, right  -->
+    <!-- at -Y. The plate rests on the world plane (bottom face z = 0)   -->
+    <!-- and the arms bolt to its top face.                              -->
+    <!-- ============================================================== -->
+    <!-- Async hardware: each arm's read()+write() runs on its own thread, so the
+         two blocking BaseCyclic::Refresh() round trips overlap instead of adding
+         up. Cores 6 and 7 are isolated (isolcpus=2,3,6,7). -->
+    <xacro:arg name="hw_is_async"       default="true"/>
+    <xacro:arg name="left_async_cores"  default="[6]"/>
+    <xacro:arg name="right_async_cores" default="[7]"/>
+    <xacro:arg name="hw_async_priority" default="80"/>
+    <!-- Workspace walls: a fixed enclosure MoveIt collision-checks against, so
+         planned paths cannot leave the cell. Faces sit wall_offset from each
+         arm's BASE CENTRE: +/-wall_offset in X (both arms are at x=0) and
+         +/-(base_separation/2 + wall_offset) in Y.
+         Reference numbers for this arm (gen3 7dof + 2f-85, measured from the
+         URDF): max horizontal reach 1.007 m, max vertical reach 1.291 m above
+         the base. wall_height therefore defaults to 1.35 m so the arm cannot
+         arc over the top; drop it if you only want a lateral fence.
+         All three SRDF named poses fit inside the default 0.7 m offset:
+         "Home" reaches 0.559 m horizontally (+X, 141 mm margin), "Retract"
+         0.150 m, "Vertical" 0.072 m. Below ~0.62 m Home starts inside the +X
+         wall and MoveIt refuses to plan from it.
+         NOTE robot.launch.py always forwards wall_offset into the xacro
+         mappings, so the launch argument's default WINS over the one below.
+         Keep the two in sync. -->
+    <xacro:arg name="enable_walls"   default="true"/>
+    <xacro:arg name="wall_offset"    default="0.7"/>   <!-- m from each arm base centre -->
+    <xacro:arg name="wall_height"    default="1.35"/>  <!-- m above the plate top face -->
+    <xacro:arg name="wall_thickness" default="0.02"/>  <!-- m -->
+    <xacro:arg name="struct_name"     default="dual_arm_structure"/>
+    <xacro:arg name="base_separation" default="0.585"/>   <!-- centre-to-centre, m -->
+    <xacro:arg name="plate_length"    default="2.0"/>  <!-- X extent, m -->
+    <xacro:arg name="plate_thickness" default="0.05"/>  <!-- Z extent, m -->
+    <xacro:arg name="plate_margin"    default="1.0"/>  <!-- Y overhang past each base, m -->
+    <xacro:property name="base_sep"   value="$(arg base_separation)"/>
+    <xacro:property name="plate_len"  value="$(arg plate_length)"/>
+    <xacro:property name="plate_th"   value="$(arg plate_thickness)"/>
+    <xacro:property name="plate_marg" value="$(arg plate_margin)"/>
+    <xacro:property name="plate_wid"  value="${base_sep + 2 * plate_marg}"/>
+    <xacro:property name="wall_off"   value="$(arg wall_offset)"/>
+    <xacro:property name="wall_h"     value="$(arg wall_height)"/>
+    <xacro:property name="wall_t"     value="$(arg wall_thickness)"/>
+    <!-- inner faces of the enclosure, in the plate link frame -->
+    <xacro:property name="wall_hx"    value="${wall_off}"/>
+    <xacro:property name="wall_hy"    value="${base_sep / 2 + wall_off}"/>
+    <!-- plate link frame sits at the plate mid-height, so its top face is +plate_th/2 -->
+    <xacro:property name="wall_cz"    value="${plate_th / 2 + wall_h / 2}"/>
     <xacro:include filename="$(find kortex_description)/robots/kortex_robot.xacro"/>
     <xacro:include filename="$(find kortex_description)/multiple_robots/dual_arm_structure.xacro"/>
@@ -68,9 +110,48 @@
         parent="world"
         name="$(arg struct_name)"
-        length="$(arg struct_length)"
-        width="$(arg struct_width)"
-        height="$(arg struct_height)">
-        <origin xyz="$(arg struct_xyz)" rpy="$(arg struct_rpy)"/>
+        length="${plate_len}"
+        width="${plate_wid}"
+        height="${plate_th}">
+        <origin xyz="0 0 ${plate_th / 2}" rpy="0 0 0"/>
     </xacro:load_dual_arm_structure>
+    <!-- ============================================================== -->
+    <!-- Workspace walls                                                -->
+    <!-- All four walls are collision/visual geometry on ONE link. That -->
+    <!-- is deliberate: MoveIt never self-collision-checks within a     -->
+    <!-- single link, so the corners can overlap without producing a    -->
+    <!-- permanent wall-vs-wall collision, and the only ACM entry that  -->
+    <!-- matters (wall vs plate) is auto-disabled because the two are   -->
+    <!-- adjacent across a fixed joint.                                 -->
+    <!-- ============================================================== -->
+    <xacro:if value="$(arg enable_walls)">
+      <link name="workspace_walls_link">
+        <xacro:macro name="wall_box" params="sx sy sz x y z">
+          <visual>
+            <geometry><box size="${sx} ${sy} ${sz}"/></geometry>
+            <origin xyz="${x} ${y} ${z}" rpy="0 0 0"/>
+            <material name="workspace_wall"><color rgba="0.8 0.2 0.2 0.25"/></material>
+          </visual>
+          <collision>
+            <geometry><box size="${sx} ${sy} ${sz}"/></geometry>
+            <origin xyz="${x} ${y} ${z}" rpy="0 0 0"/>
+          </collision>
+        </xacro:macro>
+        <!-- +/-X walls: span the full inner Y extent -->
+        <xacro:wall_box sx="${wall_t}" sy="${2 * wall_hy}" sz="${wall_h}"
+                        x="${ wall_hx + wall_t / 2}" y="0" z="${wall_cz}"/>
+        <xacro:wall_box sx="${wall_t}" sy="${2 * wall_hy}" sz="${wall_h}"
+                        x="${-wall_hx - wall_t / 2}" y="0" z="${wall_cz}"/>
+        <!-- +/-Y walls: overrun in X by one thickness each side to close the corners -->
+        <xacro:wall_box sx="${2 * (wall_hx + wall_t)}" sy="${wall_t}" sz="${wall_h}"
+                        x="0" y="${ wall_hy + wall_t / 2}" z="${wall_cz}"/>
+        <xacro:wall_box sx="${2 * (wall_hx + wall_t)}" sy="${wall_t}" sz="${wall_h}"
+                        x="0" y="${-wall_hy - wall_t / 2}" z="${wall_cz}"/>
+      </link>
+      <joint name="workspace_walls_joint" type="fixed">
+        <parent link="${struct_name_prop}_link"/>
+        <child link="workspace_walls_link"/>
+        <origin xyz="0 0 0" rpy="0 0 0"/>
+      </joint>
+    </xacro:if>
     <xacro:load_robot
         parent="${struct_name_prop}_link"
@@ -96,6 +177,9 @@
         sim_isaac="$(arg sim_isaac)"
         use_external_cable="$(arg use_external_cable)"
-        initial_positions="${xacro.load_yaml(initial_positions_file)}">
-        <origin xyz="$(arg left_xyz)" rpy="$(arg left_rpy)"/>
+        initial_positions="${xacro.load_yaml(initial_positions_file)}"
+        hw_is_async="$(arg hw_is_async)"
+        hw_async_cores="$(arg left_async_cores)"
+        hw_async_priority="$(arg hw_async_priority)">
+        <origin xyz="0 ${ base_sep / 2} ${plate_th / 2}" rpy="$(arg left_rpy)"/>
     </xacro:load_robot>
     <xacro:load_robot
@@ -122,6 +206,9 @@
         sim_isaac="$(arg sim_isaac)"
         use_external_cable="$(arg use_external_cable)"
-        initial_positions="${xacro.load_yaml(initial_positions_file)}">
-        <origin xyz="$(arg right_xyz)" rpy="$(arg right_rpy)"/>
+        initial_positions="${xacro.load_yaml(initial_positions_file)}"
+        hw_is_async="$(arg hw_is_async)"
+        hw_async_cores="$(arg right_async_cores)"
+        hw_async_priority="$(arg hw_async_priority)">
+        <origin xyz="0 ${-base_sep / 2} ${plate_th / 2}" rpy="$(arg right_rpy)"/>
     </xacro:load_robot>
 </robot>

File: kortex_description/robots/kortex_robot.xacro (robot description, xacro)
@@ -29,5 +29,8 @@
     gripper_max_force:=100.0
     gripper_com_port:=/dev/ttyUSB0
-    moveit_active:=false">
+    moveit_active:=false
+    hw_is_async:=false
+    hw_async_cores:=[]
+    hw_async_priority:=80">
     <!-- Include and load arm macro files -->
     <xacro:include filename="$(find kortex_description)/arms/${arm}/${dof}dof/urdf/${arm}_macro.xacro" />
@@ -58,5 +61,8 @@
       use_external_cable="${use_external_cable}"
       initial_positions="${initial_positions}"
-      moveit_active="${moveit_active}">
+      moveit_active="${moveit_active}"
+      hw_is_async="${hw_is_async}"
+      hw_async_cores="${hw_async_cores}"
+      hw_async_priority="${hw_async_priority}">
       <xacro:insert_block name="origin" />
     </xacro:load_arm>

File: kortex_moveit_config/kinova_gen3_7dof_robotiq_2f_85_dual_moveit_config/config/dual_gen3.srdf.xacro (robot description, xacro)
@@ -9,4 +9,6 @@
   <xacro:arg name="right_prefix" default="right_"/>
   <xacro:arg name="struct_name"  default="dual_arm_structure"/>
+  <!-- Must match enable_walls in kortex_dual_robots.xacro -->
+  <xacro:arg name="enable_walls" default="true"/>
   <xacro:macro name="gen3_2f85_arm_srdf" params="prefix arm_group_name gripper_group_name ee_name">
     <group name="${arm_group_name}">
@@ -210,3 +212,12 @@
   <disable_collisions link1="$(arg struct_name)_link" link2="$(arg left_prefix)base_link"  reason="Adjacent"/>
   <disable_collisions link1="$(arg struct_name)_link" link2="$(arg right_prefix)base_link" reason="Adjacent"/>
+  <!-- Workspace walls stand ON the plate top face, so the two are coincident there.
+       MoveIt builds its ACM from THIS file only - adjacency across a fixed joint is
+       NOT inferred at runtime - so without this entry the walls would report a
+       permanent collision against the plate and every plan would fail.
+       The walls are intentionally left collision-enabled against every arm link;
+       that is the entire point of them. -->
+  <xacro:if value="$(arg enable_walls)">
+    <disable_collisions link1="workspace_walls_link" link2="$(arg struct_name)_link" reason="Adjacent"/>
+  </xacro:if>
 </robot>
