Commit message: remove trailing xacro:macro

File: kortex_description/grippers/robotiq_2f_140/urdf/robotiq_2f_140_macro.xacro (robot description, xacro)
@@ -39,4 +39,3 @@
       </xacro:if>
   </xacro:macro>
-  </xacro:macro>
 </robot>

Commit message: Update gripper descriptions for use on HW
Pass though more hardware parameters for gripper control:
* `use_internal_bus_gripper_comm`: specify if gripper comms will pass
  through the robot internally
* `(gripper_)include_ros2_control`: specify if a ros2_control instance
  is needed for the gripper (will be needed if we are simulating or
  directly communicating with the gripper via USB from the PC)
* `(gripper_)com_port`: specify the port the gripper can be exected on

File: kortex_description/grippers/robotiq_2f_140/urdf/robotiq_2f_140_macro.xacro (robot description, xacro)
@@ -10,11 +10,8 @@
     isaac_joint_commands:=/isaac_joint_commands
     isaac_joint_states:=/isaac_joint_states
-    use_internal_bus_gripper_comm:=false">
+    use_internal_bus_gripper_comm:=false
+    include_ros2_control:=true
+    com_port:=/dev/ttyUSB0">
     <xacro:include filename="$(find robotiq_description)/urdf/robotiq_2f_140_macro.urdf.xacro" />
-    <!-- Hardware talks directly to the gripper so we don't need ros2_control unless we are simulating -->
-    <xacro:property name="include_ros2_control" value="false"/>
-    <xacro:if value="${sim_ignition or sim_isaac or use_fake_hardware}">
-      <xacro:property name="include_ros2_control" value="true"/>
-    </xacro:if>
     <xacro:robotiq_gripper
         name="RobotiqGripperHardwareInterface"
@@ -22,4 +19,5 @@
         parent="${parent}"
         include_ros2_control="${include_ros2_control}"
+        com_port="${com_port}"
         use_fake_hardware="${use_fake_hardware}"
         fake_sensor_commands="${fake_sensor_commands}"

File: kortex_description/grippers/robotiq_2f_85/urdf/robotiq_2f_85_macro.xacro (robot description, xacro)
@@ -10,11 +10,8 @@
     isaac_joint_commands:=/isaac_joint_commands
     isaac_joint_states:=/isaac_joint_states
-    use_internal_bus_gripper_comm:=false">
+    use_internal_bus_gripper_comm:=false
+    include_ros2_control:=true
+    com_port:=/dev/ttyUSB0">
     <xacro:include filename="$(find robotiq_description)/urdf/robotiq_2f_85_macro.urdf.xacro" />
-    <!-- Hardware talks directly to the gripper so we don't need ros2_control unless we are simulating -->
-    <xacro:property name="include_ros2_control" value="false"/>
-    <xacro:if value="${sim_ignition or sim_isaac or use_fake_hardware}">
-      <xacro:property name="include_ros2_control" value="true"/>
-    </xacro:if>
     <xacro:robotiq_gripper
         name="RobotiqGripperHardwareInterface"
@@ -22,4 +19,5 @@
         parent="${parent}"
         include_ros2_control="${include_ros2_control}"
+        com_port="${com_port}"
         use_fake_hardware="${use_fake_hardware}"
         fake_sensor_commands="${fake_sensor_commands}"

File: kortex_description/robots/gen3_robotiq_2f_140.xacro (robot description, xacro)
@@ -6,7 +6,20 @@
     <xacro:arg name="vision" default="true" />
     <xacro:arg name="gripper" default="robotiq_2f_140" />
+    <xacro:arg name="use_internal_bus_gripper_comm" default="false" />
+    <xacro:arg name="gripper_include_ros2_control" default="true" />
+    <xacro:arg name="gripper_com_port" default="/dev/ttyUSB0" />
     <xacro:arg name="sim" default="false" />
     <xacro:arg name="prefix" default="" />
     <xacro:include filename="$(find kortex_description)/robots/kortex_robot.xacro" />
-    <xacro:load_robot arm="$(arg arm)" gripper="$(arg gripper)" dof="$(arg dof)" vision="$(arg vision)" sim="$(arg sim)" prefix="$(arg prefix)"/>
+    <xacro:load_robot
+      arm="$(arg arm)"
+      gripper="$(arg gripper)"
+      dof="$(arg dof)"
+      vision="$(arg vision)"
+      sim="$(arg sim)"
+      prefix="$(arg prefix)"
+      use_internal_bus_gripper_comm="$(arg use_internal_bus_gripper_comm)"
+      gripper_include_ros2_control="$(arg gripper_include_ros2_control)"
+      gripper_com_port="$(arg gripper_com_port)">
+    </xacro:robotiq_gripper>
 </robot>

File: kortex_description/robots/gen3_robotiq_2f_85.xacro (robot description, xacro)
@@ -6,7 +6,20 @@
     <xacro:arg name="vision" default="true" />
     <xacro:arg name="gripper" default="robotiq_2f_85" />
+    <xacro:arg name="use_internal_bus_gripper_comm" default="false" />
+    <xacro:arg name="gripper_include_ros2_control" default="true" />
+    <xacro:arg name="gripper_com_port" default="/dev/ttyUSB0" />
     <xacro:arg name="sim" default="false" />
     <xacro:arg name="prefix" default="" />
     <xacro:include filename="$(find kortex_description)/robots/kortex_robot.xacro" />
-    <xacro:load_robot arm="$(arg arm)" gripper="$(arg gripper)" dof="$(arg dof)" vision="$(arg vision)" sim="$(arg sim)" prefix="$(arg prefix)" />
+    <xacro:load_robot
+      arm="$(arg arm)"
+      gripper="$(arg gripper)"
+      dof="$(arg dof)"
+      vision="$(arg vision)"
+      sim="$(arg sim)"
+      prefix="$(arg prefix)"
+      use_internal_bus_gripper_comm="$(arg use_internal_bus_gripper_comm)"
+      gripper_include_ros2_control="$(arg gripper_include_ros2_control)"
+      gripper_com_port="$(arg gripper_com_port)">
+    </xacro:robotiq_gripper>
 </robot>

File: kortex_description/robots/kortex_robot.xacro (robot description, xacro)
@@ -28,5 +28,7 @@
     initial_positions:=${dict(joint_1=0.0,joint_2=0.0,joint_3=0.0,joint_4=0.0,joint_5=0.0,joint_6=0.0,joint_7=0.0)}
     gripper_max_velocity:=100.0
-    gripper_max_force:=100.0">
+    gripper_max_force:=100.0
+    gripper_include_ros2_control:=true
+    gripper_com_port:=/dev/ttyUSB0">
     <!-- Include and load arm macro files -->
     <xacro:include filename="$(find kortex_description)/arms/${arm}/${dof}dof/urdf/${arm}_macro.xacro" />
@@ -82,5 +84,7 @@
         isaac_joint_commands="${isaac_joint_commands}"
         isaac_joint_states="${isaac_joint_states}"
-        use_internal_bus_gripper_comm="${use_internal_bus_gripper_comm}"/>
+        use_internal_bus_gripper_comm="${use_internal_bus_gripper_comm}"
+        include_ros2_control="${gripper_include_ros2_control}"
+        com_port="${gripper_com_port}"/>
     </xacro:unless>
   </xacro:macro>

Commit message: Use internal comm param in gripper macros
Add `use_internal_bus_gripper_comm` param back into `load_gripper` macro
and use it to determine whether or not to launch a ros2_control instance
for the gripper. We expect `use_internal_bus_gripper_comm` to be false
if we are running the gripper in simulation or the gripper is
connected to the PC via USB rather than through the internal kinova
bus. In those cases we need to launch a ros2_control instance to control
the gripper.

Remove `gripper_include_ros2_control` param from macros since we're
using the `use_internal_bus_gripper_comm` param and the simulation
params to determine if we need to launch a ros2_control instance for the
gripper.

Update the kortex_description readme to reflect these changes.

File: kortex_description/grippers/robotiq_2f_140/urdf/robotiq_2f_140_macro.xacro (robot description, xacro)
@@ -10,7 +10,12 @@
     isaac_joint_commands:=/isaac_joint_commands
     isaac_joint_states:=/isaac_joint_states
-    include_ros2_control:=true
+    use_internal_bus_gripper_comm:=false
     com_port:=/dev/ttyUSB0">
     <xacro:include filename="$(find robotiq_description)/urdf/robotiq_2f_140_macro.urdf.xacro" />
+    <!-- Hardware talks directly to the gripper so we don't need ros2_control unless we are simulating -->
+    <xacro:property name="include_ros2_control" value="false"/>
+    <xacro:if value="${sim_ignition or sim_isaac or use_fake_hardware or not use_internal_bus_gripper_comm}">
+      <xacro:property name="include_ros2_control" value="true"/>
+    </xacro:if>
     <xacro:robotiq_gripper
         name="RobotiqGripperHardwareInterface"

File: kortex_description/grippers/robotiq_2f_85/urdf/robotiq_2f_85_macro.xacro (robot description, xacro)
@@ -10,7 +10,12 @@
     isaac_joint_commands:=/isaac_joint_commands
     isaac_joint_states:=/isaac_joint_states
-    include_ros2_control:=true
+    use_internal_bus_gripper_comm:=false
     com_port:=/dev/ttyUSB0">
     <xacro:include filename="$(find robotiq_description)/urdf/robotiq_2f_85_macro.urdf.xacro" />
+    <!-- Hardware talks directly to the gripper so we don't need ros2_control unless we are simulating -->
+    <xacro:property name="include_ros2_control" value="false"/>
+    <xacro:if value="${sim_ignition or sim_isaac or use_fake_hardware or not use_internal_bus_gripper_comm}">
+      <xacro:property name="include_ros2_control" value="true"/>
+    </xacro:if>
     <xacro:robotiq_gripper
         name="RobotiqGripperHardwareInterface"

File: kortex_description/robots/gen3_robotiq_2f_140.xacro (robot description, xacro)
@@ -7,5 +7,4 @@
     <xacro:arg name="gripper" default="robotiq_2f_140" />
     <xacro:arg name="use_internal_bus_gripper_comm" default="false" />
-    <xacro:arg name="gripper_include_ros2_control" default="true" />
     <xacro:arg name="gripper_com_port" default="/dev/ttyUSB0" />
     <xacro:arg name="sim" default="false" />
@@ -20,5 +19,4 @@
       prefix="$(arg prefix)"
       use_internal_bus_gripper_comm="$(arg use_internal_bus_gripper_comm)"
-      gripper_include_ros2_control="$(arg gripper_include_ros2_control)"
       gripper_com_port="$(arg gripper_com_port)">
     </xacro:load_robot>

File: kortex_description/robots/gen3_robotiq_2f_85.xacro (robot description, xacro)
@@ -7,5 +7,4 @@
     <xacro:arg name="gripper" default="robotiq_2f_85" />
     <xacro:arg name="use_internal_bus_gripper_comm" default="false" />
-    <xacro:arg name="gripper_include_ros2_control" default="true" />
     <xacro:arg name="gripper_com_port" default="/dev/ttyUSB0" />
     <xacro:arg name="sim" default="false" />
@@ -20,5 +19,4 @@
       prefix="$(arg prefix)"
       use_internal_bus_gripper_comm="$(arg use_internal_bus_gripper_comm)"
-      gripper_include_ros2_control="$(arg gripper_include_ros2_control)"
       gripper_com_port="$(arg gripper_com_port)">
     </xacro:load_robot>

File: kortex_description/robots/kortex_robot.xacro (robot description, xacro)
@@ -29,5 +29,4 @@
     gripper_max_velocity:=100.0
     gripper_max_force:=100.0
-    gripper_include_ros2_control:=true
     gripper_com_port:=/dev/ttyUSB0">
     <!-- Include and load arm macro files -->
@@ -84,5 +83,5 @@
         isaac_joint_commands="${isaac_joint_commands}"
         isaac_joint_states="${isaac_joint_states}"
-        include_ros2_control="${gripper_include_ros2_control}"
+        use_internal_bus_gripper_comm="${use_internal_bus_gripper_comm}"
         com_port="${gripper_com_port}"/>
     </xacro:unless>
