Commit message: Gen3_Lite Moveit_Package rectification

File: kortex_moveit_config/kinova_gen3_lite_moveit_config/config/gen3_lite_gen3_lite_2f.ros2_control.xacro (robot description, xacro)
@@ -1,5 +1,5 @@
 <?xml version="1.0"?>
 <robot xmlns:xacro="http://www.ros.org/wiki/xacro">
-    <xacro:macro name="gen3_lite_ros2_control" params="name initial_positions_file">
+    <xacro:macro name="gen3_lite_gen3_lite_2f_ros2_control" params="name initial_positions_file">
         <xacro:property name="initial_positions" value="${load_yaml(initial_positions_file)['initial_positions']}"/>
         <ros2_control name="${name}" type="system">
