Commit message: Add support for ros2_control of the kinova gen3 lite

File: kortex_description/arms/gen3_lite/6dof/urdf/gen3_lite_macro.xacro (robot description, xacro)
@@ -3,5 +3,46 @@
   <!-- Propagate last link name information because it is the gripper's parent link -->
   <xacro:property name="last_arm_link" value="dummy_link"/>
-  <xacro:macro name="load_arm" params="parent:='' dof vision prefix *origin">
+  <xacro:macro name="load_arm" params="
+    parent
+    dof
+    vision
+    prefix
+    *origin
+    robot_ip
+    username:=admin
+    password:=admin
+    port:=10000
+    port_realtime:=10001
+    session_inactivity_timeout_ms:=6000
+    connection_inactivity_timeout_ms:=2000
+    use_internal_bus_gripper_comm:=false
+    use_fake_hardware:=false
+    fake_sensor_commands:=false
+    sim_gazebo:=false
+    sim_ignition:=false
+    initial_positions:=${dict(joint_1=0.0,joint_2=0.0,joint_3=0.0,joint_4=0.0,joint_5=0.0,joint_6=0.0)}" >
+    <!-- ros2 control include -->
+    <xacro:include filename="$(find kortex_description)/arms/gen3_lite/${dof}dof/urdf/kortex.ros2_control.xacro" />
+    <xacro:kortex_ros2_control
+      name="${prefix}KortexMultiInterfaceHardware" prefix="${prefix}"
+      use_fake_hardware="${use_fake_hardware}"
+      fake_sensor_commands="${fake_sensor_commands}"
+      sim_gazebo="${sim_gazebo}"
+      sim_ignition="${sim_ignition}"
+      tf_prefix=""
+      initial_positions="${initial_positions}"
+      robot_ip="${robot_ip}"
+      username="${username}"
+      password="${password}"
+      port="${port}"
+      port_realtime="${port_realtime}"
+      session_inactivity_timeout_ms="${session_inactivity_timeout_ms}"
+      connection_inactivity_timeout_ms="${connection_inactivity_timeout_ms}"
+      use_internal_bus_gripper_comm="${use_internal_bus_gripper_comm}" />
+    <joint name="${prefix}base_joint" type="fixed">
+      <xacro:insert_block name="origin" />
+      <parent link="${parent}"/>
+      <child link="${prefix}base_link" />
+    </joint>
     <link name="${prefix}base_link">
       <inertial>

Commit message: Support Gen3 lite Hardware

File: kortex_description/arms/gen3_lite/6dof/urdf/gen3_lite_macro.xacro (robot description, xacro)
@@ -24,6 +24,12 @@
     <!-- ros2 control include -->
     <xacro:include filename="$(find kortex_description)/arms/gen3_lite/${dof}dof/urdf/kortex.ros2_control.xacro" />
+    <xacro:if value="${sim_ignition or sim_gazebo}">
+      <xacro:property name="ros2_control_name" value="IgnitionSystem"/>
+    </xacro:if>
+    <xacro:unless value="${use_fake_hardware or sim_ignition or sim_gazebo}">
+      <xacro:property name="ros2_control_name" value="${prefix}KortexMultiInterfaceHardware"/>
+    </xacro:unless>
     <xacro:kortex_ros2_control
-      name="${prefix}KortexMultiInterfaceHardware" prefix="${prefix}"
+      name="${ros2_control_name}" prefix="${prefix}"
       use_fake_hardware="${use_fake_hardware}"
       fake_sensor_commands="${fake_sensor_commands}"

File: kortex_description/arms/gen3_lite/6dof/urdf/kortex.ros2_control.xacro (robot description, xacro)
@@ -42,5 +42,5 @@
           <param name="tf_prefix">"${tf_prefix}"</param>
           <param name="use_internal_bus_gripper_comm">${use_internal_bus_gripper_comm}</param>
-          <param name="gripper_joint_name">finger_joint</param>
+          <param name="gripper_joint_name">${prefix}right_finger_bottom_joint</param>
         </xacro:unless>
       </hardware>
@@ -48,5 +48,5 @@
         <command_interface name="position">
           <param name="min">-2.69</param>
-          <param name="max">2.68</param>
+          <param name="max">2.69</param>
         </command_interface>
         <command_interface name="velocity">
@@ -63,5 +63,5 @@
         <command_interface name="position">
           <param name="min">-2.69</param>
-          <param name="max">2.69</param>
+          <param name="max">2.36</param>
         </command_interface>
         <command_interface name="velocity">

Commit message: Fix launch for use_fake_hardware

File: kortex_description/arms/gen3_lite/6dof/urdf/gen3_lite_macro.xacro (robot description, xacro)
@@ -27,4 +27,7 @@
       <xacro:property name="ros2_control_name" value="IgnitionSystem"/>
     </xacro:if>
+     <xacro:if value="${use_fake_hardware}">
+      <xacro:property name="ros2_control_name" value="GenericSystem"/>
+    </xacro:if>
     <xacro:unless value="${use_fake_hardware or sim_ignition or sim_gazebo}">
       <xacro:property name="ros2_control_name" value="${prefix}KortexMultiInterfaceHardware"/>

Commit message: Support Gen3 lite Hardware (#73)
* Support Gen3 lite Hardware
* Fix launch for use_fake_hardware
* reverse gripper joints in URDF
* Improve Protective Stop Reset and General Driver Robusteness (#75)
* Add test huge joint space jump.

Co-authored-by: Abishalini <abi.gpuram@gmail.com>
Co-authored-by: livanov93 <lovro.ivanov@gmail.com>

File: kortex_description/arms/gen3_lite/6dof/urdf/gen3_lite_macro.xacro (robot description, xacro)
@@ -24,6 +24,15 @@
     <!-- ros2 control include -->
     <xacro:include filename="$(find kortex_description)/arms/gen3_lite/${dof}dof/urdf/kortex.ros2_control.xacro" />
+    <xacro:if value="${sim_ignition or sim_gazebo}">
+      <xacro:property name="ros2_control_name" value="IgnitionSystem"/>
+    </xacro:if>
+     <xacro:if value="${use_fake_hardware}">
+      <xacro:property name="ros2_control_name" value="GenericSystem"/>
+    </xacro:if>
+    <xacro:unless value="${use_fake_hardware or sim_ignition or sim_gazebo}">
+      <xacro:property name="ros2_control_name" value="${prefix}KortexMultiInterfaceHardware"/>
+    </xacro:unless>
     <xacro:kortex_ros2_control
-      name="${prefix}KortexMultiInterfaceHardware" prefix="${prefix}"
+      name="${ros2_control_name}" prefix="${prefix}"
       use_fake_hardware="${use_fake_hardware}"
       fake_sensor_commands="${fake_sensor_commands}"

Commit message: Clean up gen3 lite macro

File: kortex_description/arms/gen3_lite/6dof/urdf/gen3_lite_macro.xacro (robot description, xacro)
@@ -29,13 +29,4 @@
     <!-- ros2 control include -->
     <xacro:include filename="$(find kortex_description)/arms/gen3_lite/${dof}dof/urdf/kortex.ros2_control.xacro" />
-    <xacro:if value="${sim_ignition or sim_gazebo}">
-      <xacro:property name="ros2_control_name" value="IgnitionSystem"/>
-    </xacro:if>
-     <xacro:if value="${use_fake_hardware}">
-      <xacro:property name="ros2_control_name" value="GenericSystem"/>
-    </xacro:if>
-    <xacro:unless value="${use_fake_hardware or sim_ignition or sim_gazebo}">
-      <xacro:property name="ros2_control_name" value="${prefix}KortexMultiInterfaceHardware"/>
-    </xacro:unless>
     <xacro:kortex_ros2_control
       name="${ros2_control_name}" prefix="${prefix}"

Commit message: Update gen3_lite macros
Update the kinova gen3_lite macros to pass through the required
parameters.

File: kortex_description/arms/gen3_lite/6dof/urdf/gen3_lite_macro.xacro (robot description, xacro)
@@ -17,8 +17,15 @@
     connection_inactivity_timeout_ms:=2000
     use_internal_bus_gripper_comm:=false
+    gripper_joint_name
+    gripper_max_velocity:=100.0
+    gripper_max_force:=100.0
     use_fake_hardware:=false
     fake_sensor_commands:=false
     sim_gazebo:=false
     sim_ignition:=false
+    sim_isaac:=false
+    isaac_joint_commands:=/isaac_joint_commands
+    isaac_joint_states:=/isaac_joint_states
+    use_external_cable:=false
     initial_positions:=${dict(joint_1=0.0,joint_2=0.0,joint_3=0.0,joint_4=0.0,joint_5=0.0,joint_6=0.0)}" >
     <!-- ros2 control include -->
@@ -39,4 +46,7 @@
       sim_gazebo="${sim_gazebo}"
       sim_ignition="${sim_ignition}"
+      sim_isaac="${sim_isaac}"
+      isaac_joint_commands="${isaac_joint_commands}"
+      isaac_joint_states="${isaac_joint_states}"
       tf_prefix=""
       initial_positions="${initial_positions}"
@@ -48,5 +58,8 @@
       session_inactivity_timeout_ms="${session_inactivity_timeout_ms}"
       connection_inactivity_timeout_ms="${connection_inactivity_timeout_ms}"
-      use_internal_bus_gripper_comm="${use_internal_bus_gripper_comm}" />
+      use_internal_bus_gripper_comm="${use_internal_bus_gripper_comm}"
+      gripper_max_velocity="${gripper_max_velocity}"
+      gripper_max_force="${gripper_max_force}"
+      gripper_joint_name="${gripper_joint_name}"/>
     <joint name="${prefix}base_joint" type="fixed">
       <xacro:insert_block name="origin" />

File: kortex_description/arms/gen3_lite/6dof/urdf/kortex.ros2_control.xacro (robot description, xacro)
@@ -8,4 +8,7 @@
     sim_gazebo:=false
     sim_ignition:=false
+    sim_isaac:=false
+    isaac_joint_commands:=/isaac_joint_commands
+    isaac_joint_states:=/isaac_joint_states
     use_internal_bus_gripper_comm:=false
     tf_prefix
@@ -17,5 +20,8 @@
     port_realtime
     session_inactivity_timeout_ms
-    connection_inactivity_timeout_ms">
+    connection_inactivity_timeout_ms
+    gripper_joint_name
+    gripper_max_velocity:=100.0
+    gripper_max_force:=100.0">
     <ros2_control name="${name}" type="system">
       <hardware>
@@ -26,4 +32,9 @@
           <plugin>ign_ros2_control/IgnitionSystem</plugin>
         </xacro:if>
+        <xacro:if value="${sim_isaac}">
+          <plugin>topic_based_ros2_control/TopicBasedSystem</plugin>
+          <param name="joint_commands_topic">${isaac_joint_commands}</param>
+          <param name="joint_states_topic">${isaac_joint_states}</param>
+        </xacro:if>
         <xacro:if value="${use_fake_hardware}">
           <plugin>fake_components/GenericSystem</plugin>
@@ -31,5 +42,5 @@
           <param name="state_following_offset">0.0</param>
         </xacro:if>
-        <xacro:unless value="${use_fake_hardware or sim_gazebo or sim_ignition}">
+        <xacro:unless value="${use_fake_hardware or sim_gazebo or sim_ignition or sim_isaac}">
           <plugin>kortex_driver/KortexMultiInterfaceHardware</plugin>
           <param name="robot_ip">${robot_ip}</param>
@@ -42,5 +53,7 @@
           <param name="tf_prefix">"${tf_prefix}"</param>
           <param name="use_internal_bus_gripper_comm">${use_internal_bus_gripper_comm}</param>
-          <param name="gripper_joint_name">${prefix}right_finger_bottom_joint</param>
+          <param name="gripper_joint_name">${gripper_joint_name}</param>
+          <param name="gripper_max_velocity">${gripper_max_velocity}</param>
+          <param name="gripper_max_force">${gripper_max_force}</param>
         </xacro:unless>
       </hardware>

File: kortex_description/grippers/gen3_lite_2f/urdf/gen3_lite_2f_macro.xacro (robot description, xacro)
@@ -1,5 +1,14 @@
 <?xml version="1.0"?>
 <robot name="gen3_lite_2f_gripper" xmlns:xacro="http://ros.org/wiki/xacro">
-  <xacro:macro name="load_gripper" params="parent prefix">
+  <xacro:macro name="load_gripper" params="
+    parent
+    prefix
+    use_fake_hardware:=false
+    fake_sensor_commands:=false
+    sim_ignition:=false
+    sim_isaac:=false
+    isaac_joint_commands:=/isaac_joint_commands
+    isaac_joint_states:=/isaac_joint_states
+    use_internal_bus_gripper_comm:=true">
     <!-- Tool frame used by the arm -->
     <link name="${prefix}tool_frame"/>
