Commit message: Creating Gen3 Lite specific instructions and launch file

File: kortex_description/arms/gen3_lite/6dof/urdf/gen3_lite_macro.xacro (robot description, xacro)
@@ -16,5 +16,5 @@
     session_inactivity_timeout_ms:=6000
     connection_inactivity_timeout_ms:=2000
-    use_internal_bus_gripper_comm:=false
+    use_internal_bus_gripper_comm:=true
     gripper_joint_name
     gripper_max_velocity:=100.0
@@ -76,14 +76,14 @@
         <origin xyz="0 0 0" rpy="0 0 0" />
         <geometry>
-          <mesh filename="package://kortex_description/arms/gen3_lite/${dof}dof/meshes/base_link.STL" />
-        </geometry>
-        <material name="">
-          <color rgba="0.803 0.824 0.820 1" />
-        </material>
-      </visual>
-      <collision>
-        <origin xyz="0 0 0" rpy="0 0 0" />
-        <geometry>
-          <mesh filename="package://kortex_description/arms/gen3_lite/${dof}dof/meshes/base_link.STL" />
+          <mesh filename="file://$(find kortex_description)/arms/gen3_lite/${dof}dof/meshes/base_link.STL" />
+        </geometry>
+        <material name="">
+          <color rgba="0.803 0.824 0.820 1" />
+        </material>
+      </visual>
+      <collision>
+        <origin xyz="0 0 0" rpy="0 0 0" />
+        <geometry>
+          <mesh filename="file://$(find kortex_description)/arms/gen3_lite/${dof}dof/meshes/base_link.STL" />
         </geometry>
       </collision>
@@ -101,14 +101,14 @@
         <origin xyz="0 0 0" rpy="0 0 0" />
         <geometry>
-          <mesh filename="package://kortex_description/arms/gen3_lite/${dof}dof/meshes/shoulder_link.STL" />
-        </geometry>
-        <material name="">
-          <color rgba="0.803 0.824 0.820 1" />
-        </material>
-      </visual>
-      <collision>
-        <origin xyz="0 0 0" rpy="0 0 0" />
-        <geometry>
-          <mesh filename="package://kortex_description/arms/gen3_lite/${dof}dof/meshes/shoulder_link.STL" />
+          <mesh filename="file://$(find kortex_description)/arms/gen3_lite/${dof}dof/meshes/shoulder_link.STL" />
+        </geometry>
+        <material name="">
+          <color rgba="0.803 0.824 0.820 1" />
+        </material>
+      </visual>
+      <collision>
+        <origin xyz="0 0 0" rpy="0 0 0" />
+        <geometry>
+          <mesh filename="file://$(find kortex_description)/arms/gen3_lite/${dof}dof/meshes/shoulder_link.STL" />
         </geometry>
       </collision>
@@ -133,14 +133,14 @@
         <origin xyz="0 0 0" rpy="0 0 0" />
         <geometry>
-          <mesh filename="package://kortex_description/arms/gen3_lite/${dof}dof/meshes/arm_link.STL" />
-        </geometry>
-        <material name="">
-          <color rgba="0.803 0.824 0.820 1" />
-        </material>
-      </visual>
-      <collision>
-        <origin xyz="0 0 0" rpy="0 0 0" />
-        <geometry>
-          <mesh filename="package://kortex_description/arms/gen3_lite/${dof}dof/meshes/arm_link.STL" />
+          <mesh filename="file://$(find kortex_description)/arms/gen3_lite/${dof}dof/meshes/arm_link.STL" />
+        </geometry>
+        <material name="">
+          <color rgba="0.803 0.824 0.820 1" />
+        </material>
+      </visual>
+      <collision>
+        <origin xyz="0 0 0" rpy="0 0 0" />
+        <geometry>
+          <mesh filename="file://$(find kortex_description)/arms/gen3_lite/${dof}dof/meshes/arm_link.STL" />
         </geometry>
       </collision>
@@ -165,14 +165,14 @@
         <origin xyz="0 0 0" rpy="0 0 0" />
         <geometry>
-          <mesh filename="package://kortex_description/arms/gen3_lite/${dof}dof/meshes/forearm_link.STL" />
-        </geometry>
-        <material name="">
-          <color rgba="0.803 0.824 0.820 1" />
-        </material>
-      </visual>
-      <collision>
-        <origin xyz="0 0 0" rpy="0 0 0" />
-        <geometry>
-          <mesh filename="package://kortex_description/arms/gen3_lite/${dof}dof/meshes/forearm_link.STL" />
+          <mesh filename="file://$(find kortex_description)/arms/gen3_lite/${dof}dof/meshes/forearm_link.STL" />
+        </geometry>
+        <material name="">
+          <color rgba="0.803 0.824 0.820 1" />
+        </material>
+      </visual>
+      <collision>
+        <origin xyz="0 0 0" rpy="0 0 0" />
+        <geometry>
+          <mesh filename="file://$(find kortex_description)/arms/gen3_lite/${dof}dof/meshes/forearm_link.STL" />
         </geometry>
       </collision>
@@ -197,14 +197,14 @@
         <origin xyz="0 0 0" rpy="0 0 0" />
         <geometry>
-          <mesh filename="package://kortex_description/arms/gen3_lite/${dof}dof/meshes/lower_wrist_link.STL" />
-        </geometry>
-        <material name="">
-          <color rgba="0.803 0.824 0.820 1" />
-        </material>
-      </visual>
-      <collision>
-        <origin xyz="0 0 0" rpy="0 0 0" />
-        <geometry>
-          <mesh filename="package://kortex_description/arms/gen3_lite/${dof}dof/meshes/lower_wrist_link.STL" />
+          <mesh filename="file://$(find kortex_description)/arms/gen3_lite/${dof}dof/meshes/lower_wrist_link.STL" />
+        </geometry>
+        <material name="">
+          <color rgba="0.803 0.824 0.820 1" />
+        </material>
+      </visual>
+      <collision>
+        <origin xyz="0 0 0" rpy="0 0 0" />
+        <geometry>
+          <mesh filename="file://$(find kortex_description)/arms/gen3_lite/${dof}dof/meshes/lower_wrist_link.STL" />
         </geometry>
       </collision>
@@ -229,14 +229,14 @@
         <origin xyz="0 0 0" rpy="0 0 0" />
         <geometry>
-          <mesh filename="package://kortex_description/arms/gen3_lite/${dof}dof/meshes/upper_wrist_link.STL" />
-        </geometry>
-        <material name="">
-          <color rgba="0.803 0.824 0.820 1" />
-        </material>
-      </visual>
-      <collision>
-        <origin xyz="0 0 0" rpy="0 0 0" />
-        <geometry>
-          <mesh filename="package://kortex_description/arms/gen3_lite/${dof}dof/meshes/upper_wrist_link.STL" />
+          <mesh filename="file://$(find kortex_description)/arms/gen3_lite/${dof}dof/meshes/upper_wrist_link.STL" />
+        </geometry>
+        <material name="">
+          <color rgba="0.803 0.824 0.820 1" />
+        </material>
+      </visual>
+      <collision>
+        <origin xyz="0 0 0" rpy="0 0 0" />
+        <geometry>
+          <mesh filename="file://$(find kortex_description)/arms/gen3_lite/${dof}dof/meshes/upper_wrist_link.STL" />
         </geometry>
       </collision>

File: kortex_description/arms/gen3_lite/6dof/urdf/kortex.ros2_control.xacro (robot description, xacro)
@@ -11,5 +11,5 @@
     isaac_joint_commands:=/isaac_joint_commands
     isaac_joint_states:=/isaac_joint_states
-    use_internal_bus_gripper_comm:=false
+    use_internal_bus_gripper_comm:=true
     tf_prefix
     initial_positions:=${dict(joint_1=0.0,joint_2=0.0,joint_3=0.0,joint_4=0.0,joint_5=0.0,joint_6=0.0)}
@@ -124,13 +124,9 @@
         <state_interface name="effort"/>
       </joint>
-      <xacro:unless value="${use_fake_hardware or sim_gazebo or sim_ignition or sim_isaac}">
-        <xacro:if value="${use_internal_bus_gripper_comm}">
-          <joint name="${prefix}right_finger_bottom_joint">
-            <command_interface name="position"/>
-            <state_interface name="position"/>
-            <state_interface name="velocity"/>
-          </joint>
-        </xacro:if>
-      </xacro:unless>
+      <joint name="${prefix}right_finger_bottom_joint">
+        <command_interface name="position"/>
+        <state_interface name="position"/>
+        <state_interface name="velocity"/>
+      </joint>
     </ros2_control>
   </xacro:macro>

File: kortex_description/grippers/gen3_lite_2f/urdf/gen3_lite_2f.ros2_control.xacro (robot description, xacro)
@@ -9,5 +9,16 @@
         isaac_joint_commands:=/isaac_joint_commands
         isaac_joint_states:=/isaac_joint_states
-        use_internal_bus_gripper_comm:=false">
+        use_internal_bus_gripper_comm:=true
+        gripper_joint_name:=right_finger_bottom_joint
+        tf_prefix:=''
+        robot_ip:=192.168.1.10
+        username:=admin
+        password:=admin
+        port:=10000
+        port_realtime:=10001
+        session_inactivity_timeout_ms:=60000
+        connection_inactivity_timeout_ms:=2000
+        gripper_max_velocity:=100.0
+        gripper_max_force:=100.0">
         <ros2_control name="GripperHardwareInterface" type="system">
             <hardware>
@@ -23,7 +34,22 @@
                 <xacro:if value="${use_fake_hardware}">
                     <plugin>mock_components/GenericSystem</plugin>
-                    <param name="fake_sensor_commands">${fake_sensor_commands}</param>
+                    <param name="mock_sensor_commands">${fake_sensor_commands}</param>
                     <param name="state_following_offset">0.0</param>
                 </xacro:if>
+                <xacro:unless value="${sim_isaac or sim_ignition or use_fake_hardware}">
+                    <plugin>kortex_driver/KortexMultiInterfaceHardware</plugin>
+                    <param name="robot_ip">${robot_ip}</param>
+                    <param name="username">${username}</param>
+                    <param name="password">${password}</param>
+                    <param name="port">${port}</param>
+                    <param name="port_realtime">${port_realtime}</param>
+                    <param name="session_inactivity_timeout_ms">${session_inactivity_timeout_ms}</param>
+                    <param name="connection_inactivity_timeout_ms">${connection_inactivity_timeout_ms}</param>
+                    <param name="tf_prefix">"${tf_prefix}"</param>
+                    <param name="use_internal_bus_gripper_comm">${use_internal_bus_gripper_comm}</param>
+                    <param name="gripper_joint_name">${gripper_joint_name}</param>
+                    <param name="gripper_max_velocity">${gripper_max_velocity}</param>
+                    <param name="gripper_max_force">${gripper_max_force}</param>
+                </xacro:unless>
             </hardware>
             <!-- Joint interfaces -->
@@ -32,7 +58,9 @@
                 <command_interface name="position" />
                 <state_interface name="position">
-                    <param name="initial_value">0.85</param>
+                    <param name="initial_value">0.0</param>
                 </state_interface>
-                <state_interface name="velocity"/>
+                <state_interface name="velocity">
+                    <param name="initial_value">0.0</param>
+                </state_interface>
             </joint>
             <!-- When simulating we need to include the rest of the gripper joints -->

File: kortex_description/grippers/gen3_lite_2f/urdf/gen3_lite_2f_macro.xacro (robot description, xacro)
@@ -4,4 +4,5 @@
     parent
     prefix
+    com_port
     use_fake_hardware:=false
     fake_sensor_commands:=false
@@ -11,14 +12,4 @@
     isaac_joint_states:=/isaac_joint_states
     use_internal_bus_gripper_comm:=true">
-    <xacro:include filename="$(find kortex_description)/grippers/gen3_lite_2f/urdf/gen3_lite_2f.ros2_control.xacro" />
-    <xacro:gripper_ros2_control
-      prefix="${prefix}"
-      use_fake_hardware="${use_fake_hardware}"
-      fake_sensor_commands="${fake_sensor_commands}"
-      sim_ignition="${sim_ignition}"
-      sim_isaac="${sim_isaac}"
-      isaac_joint_commands="${isaac_joint_commands}"
-      isaac_joint_states="${isaac_joint_states}"
-      use_internal_bus_gripper_comm="${use_internal_bus_gripper_comm}"/>
     <!-- Tool frame used by the arm -->
     <link name="${prefix}tool_frame"/>
@@ -45,5 +36,5 @@
         <origin xyz="0 0 0" rpy="0 0 0" />
         <geometry>
-          <mesh filename="package://kortex_description/grippers/gen3_lite_2f/meshes/gripper_base_link.STL" />
+          <mesh filename="file://$(find kortex_description)/grippers/gen3_lite_2f/meshes/gripper_base_link.STL" />
         </geometry>
         <material name="">
@@ -54,5 +45,5 @@
         <origin xyz="0 0 0" rpy="0 0 0" />
         <geometry>
-          <mesh filename="package://kortex_description/grippers/gen3_lite_2f/meshes/gripper_base_link.STL" />
+          <mesh filename="file://$(find kortex_description)/grippers/gen3_lite_2f/meshes/gripper_base_link.STL" />
         </geometry>
       </collision>
@@ -70,5 +61,5 @@
       <origin xyz="0 0 0" rpy="0 0 0" />
       <geometry>
-        <mesh filename="package://kortex_description/grippers/gen3_lite_2f/meshes/right_finger_prox_link.STL" />
+        <mesh filename="file://$(find kortex_description)/grippers/gen3_lite_2f/meshes/right_finger_prox_link.STL" />
       </geometry>
       <material name="">
@@ -79,5 +70,5 @@
       <origin xyz="0 0 0" rpy="0 0 0" />
       <geometry>
-        <mesh filename="package://kortex_description/grippers/gen3_lite_2f/meshes/right_finger_prox_link.STL" />
+        <mesh filename="file://$(find kortex_description)/grippers/gen3_lite_2f/meshes/right_finger_prox_link.STL" />
       </geometry>
     </collision>
@@ -92,5 +83,5 @@
       <child link="${prefix}right_finger_prox_link" />
       <axis xyz="0 0 -1" />
-      <limit lower="0.0" upper="0.85" effort="1000" velocity="0.6" />
+      <limit lower="0.0" upper="0.85" effort="50" velocity="0.6" />
     </joint>
     <link name="${prefix}right_finger_dist_link">
@@ -103,5 +94,5 @@
         <origin xyz="0 0 0" rpy="0 0 0" />
         <geometry>
-          <mesh filename="package://kortex_description/grippers/gen3_lite_2f/meshes/right_finger_dist_link.STL" />
+          <mesh filename="file://$(find kortex_description)/grippers/gen3_lite_2f/meshes/right_finger_dist_link.STL" />
         </geometry>
         <material name="">
@@ -112,5 +103,5 @@
         <origin xyz="0 0 0" rpy="0 0 0" />
         <geometry>
-          <mesh filename="package://kortex_description/grippers/gen3_lite_2f/meshes/right_finger_dist_link.STL" />
+          <mesh filename="file://$(find kortex_description)/grippers/gen3_lite_2f/meshes/right_finger_dist_link.STL" />
         </geometry>
       </collision>
@@ -136,5 +127,5 @@
         <origin xyz="0 0 0" rpy="0 0 0" />
         <geometry>
-          <mesh filename="package://kortex_description/grippers/gen3_lite_2f/meshes/left_finger_prox_link.STL" />
+          <mesh filename="file://$(find kortex_description)/grippers/gen3_lite_2f/meshes/left_finger_prox_link.STL" />
         </geometry>
         <material name="">
@@ -145,5 +136,5 @@
         <origin xyz="0 0 0" rpy="0 0 0" />
         <geometry>
-          <mesh filename="package://kortex_description/grippers/gen3_lite_2f/meshes/left_finger_prox_link.STL" />
+          <mesh filename="file://$(find kortex_description)/grippers/gen3_lite_2f/meshes/left_finger_prox_link.STL" />
         </geometry>
       </collision>
@@ -169,5 +160,5 @@
         <origin xyz="0 0 0" rpy="0 0 0" />
         <geometry>
-          <mesh filename="package://kortex_description/grippers/gen3_lite_2f/meshes/left_finger_dist_link.STL" />
+          <mesh filename="file://$(find kortex_description)/grippers/gen3_lite_2f/meshes/left_finger_dist_link.STL" />
         </geometry>
         <material name="">
@@ -178,5 +169,5 @@
         <origin xyz="0 0 0" rpy="0 0 0" />
         <geometry>
-          <mesh filename="package://kortex_description/grippers/gen3_lite_2f/meshes/left_finger_dist_link.STL" />
+          <mesh filename="file://$(find kortex_description)/grippers/gen3_lite_2f/meshes/left_finger_dist_link.STL" />
         </geometry>
       </collision>

File: kortex_description/robots/gen3_lite_gen3_lite_2f.xacro (robot description, xacro)
@@ -3,11 +3,52 @@
     <!-- Arguments -->
     <xacro:arg name="arm" default="gen3_lite" />
-    <!-- Those arguments are ignored for now on Gen3 lite because there is only one supported configuration -->
     <xacro:arg name="dof" default="6" />
     <xacro:arg name="vision" default="false" />
+    <xacro:arg name="robot_ip" default="192.168.1.10" />
+    <xacro:arg name="username" default="admin" />
+    <xacro:arg name="password" default="admin" />
+    <xacro:arg name="port" default="10000" />
+    <xacro:arg name="port_realtime" default="10001" />
+    <xacro:arg name="session_inactivity_timeout_ms" default="60000" />
+    <xacro:arg name="connection_inactivity_timeout_ms" default="2000" />
     <xacro:arg name="gripper" default="gen3_lite_2f" />
-    <xacro:arg name="sim" default="false" />
+    <xacro:arg name="gripper_joint_name" default="right_finger_bottom_joint" />
+    <xacro:arg name="gripper_max_velocity" default="100.0" />
+    <xacro:arg name="gripper_max_force" default="100.0" />
+    <xacro:arg name="sim_gazebo" default="false" />
+    <xacro:arg name="sim_ignition" default="false" />
+    <xacro:arg name="sim_isaac" default="false" />
     <xacro:arg name="prefix" default="" />
+    <xacro:arg name="use_fake_hardware" default="false" />
+    <xacro:arg name="fake_sensor_commands" default="false" />
+    <xacro:arg name="use_internal_bus_gripper_comm" default="true" />
+    <xacro:arg name="use_external_cable" default="false" />
     <xacro:include filename="$(find kortex_description)/robots/kortex_robot.xacro" />
-    <xacro:load_robot arm="$(arg arm)" gripper="$(arg gripper)" dof="$(arg dof)" vision="false" sim="$(arg sim)"  prefix="$(arg prefix)" />
+    <link name="world" />
+    <xacro:load_robot
+        parent="world"
+        arm="$(arg arm)"
+        gripper="$(arg gripper)"
+        gripper_joint_name="$(arg gripper_joint_name)"
+        gripper_max_velocity="$(arg gripper_max_velocity)"
+        gripper_max_force="$(arg gripper_max_force)"
+        dof="$(arg dof)"
+        vision="$(arg vision)"
+        robot_ip="$(arg robot_ip)"
+        username="$(arg username)"
+        password="$(arg password)"
+        port="$(arg port)"
+        port_realtime="$(arg port_realtime)"
+        session_inactivity_timeout_ms="$(arg session_inactivity_timeout_ms)"
+        connection_inactivity_timeout_ms="$(arg connection_inactivity_timeout_ms)"
+        use_internal_bus_gripper_comm="$(arg use_internal_bus_gripper_comm)"
+        prefix="$(arg prefix)"
+        use_fake_hardware="$(arg use_fake_hardware)"
+        fake_sensor_commands="$(arg fake_sensor_commands)"
+        sim_gazebo="$(arg sim_gazebo)"
+        sim_ignition="$(arg sim_ignition)"
+        sim_isaac="$(arg sim_isaac)"
+        use_external_cable="$(arg use_external_cable)" >
+        <origin xyz="0 0 0" rpy="0 0 0" />  <!-- position robot in the world -->
+    </xacro:load_robot>
 </robot>

File: kortex_description/robots/kortex_robot.xacro (robot description, xacro)
@@ -83,6 +83,6 @@
         isaac_joint_commands="${isaac_joint_commands}"
         isaac_joint_states="${isaac_joint_states}"
-        use_internal_bus_gripper_comm="${use_internal_bus_gripper_comm}"
-        com_port="${gripper_com_port}"/>
+        com_port="${gripper_com_port}"
+        use_internal_bus_gripper_comm="${use_internal_bus_gripper_comm}"/>
     </xacro:unless>
   </xacro:macro>
