Commit message: Add a flag to include ros2_control tag

File: kortex_description/arms/gen3_lite/6dof/urdf/gen3_lite_macro.xacro (robot description, xacro)
@@ -28,38 +28,41 @@
     isaac_joint_states:=/isaac_joint_states
     use_external_cable:=false
+    include_ros2_control:=true
     initial_positions:=${dict(joint_1=0.0,joint_2=0.0,joint_3=0.0,joint_4=0.0,joint_5=0.0,joint_6=0.0)}" >
-    <!-- ros2 control include -->
-    <xacro:include filename="$(find kortex_description)/arms/gen3_lite/${dof}dof/urdf/kortex.ros2_control.xacro" />
-    <xacro:if value="${sim_ignition or sim_gazebo}">
-      <xacro:property name="ros2_control_name" value="IgnitionSystem"/>
+    <xacro:if value="${include_ros2_control}">
+      <!-- ros2 control include -->
+      <xacro:include filename="$(find kortex_description)/arms/gen3_lite/${dof}dof/urdf/kortex.ros2_control.xacro" />
+      <xacro:if value="${sim_ignition or sim_gazebo}">
+        <xacro:property name="ros2_control_name" value="IgnitionSystem"/>
+      </xacro:if>
+       <xacro:if value="${use_fake_hardware}">
+        <xacro:property name="ros2_control_name" value="GenericSystem"/>
+      </xacro:if>
+      <xacro:unless value="${use_fake_hardware or sim_ignition or sim_gazebo}">
+        <xacro:property name="ros2_control_name" value="${prefix}KortexMultiInterfaceHardware"/>
+      </xacro:unless>
+      <xacro:kortex_ros2_control
+        name="${ros2_control_name}" prefix="${prefix}"
+        use_fake_hardware="${use_fake_hardware}"
+        fake_sensor_commands="${fake_sensor_commands}"
+        sim_gazebo="${sim_gazebo}"
+        sim_ignition="${sim_ignition}"
+        sim_isaac="${sim_isaac}"
+        isaac_joint_commands="${isaac_joint_commands}"
+        isaac_joint_states="${isaac_joint_states}"
+        tf_prefix=""
+        initial_positions="${initial_positions}"
+        robot_ip="${robot_ip}"
+        username="${username}"
+        password="${password}"
+        port="${port}"
+        port_realtime="${port_realtime}"
+        session_inactivity_timeout_ms="${session_inactivity_timeout_ms}"
+        connection_inactivity_timeout_ms="${connection_inactivity_timeout_ms}"
+        use_internal_bus_gripper_comm="${use_internal_bus_gripper_comm}"
+        gripper_max_velocity="${gripper_max_velocity}"
+        gripper_max_force="${gripper_max_force}"
+        gripper_joint_name="${gripper_joint_name}"/>
     </xacro:if>
-     <xacro:if value="${use_fake_hardware}">
-      <xacro:property name="ros2_control_name" value="GenericSystem"/>
-    </xacro:if>
-    <xacro:unless value="${use_fake_hardware or sim_ignition or sim_gazebo}">
-      <xacro:property name="ros2_control_name" value="${prefix}KortexMultiInterfaceHardware"/>
-    </xacro:unless>
-    <xacro:kortex_ros2_control
-      name="${ros2_control_name}" prefix="${prefix}"
-      use_fake_hardware="${use_fake_hardware}"
-      fake_sensor_commands="${fake_sensor_commands}"
-      sim_gazebo="${sim_gazebo}"
-      sim_ignition="${sim_ignition}"
-      sim_isaac="${sim_isaac}"
-      isaac_joint_commands="${isaac_joint_commands}"
-      isaac_joint_states="${isaac_joint_states}"
-      tf_prefix=""
-      initial_positions="${initial_positions}"
-      robot_ip="${robot_ip}"
-      username="${username}"
-      password="${password}"
-      port="${port}"
-      port_realtime="${port_realtime}"
-      session_inactivity_timeout_ms="${session_inactivity_timeout_ms}"
-      connection_inactivity_timeout_ms="${connection_inactivity_timeout_ms}"
-      use_internal_bus_gripper_comm="${use_internal_bus_gripper_comm}"
-      gripper_max_velocity="${gripper_max_velocity}"
-      gripper_max_force="${gripper_max_force}"
-      gripper_joint_name="${gripper_joint_name}"/>
     <joint name="${prefix}base_joint" type="fixed">
       <xacro:insert_block name="origin" />

File: kortex_description/robots/kortex_robot.xacro (robot description, xacro)
@@ -26,4 +26,5 @@
     isaac_joint_states:=/isaac_joint_states
     use_external_cable:=false
+    include_ros2_control:=true
     initial_positions:=${dict(joint_1=0.0,joint_2=0.0,joint_3=0.0,joint_4=0.0,joint_5=0.0,joint_6=0.0,joint_7=0.0)}
     gripper_max_velocity:=100.0
@@ -57,4 +58,5 @@
       gripper_max_force="${gripper_max_force}"
       use_external_cable="${use_external_cable}"
+      include_ros2_control="${include_ros2_control}"
       initial_positions="${initial_positions}">
       <xacro:insert_block name="origin" />
@@ -83,4 +85,5 @@
         isaac_joint_commands="${isaac_joint_commands}"
         isaac_joint_states="${isaac_joint_states}"
+        include_ros2_control="${include_ros2_control}"
         com_port="${gripper_com_port}"
         use_internal_bus_gripper_comm="${use_internal_bus_gripper_comm}"/>

Commit message: Rectified the entire system (Moveit with RL and Sim) for Gen3_Lite

File: kortex_description/arms/gen3_lite/6dof/urdf/gen3_lite_macro.xacro (robot description, xacro)
@@ -28,16 +28,26 @@
     isaac_joint_states:=/isaac_joint_states
     use_external_cable:=false
-    initial_positions:=${dict(joint_1=0.0,joint_2=0.0,joint_3=0.0,joint_4=0.0,joint_5=0.0,joint_6=0.0)}" >
+    initial_positions:=${dict(joint_1=0.0,joint_2=0.0,joint_3=0.0,joint_4=0.0,joint_5=0.0,joint_6=0.0)}
+    moveit_active" >
     <!-- ros2 control include -->
     <xacro:include filename="$(find kortex_description)/arms/gen3_lite/${dof}dof/urdf/kortex.ros2_control.xacro" />
     <xacro:if value="${sim_ignition or sim_gazebo}">
-      <xacro:property name="ros2_control_name" value="IgnitionSystem"/>
+      <xacro:unless value="${moveit_active}">
+        <xacro:property name="ros2_control_name" value="IgnitionSystem"/>
+      </xacro:unless>
     </xacro:if>
      <xacro:if value="${use_fake_hardware}">
-      <xacro:property name="ros2_control_name" value="GenericSystem"/>
+      <xacro:unless value="${moveit_active}">
+        <xacro:property name="ros2_control_name" value="GenericSystem"/>
+      </xacro:unless>
     </xacro:if>
     <xacro:unless value="${use_fake_hardware or sim_ignition or sim_gazebo}">
+      <xacro:unless value="${moveit_active}">
+        <xacro:property name="ros2_control_name" value="${prefix}KortexMultiInterfaceHardware"/>
+      </xacro:unless>
+    </xacro:unless>
+    <xacro:if value="${moveit_active}">
       <xacro:property name="ros2_control_name" value="${prefix}KortexMultiInterfaceHardware"/>
-    </xacro:unless>
+    </xacro:if>
     <xacro:kortex_ros2_control
       name="${ros2_control_name}" prefix="${prefix}"
@@ -61,5 +71,6 @@
       gripper_max_velocity="${gripper_max_velocity}"
       gripper_max_force="${gripper_max_force}"
-      gripper_joint_name="${gripper_joint_name}"/>
+      gripper_joint_name="${gripper_joint_name}"
+      moveit_active="${moveit_active}"/>
     <joint name="${prefix}base_joint" type="fixed">
       <xacro:insert_block name="origin" />

File: kortex_description/arms/gen3_lite/6dof/urdf/kortex.ros2_control.xacro (robot description, xacro)
@@ -23,24 +23,50 @@
     gripper_joint_name
     gripper_max_velocity:=100.0
-    gripper_max_force:=100.0">
+    gripper_max_force:=100.0
+    moveit_active">
     <ros2_control name="${name}" type="system">
       <hardware>
         <xacro:if value="${sim_gazebo}">
-          <plugin>gazebo_ros2_control/GazeboSystem</plugin>
+          <xacro:unless value="${moveit_active}">
+            <plugin>gazebo_ros2_control/GazeboSystem</plugin>
+          </xacro:unless>
         </xacro:if>
         <xacro:if value="${sim_ignition}">
-          <plugin>ign_ros2_control/IgnitionSystem</plugin>
+          <xacro:unless value="${moveit_active}">
+            <plugin>ign_ros2_control/IgnitionSystem</plugin>
+          </xacro:unless>
         </xacro:if>
         <xacro:if value="${sim_isaac}">
-          <plugin>topic_based_ros2_control/TopicBasedSystem</plugin>
-          <param name="joint_commands_topic">${isaac_joint_commands}</param>
-          <param name="joint_states_topic">${isaac_joint_states}</param>
+          <xacro:unless value="${moveit_active}">
+            <plugin>topic_based_ros2_control/TopicBasedSystem</plugin>
+            <param name="joint_commands_topic">${isaac_joint_commands}</param>
+            <param name="joint_states_topic">${isaac_joint_states}</param>
+          </xacro:unless>
         </xacro:if>
         <xacro:if value="${use_fake_hardware}">
-          <plugin>mock_components/GenericSystem</plugin>
-          <param name="fake_sensor_commands">${fake_sensor_commands}</param>
-          <param name="state_following_offset">0.0</param>
+          <xacro:unless value="${moveit_active}">
+            <plugin>mock_components/GenericSystem</plugin>
+            <param name="fake_sensor_commands">${fake_sensor_commands}</param>
+            <param name="state_following_offset">0.0</param>
+          </xacro:unless>
         </xacro:if>
         <xacro:unless value="${use_fake_hardware or sim_gazebo or sim_ignition or sim_isaac}">
+          <xacro:unless value="${moveit_active}">
+            <plugin>kortex_driver/KortexMultiInterfaceHardware</plugin>
+            <param name="robot_ip">${robot_ip}</param>
+            <param name="username">${username}</param>
+            <param name="password">${password}</param>
+            <param name="port">${port}</param>
+            <param name="port_realtime">${port_realtime}</param>
+            <param name="session_inactivity_timeout_ms">${session_inactivity_timeout_ms}</param>
+            <param name="connection_inactivity_timeout_ms">${connection_inactivity_timeout_ms}</param>
+            <param name="tf_prefix">"${tf_prefix}"</param>
+            <param name="use_internal_bus_gripper_comm">${use_internal_bus_gripper_comm}</param>
+            <param name="gripper_joint_name">${gripper_joint_name}</param>
+            <param name="gripper_max_velocity">${gripper_max_velocity}</param>
+            <param name="gripper_max_force">${gripper_max_force}</param>
+          </xacro:unless>
+        </xacro:unless>
+        <xacro:if value="${moveit_active}">
           <plugin>kortex_driver/KortexMultiInterfaceHardware</plugin>
           <param name="robot_ip">${robot_ip}</param>
@@ -56,5 +82,5 @@
           <param name="gripper_max_velocity">${gripper_max_velocity}</param>
           <param name="gripper_max_force">${gripper_max_force}</param>
-        </xacro:unless>
+        </xacro:if>
       </hardware>
       <joint name="${prefix}joint_1">
@@ -125,4 +151,13 @@
       </joint>
       <xacro:unless value="${use_fake_hardware or sim_isaac or sim_ignition}">
+        <xacro:unless value="${moveit_active}">
+          <joint name="${prefix}right_finger_bottom_joint">
+            <command_interface name="position"/>
+            <state_interface name="position"/>
+            <state_interface name="velocity"/>
+          </joint>
+        </xacro:unless>
+      </xacro:unless>
+      <xacro:if value="${moveit_active}">
         <joint name="${prefix}right_finger_bottom_joint">
           <command_interface name="position"/>
@@ -130,5 +165,5 @@
           <state_interface name="velocity"/>
         </joint>
-      </xacro:unless>
+      </xacro:if>
     </ros2_control>
   </xacro:macro>
