Commit message: Modified the Gen3_Lite related description and ros2_control  files

File: kortex_description/arms/gen3_lite/6dof/urdf/gen3_lite_macro.xacro (robot description, xacro)
@@ -28,16 +28,26 @@
     isaac_joint_states:=/isaac_joint_states
     use_external_cable:=false
-    initial_positions:=${dict(joint_1=0.0,joint_2=0.0,joint_3=0.0,joint_4=0.0,joint_5=0.0,joint_6=0.0)}" >
+    initial_positions:=${dict(joint_1=0.0,joint_2=0.0,joint_3=0.0,joint_4=0.0,joint_5=0.0,joint_6=0.0)}
+    moveit_active" >
     <!-- ros2 control include -->
     <xacro:include filename="$(find kortex_description)/arms/gen3_lite/${dof}dof/urdf/kortex.ros2_control.xacro" />
     <xacro:if value="${sim_ignition or sim_gazebo}">
-      <xacro:property name="ros2_control_name" value="IgnitionSystem"/>
+      <xacro:unless value="${moveit_active}">
+        <xacro:property name="ros2_control_name" value="IgnitionSystem"/>
+      </xacro:unless>
     </xacro:if>
      <xacro:if value="${use_fake_hardware}">
-      <xacro:property name="ros2_control_name" value="GenericSystem"/>
+      <xacro:unless value="${moveit_active}">
+        <xacro:property name="ros2_control_name" value="GenericSystem"/>
+      </xacro:unless>
     </xacro:if>
     <xacro:unless value="${use_fake_hardware or sim_ignition or sim_gazebo}">
+      <xacro:unless value="${moveit_active}">
+        <xacro:property name="ros2_control_name" value="${prefix}KortexMultiInterfaceHardware"/>
+      </xacro:unless>
+    </xacro:unless>
+    <xacro:if value="${moveit_active}">
       <xacro:property name="ros2_control_name" value="${prefix}KortexMultiInterfaceHardware"/>
-    </xacro:unless>
+    </xacro:if>
     <xacro:kortex_ros2_control
       name="${ros2_control_name}" prefix="${prefix}"
@@ -61,5 +71,6 @@
       gripper_max_velocity="${gripper_max_velocity}"
       gripper_max_force="${gripper_max_force}"
-      gripper_joint_name="${gripper_joint_name}"/>
+      gripper_joint_name="${gripper_joint_name}"
+      moveit_active="${moveit_active}"/>
     <joint name="${prefix}base_joint" type="fixed">
       <xacro:insert_block name="origin" />

File: kortex_description/arms/gen3_lite/6dof/urdf/kortex.ros2_control.xacro (robot description, xacro)
@@ -23,24 +23,50 @@
     gripper_joint_name
     gripper_max_velocity:=100.0
-    gripper_max_force:=100.0">
+    gripper_max_force:=100.0
+    moveit_active">
     <ros2_control name="${name}" type="system">
       <hardware>
         <xacro:if value="${sim_gazebo}">
-          <plugin>gazebo_ros2_control/GazeboSystem</plugin>
+          <xacro:unless value="${moveit_active}">
+            <plugin>gazebo_ros2_control/GazeboSystem</plugin>
+          </xacro:unless>
         </xacro:if>
         <xacro:if value="${sim_ignition}">
-          <plugin>ign_ros2_control/IgnitionSystem</plugin>
+          <xacro:unless value="${moveit_active}">
+            <plugin>ign_ros2_control/IgnitionSystem</plugin>
+          </xacro:unless>
         </xacro:if>
         <xacro:if value="${sim_isaac}">
-          <plugin>topic_based_ros2_control/TopicBasedSystem</plugin>
-          <param name="joint_commands_topic">${isaac_joint_commands}</param>
-          <param name="joint_states_topic">${isaac_joint_states}</param>
+          <xacro:unless value="${moveit_active}">
+            <plugin>topic_based_ros2_control/TopicBasedSystem</plugin>
+            <param name="joint_commands_topic">${isaac_joint_commands}</param>
+            <param name="joint_states_topic">${isaac_joint_states}</param>
+          </xacro:unless>
         </xacro:if>
         <xacro:if value="${use_fake_hardware}">
-          <plugin>mock_components/GenericSystem</plugin>
-          <param name="fake_sensor_commands">${fake_sensor_commands}</param>
-          <param name="state_following_offset">0.0</param>
+          <xacro:unless value="${moveit_active}">
+            <plugin>mock_components/GenericSystem</plugin>
+            <param name="fake_sensor_commands">${fake_sensor_commands}</param>
+            <param name="state_following_offset">0.0</param>
+          </xacro:unless>
         </xacro:if>
         <xacro:unless value="${use_fake_hardware or sim_gazebo or sim_ignition or sim_isaac}">
+          <xacro:unless value="${moveit_active}">
+            <plugin>kortex_driver/KortexMultiInterfaceHardware</plugin>
+            <param name="robot_ip">${robot_ip}</param>
+            <param name="username">${username}</param>
+            <param name="password">${password}</param>
+            <param name="port">${port}</param>
+            <param name="port_realtime">${port_realtime}</param>
+            <param name="session_inactivity_timeout_ms">${session_inactivity_timeout_ms}</param>
+            <param name="connection_inactivity_timeout_ms">${connection_inactivity_timeout_ms}</param>
+            <param name="tf_prefix">"${tf_prefix}"</param>
+            <param name="use_internal_bus_gripper_comm">${use_internal_bus_gripper_comm}</param>
+            <param name="gripper_joint_name">${gripper_joint_name}</param>
+            <param name="gripper_max_velocity">${gripper_max_velocity}</param>
+            <param name="gripper_max_force">${gripper_max_force}</param>
+          </xacro:unless>
+        </xacro:unless>
+        <xacro:if value="${moveit_active}">
           <plugin>kortex_driver/KortexMultiInterfaceHardware</plugin>
           <param name="robot_ip">${robot_ip}</param>
@@ -56,5 +82,5 @@
           <param name="gripper_max_velocity">${gripper_max_velocity}</param>
           <param name="gripper_max_force">${gripper_max_force}</param>
-        </xacro:unless>
+        </xacro:if>
       </hardware>
       <joint name="${prefix}joint_1">
@@ -124,9 +150,20 @@
         <state_interface name="effort"/>
       </joint>
-      <joint name="${prefix}right_finger_bottom_joint">
-        <command_interface name="position"/>
-        <state_interface name="position"/>
-        <state_interface name="velocity"/>
-      </joint>
+      <xacro:unless value="${use_fake_hardware or sim_isaac or sim_ignition}">
+        <xacro:unless value="${moveit_active}">
+          <joint name="${prefix}right_finger_bottom_joint">
+            <command_interface name="position"/>
+            <state_interface name="position"/>
+            <state_interface name="velocity"/>
+          </joint>
+        </xacro:unless>
+      </xacro:unless>
+      <xacro:if value="${moveit_active}">
+        <joint name="${prefix}right_finger_bottom_joint">
+          <command_interface name="position"/>
+          <state_interface name="position"/>
+          <state_interface name="velocity"/>
+        </joint>
+      </xacro:if>
     </ros2_control>
   </xacro:macro>
