Commit message: Modified the Gen3_Lite related description and ros2_control  files

File: kortex_description/grippers/gen3_lite_2f/urdf/gen3_lite_2f_macro.xacro (robot description, xacro)
@@ -11,21 +11,393 @@
     isaac_joint_commands:=/isaac_joint_commands
     isaac_joint_states:=/isaac_joint_states
-    use_internal_bus_gripper_comm:=true">
-    <!-- Tool frame used by the arm -->
-    <link name="${prefix}tool_frame"/>
-    <joint name="${prefix}tool_frame_joint" type="fixed">
+    use_internal_bus_gripper_comm:=true
+    moveit_active">
+  <xacro:if value="${use_fake_hardware or sim_isaac or sim_ignition}">
+    <xacro:unless value="${moveit_active}">
+    <!-- ros2 control include -->
+      <xacro:include filename="$(find kortex_description)/grippers/gen3_lite_2f/urdf/gen3_lite_2f.ros2_control.xacro" />
+      <xacro:if value="${sim_ignition or sim_gazebo}">
+        <xacro:property name="ros2_control_name" value="IgnitionSystem"/>
+      </xacro:if>
+      <xacro:if value="${use_fake_hardware}">
+        <xacro:property name="ros2_control_name" value="GenericSystem"/>
+      </xacro:if>
+      <xacro:unless value="${use_fake_hardware or sim_ignition or sim_gazebo}">
+        <xacro:property name="ros2_control_name" value="${prefix}KortexMultiInterfaceHardware"/>
+      </xacro:unless>
+      <xacro:gripper_ros2_control
+        prefix="${prefix}"
+        use_fake_hardware="${use_fake_hardware}"
+        fake_sensor_commands="${fake_sensor_commands}"
+        sim_ignition="${sim_ignition}"
+        sim_isaac="${sim_isaac}"
+        isaac_joint_commands="${isaac_joint_commands}"
+        isaac_joint_states="${isaac_joint_states}"
+        tf_prefix=""/>
+  <!-- Tool frame used by the arm -->
+      <link name="${prefix}tool_frame"/>
+      <joint name="${prefix}tool_frame_joint" type="fixed">
+          <origin xyz="0 0 0.130" rpy="0 0 1.57079632679" />
+          <parent link="${parent}" />
+          <child link="${prefix}tool_frame" />
+          <axis xyz="0 0 0" />
+      </joint>
+      <!-- Gripper description -->
+      <joint name="${prefix}gripper_base_joint" type="fixed">
+        <origin xyz="0 0 0" rpy="0 0 0" />
+        <parent link="${parent}" />
+        <child link="${prefix}gripper_base_link" />
+        <axis xyz="0 0 0" />
+      </joint>
+      <link name="${prefix}gripper_base_link">
+        <inertial>
+          <origin xyz="4.03E-06 1.08E-05 0.041397" rpy="0 0 0" />
+          <mass value="0.1395" />
+          <inertia ixx="0.00011614" ixy="1E-08" ixz="4E-08" iyy="0.00010327" iyz="0" izz="9.707E-05" />
+        </inertial>
+        <visual>
+          <origin xyz="0 0 0" rpy="0 0 0" />
+          <geometry>
+            <mesh filename="file://$(find kortex_description)/grippers/gen3_lite_2f/meshes/gripper_base_link.STL" />
+          </geometry>
+          <material name="">
+            <color rgba="0.803 0.824 0.820 1" />
+          </material>
+        </visual>
+        <collision>
+          <origin xyz="0 0 0" rpy="0 0 0" />
+          <geometry>
+            <mesh filename="file://$(find kortex_description)/grippers/gen3_lite_2f/meshes/gripper_base_link.STL" />
+          </geometry>
+        </collision>
+      </link>
+      <gazebo reference="${prefix}gripper_base_link">
+        <material>Kortex/Gray</material>
+      </gazebo>
+      <link name="${prefix}right_finger_prox_link">
+      <inertial>
+        <origin xyz="0.020257 0.0063483 6.991E-05" rpy="0 0 0" />
+        <mass value="0.018385" />
+        <inertia ixx="2.29E-06" ixy="1.43E-06" ixz="0" iyy="4.56E-06" iyz="0" izz="4.77E-06" />
+      </inertial>
+      <visual>
+        <origin xyz="0 0 0" rpy="0 0 0" />
+        <geometry>
+          <mesh filename="file://$(find kortex_description)/grippers/gen3_lite_2f/meshes/right_finger_prox_link.STL" />
+        </geometry>
+        <material name="">
+            <color rgba="0.803 0.824 0.820 1" />
+        </material>
+      </visual>
+      <collision>
+        <origin xyz="0 0 0" rpy="0 0 0" />
+        <geometry>
+          <mesh filename="file://$(find kortex_description)/grippers/gen3_lite_2f/meshes/right_finger_prox_link.STL" />
+        </geometry>
+      </collision>
+      </link>
+      <gazebo reference="${prefix}right_finger_prox_link">
+        <material>Kortex/Gray</material>
+      </gazebo>
+      <joint name="${prefix}right_finger_bottom_joint" type="revolute">
+        <origin xyz="0 -0.030501 0.070003" rpy="0 1.5708 0" />
+        <parent link="${prefix}gripper_base_link" />
+        <child link="${prefix}right_finger_prox_link" />
+        <axis xyz="0 0 1" />
+        <limit lower="-0.09" upper="0.96" effort="10" velocity="0.6" />
+        <dynamics damping="0.1" friction="1"/>
+      </joint>
+      <link name="${prefix}right_finger_dist_link">
+        <inertial>
+          <origin xyz="0.018488 0.0011091 0" rpy="0 0 0" />
+          <mass value="0.010748" />
+          <inertia ixx="6.3E-07" ixy="3.2E-07" ixz="0" iyy="1.83E-06" iyz="0" izz="1.61E-06" />
+        </inertial>
+        <visual>
+          <origin xyz="0 0 0" rpy="0 0 0" />
+          <geometry>
+            <mesh filename="file://$(find kortex_description)/grippers/gen3_lite_2f/meshes/right_finger_dist_link.STL" />
+          </geometry>
+          <material name="">
+            <color rgba="0 0.055 0.525 1" />
+          </material>
+        </visual>
+        <collision>
+          <origin xyz="0 0 0" rpy="0 0 0" />
+          <geometry>
+            <mesh filename="file://$(find kortex_description)/grippers/gen3_lite_2f/meshes/right_finger_dist_link.STL" />
+          </geometry>
+        </collision>
+      </link>
+      <gazebo reference="${prefix}right_finger_dist_link">
+        <material>Kortex/Blue</material>
+      </gazebo>
+      <joint name="${prefix}right_finger_tip_joint" type="revolute">
+        <origin xyz="-0.045636 0.020423 0" rpy="0 0 0" />
+        <parent link="${prefix}right_finger_prox_link" />
+        <child link="${prefix}right_finger_dist_link" />
+        <axis xyz="0 0 1" />
+        <limit lower="-0.50" upper="0.21" effort="1000" velocity="1000" /> <!--limit lower="-1.03" upper="0.21" effort="1000" velocity="1000" /-->
+      </joint>
+      <link name="${prefix}left_finger_prox_link">
+        <inertial>
+          <origin xyz="0.020257 0.0063483 6.99E-05" rpy="0 0 0" />
+          <mass value="0.018385" />
+          <inertia ixx="2.29E-06" ixy="1.43E-06" ixz="0" iyy="4.56E-06" iyz="0" izz="4.77E-06" />
+        </inertial>
+        <visual>
+          <origin xyz="0 0 0" rpy="0 0 0" />
+          <geometry>
+            <mesh filename="file://$(find kortex_description)/grippers/gen3_lite_2f/meshes/left_finger_prox_link.STL" />
+          </geometry>
+          <material name="">
+            <color rgba="0.803 0.824 0.820 1" />
+          </material>
+        </visual>
+        <collision>
+          <origin xyz="0 0 0" rpy="0 0 0" />
+          <geometry>
+            <mesh filename="file://$(find kortex_description)/grippers/gen3_lite_2f/meshes/left_finger_prox_link.STL" />
+          </geometry>
+        </collision>
+      </link>
+      <gazebo reference="${prefix}left_finger_prox_link">
+        <material>Kortex/Gray</material>
+      </gazebo>
+      <joint name="${prefix}left_finger_bottom_joint" type="revolute">
+        <origin xyz="0 0.0305 0.070003" rpy="0 1.5708 0" />
+        <parent link="${prefix}gripper_base_link" />
+        <child link="${prefix}left_finger_prox_link" />
+        <axis xyz="0 0 1" />
+        <limit lower="-0.96" upper="0.09" effort="10" velocity="0.6" />
+        <dynamics damping="0.1" friction="1"/>
+      </joint>
+      <link name="${prefix}left_finger_dist_link">
+        <inertial>
+          <origin xyz="-0.018488 0.0011091 0" rpy="0 0 0" />
+          <mass value="0.010748" />
+          <inertia ixx="6.3E-07" ixy="3.2E-07" ixz="0" iyy="1.83E-06" iyz="0" izz="1.61E-06" />
+        </inertial>
+        <visual>
+          <origin xyz="0 0 0" rpy="0 0 0" />
+          <geometry>
+            <mesh filename="file://$(find kortex_description)/grippers/gen3_lite_2f/meshes/left_finger_dist_link.STL" />
+          </geometry>
+          <material name="">
+            <color rgba="0 0.055 0.525 1" />
+          </material>
+        </visual>
+        <collision>
+          <origin xyz="0 0 0" rpy="0 0 0" />
+          <geometry>
+            <mesh filename="file://$(find kortex_description)/grippers/gen3_lite_2f/meshes/left_finger_dist_link.STL" />
+          </geometry>
+        </collision>
+      </link>
+      <gazebo reference="${prefix}left_finger_dist_link">
+        <material>Kortex/Blue</material>
+      </gazebo>
+      <joint name="${prefix}left_finger_tip_joint" type="revolute">
+        <origin xyz="-0.045636 -0.020423 6.9901E-05" rpy="0 0 0" />
+        <parent link="${prefix}left_finger_prox_link" />
+        <child link="${prefix}left_finger_dist_link" />
+        <axis xyz="0 0 -1" />
+        <limit lower="-0.50" upper="0.21" effort="1000" velocity="1000" /> <!--limit lower="-1.03" upper="0.21" effort="1000" velocity="1000" /-->
+      </joint>
+    </xacro:unless>
+  </xacro:if>
+  <xacro:unless value="${use_fake_hardware or sim_isaac or sim_ignition}">
+    <xacro:unless value="${moveit_active}">
+        <!-- Tool frame used by the arm -->
+      <link name="${prefix}tool_frame"/>
+      <joint name="${prefix}tool_frame_joint" type="fixed">
+          <origin xyz="0 0 0.130" rpy="0 0 1.57079632679" />
+          <parent link="${parent}" />
+          <child link="${prefix}tool_frame" />
+          <axis xyz="0 0 0" />
+      </joint>
+      <!-- Gripper description -->
+      <joint name="${prefix}gripper_base_joint" type="fixed">
+        <origin xyz="0 0 0" rpy="0 0 0" />
+        <parent link="${parent}" />
+        <child link="${prefix}gripper_base_link" />
+        <axis xyz="0 0 0" />
+      </joint>
+      <link name="${prefix}gripper_base_link">
+        <inertial>
+          <origin xyz="4.03E-06 1.08E-05 0.041397" rpy="0 0 0" />
+          <mass value="0.1395" />
+          <inertia ixx="0.00011614" ixy="1E-08" ixz="4E-08" iyy="0.00010327" iyz="0" izz="9.707E-05" />
+        </inertial>
+        <visual>
+          <origin xyz="0 0 0" rpy="0 0 0" />
+          <geometry>
+            <mesh filename="file://$(find kortex_description)/grippers/gen3_lite_2f/meshes/gripper_base_link.STL" />
+          </geometry>
+          <material name="">
+            <color rgba="0.803 0.824 0.820 1" />
+          </material>
+        </visual>
+        <collision>
+          <origin xyz="0 0 0" rpy="0 0 0" />
+          <geometry>
+            <mesh filename="file://$(find kortex_description)/grippers/gen3_lite_2f/meshes/gripper_base_link.STL" />
+          </geometry>
+        </collision>
+      </link>
+      <gazebo reference="${prefix}gripper_base_link">
+        <material>Kortex/Gray</material>
+      </gazebo>
+      <link name="${prefix}right_finger_prox_link">
+      <inertial>
+        <origin xyz="0.020257 0.0063483 6.991E-05" rpy="0 0 0" />
+        <mass value="0.018385" />
+        <inertia ixx="2.29E-06" ixy="1.43E-06" ixz="0" iyy="4.56E-06" iyz="0" izz="4.77E-06" />
+      </inertial>
+      <visual>
+        <origin xyz="0 0 0" rpy="0 0 0" />
+        <geometry>
+          <mesh filename="file://$(find kortex_description)/grippers/gen3_lite_2f/meshes/right_finger_prox_link.STL" />
+        </geometry>
+        <material name="">
+            <color rgba="0.803 0.824 0.820 1" />
+        </material>
+      </visual>
+      <collision>
+        <origin xyz="0 0 0" rpy="0 0 0" />
+        <geometry>
+          <mesh filename="file://$(find kortex_description)/grippers/gen3_lite_2f/meshes/right_finger_prox_link.STL" />
+        </geometry>
+      </collision>
+      </link>
+      <gazebo reference="${prefix}right_finger_prox_link">
+        <material>Kortex/Gray</material>
+      </gazebo>
+      <!-- TODO(MarqRazz) look into why the joint and limits needed to be flipped and modified -->
+      <joint name="${prefix}right_finger_bottom_joint" type="revolute">
+        <origin xyz="0 -0.030501 0.070003" rpy="1.571 0.611 1.571" />
+        <parent link="${prefix}gripper_base_link" />
+        <child link="${prefix}right_finger_prox_link" />
+        <axis xyz="0 0 -1" />
+        <limit lower="0.0" upper="0.85" effort="50" velocity="0.6" />
+      </joint>
+      <link name="${prefix}right_finger_dist_link">
+        <inertial>
+          <origin xyz="0.018488 0.0011091 0" rpy="0 0 0" />
+          <mass value="0.010748" />
+          <inertia ixx="6.3E-07" ixy="3.2E-07" ixz="0" iyy="1.83E-06" iyz="0" izz="1.61E-06" />
+        </inertial>
+        <visual>
+          <origin xyz="0 0 0" rpy="0 0 0" />
+          <geometry>
+            <mesh filename="file://$(find kortex_description)/grippers/gen3_lite_2f/meshes/right_finger_dist_link.STL" />
+          </geometry>
+          <material name="">
+            <color rgba="0 0.055 0.525 1" />
+          </material>
+        </visual>
+        <collision>
+          <origin xyz="0 0 0" rpy="0 0 0" />
+          <geometry>
+            <mesh filename="file://$(find kortex_description)/grippers/gen3_lite_2f/meshes/right_finger_dist_link.STL" />
+          </geometry>
+        </collision>
+      </link>
+      <gazebo reference="${prefix}right_finger_dist_link">
+        <material>Kortex/Blue</material>
+      </gazebo>
+      <joint name="${prefix}right_finger_tip_joint" type="revolute">
+        <origin xyz="-0.045636 0.020423 0" rpy="0 0 0" />
+        <parent link="${prefix}right_finger_prox_link" />
+        <child link="${prefix}right_finger_dist_link" />
+        <axis xyz="0 0 1" />
+        <limit lower="-0.50" upper="0.21" effort="1000" velocity="1000" /> <!--limit lower="-1.03" upper="0.21" effort="1000" velocity="1000" /-->
+        <mimic joint="${prefix}right_finger_bottom_joint" multiplier="-0.276" offset="-0.1" />
+      </joint>
+      <link name="${prefix}left_finger_prox_link">
+        <inertial>
+          <origin xyz="0.020257 0.0063483 6.99E-05" rpy="0 0 0" />
+          <mass value="0.018385" />
+          <inertia ixx="2.29E-06" ixy="1.43E-06" ixz="0" iyy="4.56E-06" iyz="0" izz="4.77E-06" />
+        </inertial>
+        <visual>
+          <origin xyz="0 0 0" rpy="0 0 0" />
+          <geometry>
+            <mesh filename="file://$(find kortex_description)/grippers/gen3_lite_2f/meshes/left_finger_prox_link.STL" />
+          </geometry>
+          <material name="">
+            <color rgba="0.803 0.824 0.820 1" />
+          </material>
+        </visual>
+        <collision>
+          <origin xyz="0 0 0" rpy="0 0 0" />
+          <geometry>
+            <mesh filename="file://$(find kortex_description)/grippers/gen3_lite_2f/meshes/left_finger_prox_link.STL" />
+          </geometry>
+        </collision>
+      </link>
+      <gazebo reference="${prefix}left_finger_prox_link">
+        <material>Kortex/Gray</material>
+      </gazebo>
+      <joint name="${prefix}left_finger_bottom_joint" type="revolute">
+        <origin xyz="0 0.0305 0.070003" rpy="-1.571 0.611 -1.571" />
+        <parent link="${prefix}gripper_base_link" />
+        <child link="${prefix}left_finger_prox_link" />
+        <axis xyz="0 0 1" />
+        <limit lower="0.0" upper="0.85" effort="1000" velocity="1000" />
+        <mimic joint="${prefix}right_finger_bottom_joint" multiplier="1.0" offset="0.0" />
+      </joint>
+      <link name="${prefix}left_finger_dist_link">
+        <inertial>
+          <origin xyz="-0.018488 0.0011091 0" rpy="0 0 0" />
+          <mass value="0.010748" />
+          <inertia ixx="6.3E-07" ixy="3.2E-07" ixz="0" iyy="1.83E-06" iyz="0" izz="1.61E-06" />
+        </inertial>
+        <visual>
+          <origin xyz="0 0 0" rpy="0 0 0" />
+          <geometry>
+            <mesh filename="file://$(find kortex_description)/grippers/gen3_lite_2f/meshes/left_finger_dist_link.STL" />
+          </geometry>
+          <material name="">
+            <color rgba="0 0.055 0.525 1" />
+          </material>
+        </visual>
+        <collision>
+          <origin xyz="0 0 0" rpy="0 0 0" />
+          <geometry>
+            <mesh filename="file://$(find kortex_description)/grippers/gen3_lite_2f/meshes/left_finger_dist_link.STL" />
+          </geometry>
+        </collision>
+      </link>
+      <gazebo reference="${prefix}left_finger_dist_link">
+        <material>Kortex/Blue</material>
+      </gazebo>
+      <joint name="${prefix}left_finger_tip_joint" type="revolute">
+        <origin xyz="-0.045636 -0.020423 6.9901E-05" rpy="0 0 0" />
+        <parent link="${prefix}left_finger_prox_link" />
+        <child link="${prefix}left_finger_dist_link" />
+        <axis xyz="0 0 -1" />
+        <limit lower="-0.50" upper="0.21" effort="1000" velocity="1000" /> <!--limit lower="-1.03" upper="0.21" effort="1000" velocity="1000" /-->
+        <mimic joint="${prefix}right_finger_bottom_joint" multiplier="-0.276" offset="-0.1" />
+      </joint>
+    </xacro:unless>
+  </xacro:unless>
+  <xacro:if value="${moveit_active}">
+  <!-- Tool frame used by the arm -->
+    <link name="tool_frame"/>
+    <joint name="tool_frame_joint" type="fixed">
         <origin xyz="0 0 0.130" rpy="0 0 1.57079632679" />
-        <parent link="${parent}" />
-        <child link="${prefix}tool_frame" />
+        <parent link="dummy_link" />
+        <child link="tool_frame" />
         <axis xyz="0 0 0" />
     </joint>
     <!-- Gripper description -->
-    <joint name="${prefix}gripper_base_joint" type="fixed">
+    <joint name="gripper_base_joint" type="fixed">
       <origin xyz="0 0 0" rpy="0 0 0" />
-      <parent link="${parent}" />
-      <child link="${prefix}gripper_base_link" />
+      <parent link="dummy_link" />
+      <child link="gripper_base_link" />
       <axis xyz="0 0 0" />
     </joint>
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