Commit message: Rectified the Gen3_Lite gripper motion in Gazebo Ignition Fortress (Problem not rectified in Gazebo classic)

File: kortex_description/arms/gen3_lite/6dof/urdf/kortex.ros2_control.xacro (robot description, xacro)
@@ -124,4 +124,5 @@
         <state_interface name="effort"/>
       </joint>
+      <!--
       <joint name="${prefix}right_finger_bottom_joint">
         <command_interface name="position"/>
@@ -129,4 +130,5 @@
         <state_interface name="velocity"/>
       </joint>
+      -->
     </ros2_control>
   </xacro:macro>

File: kortex_description/grippers/gen3_lite_2f/urdf/gen3_lite_2f.ros2_control.xacro (robot description, xacro)
@@ -77,5 +77,5 @@
                 <joint name="${prefix}left_finger_bottom_joint">
                     <param name="mimic">${prefix}right_finger_bottom_joint</param>
-                    <param name="multiplier">1</param>
+                    <param name="multiplier">-1</param>
                     <xacro:unless value="${sim_ignition}">
                         <command_interface name="position"/>

File: kortex_description/grippers/gen3_lite_2f/urdf/gen3_lite_2f_macro.xacro (robot description, xacro)
@@ -12,5 +12,25 @@
     isaac_joint_states:=/isaac_joint_states
     use_internal_bus_gripper_comm:=true">
-    <!-- Tool frame used by the arm -->
+  <!-- ros2 control include -->
+    <xacro:include filename="$(find kortex_description)/grippers/gen3_lite_2f/urdf/gen3_lite_2f.ros2_control.xacro" />
+    <xacro:if value="${sim_ignition or sim_gazebo}">
+      <xacro:property name="ros2_control_name" value="IgnitionSystem"/>
+    </xacro:if>
+     <xacro:if value="${use_fake_hardware}">
+      <xacro:property name="ros2_control_name" value="GenericSystem"/>
+    </xacro:if>
+    <xacro:unless value="${use_fake_hardware or sim_ignition or sim_gazebo}">
+      <xacro:property name="ros2_control_name" value="${prefix}KortexMultiInterfaceHardware"/>
+    </xacro:unless>
+    <xacro:gripper_ros2_control
+      prefix="${prefix}"
+      use_fake_hardware="${use_fake_hardware}"
+      fake_sensor_commands="${fake_sensor_commands}"
+      sim_ignition="${sim_ignition}"
+      sim_isaac="${sim_isaac}"
+      isaac_joint_commands="${isaac_joint_commands}"
+      isaac_joint_states="${isaac_joint_states}"
+      tf_prefix=""/>
+<!-- Tool frame used by the arm -->
     <link name="${prefix}tool_frame"/>
     <joint name="${prefix}tool_frame_joint" type="fixed">
@@ -77,11 +97,10 @@
       <material>Kortex/Gray</material>
     </gazebo>
-    <!-- TODO(MarqRazz) look into why the joint and limits needed to be flipped and modified -->
     <joint name="${prefix}right_finger_bottom_joint" type="revolute">
-      <origin xyz="0 -0.030501 0.070003" rpy="1.571 0.611 1.571" />
+      <origin xyz="0 -0.030501 0.070003" rpy="0 1.5708 0" />
       <parent link="${prefix}gripper_base_link" />
       <child link="${prefix}right_finger_prox_link" />
-      <axis xyz="0 0 -1" />
-      <limit lower="0.0" upper="0.85" effort="50" velocity="0.6" />
+      <axis xyz="0 0 1" />
+      <limit lower="-0.09" upper="0.96" effort="1000" velocity="0.6" />
     </joint>
     <link name="${prefix}right_finger_dist_link">
@@ -116,5 +135,4 @@
       <axis xyz="0 0 1" />
       <limit lower="-0.50" upper="0.21" effort="1000" velocity="1000" /> <!--limit lower="-1.03" upper="0.21" effort="1000" velocity="1000" /-->
-      <mimic joint="${prefix}right_finger_bottom_joint" multiplier="-0.676" offset="0.149" />
     </joint>
     <link name="${prefix}left_finger_prox_link">
@@ -144,10 +162,9 @@
     </gazebo>
     <joint name="${prefix}left_finger_bottom_joint" type="revolute">
-      <origin xyz="0 0.0305 0.070003" rpy="-1.571 0.611 -1.571" />
+      <origin xyz="0 0.0305 0.070003" rpy="0 1.5708 0" />
       <parent link="${prefix}gripper_base_link" />
       <child link="${prefix}left_finger_prox_link" />
       <axis xyz="0 0 1" />
-      <limit lower="0.0" upper="0.85" effort="1000" velocity="1000" />
-      <mimic joint="${prefix}right_finger_bottom_joint" multiplier="1.0" offset="0.0" />
+      <limit lower="-0.96" upper="0.09" effort="1000" velocity="1000" />
     </joint>
     <link name="${prefix}left_finger_dist_link">
@@ -182,5 +199,4 @@
       <axis xyz="0 0 -1" />
       <limit lower="-0.50" upper="0.21" effort="1000" velocity="1000" /> <!--limit lower="-1.03" upper="0.21" effort="1000" velocity="1000" /-->
-      <mimic joint="${prefix}right_finger_bottom_joint" multiplier="-0.676" offset="0.149" />
     </joint>
   </xacro:macro>

File: kortex_description/robots/gen3_lite.urdf (robot description, URDF)
Before this commit: robot gen3_lite, 15 links, 14 joints
Joints:
- joint left_finger_bottom_joint: limit lower=0.0 upper=0.85 effort=1000 velocity=1000 -> lower=-0.96 upper=0.0 effort=1000 velocity=1000; mimic joint=right_finger_bottom_joint multiplier=1.0 offset=0.0 -> joint=right_finger_bottom_joint multiplier=-1.0 offset=0.0; origin xyz=0 0.0305 0.070003 rpy=-1.571 0.611 -1.571 -> xyz=0 0.0305 0.070003 rpy=0 1.5708 0
- joint right_finger_bottom_joint: axis 0 0 -1 -> 0 0 1; limit lower=0.0 upper=0.85 effort=50 velocity=0.6 -> lower=0.0 upper=0.96 effort=1000 velocity=0.6; origin xyz=0 -0.030501 0.070003 rpy=1.571 0.611 1.571 -> xyz=0 -0.030501 0.070003 rpy=0 1.5708 0

Commit message: Modifications to rectify the unintentional mess of the real-life robot control

File: kortex_description/arms/gen3_lite/6dof/urdf/kortex.ros2_control.xacro (robot description, xacro)
@@ -124,11 +124,11 @@
         <state_interface name="effort"/>
       </joint>
-      <!--
-      <joint name="${prefix}right_finger_bottom_joint">
-        <command_interface name="position"/>
-        <state_interface name="position"/>
-        <state_interface name="velocity"/>
-      </joint>
-      -->
+      <xacro:unless value="${use_fake_hardware or sim_isaac or sim_ignition}">
+        <joint name="${prefix}right_finger_bottom_joint">
+          <command_interface name="position"/>
+          <state_interface name="position"/>
+          <state_interface name="velocity"/>
+        </joint>
+      </xacro:unless>
     </ros2_control>
   </xacro:macro>

File: kortex_description/grippers/gen3_lite_2f/urdf/gen3_lite_2f_macro.xacro (robot description, xacro)
@@ -12,4 +12,5 @@
     isaac_joint_states:=/isaac_joint_states
     use_internal_bus_gripper_comm:=true">
+  <xacro:if value="${use_fake_hardware or sim_isaac or sim_ignition}">
   <!-- ros2 control include -->
     <xacro:include filename="$(find kortex_description)/grippers/gen3_lite_2f/urdf/gen3_lite_2f.ros2_control.xacro" />
@@ -200,4 +201,179 @@
       <limit lower="-0.50" upper="0.21" effort="1000" velocity="1000" /> <!--limit lower="-1.03" upper="0.21" effort="1000" velocity="1000" /-->
     </joint>
+  </xacro:if>
+  <xacro:unless value="${use_fake_hardware or sim_isaac or sim_ignition}">
+      <!-- Tool frame used by the arm -->
+    <link name="${prefix}tool_frame"/>
+    <joint name="${prefix}tool_frame_joint" type="fixed">
+        <origin xyz="0 0 0.130" rpy="0 0 1.57079632679" />
+        <parent link="${parent}" />
+        <child link="${prefix}tool_frame" />
+        <axis xyz="0 0 0" />
+    </joint>
+    <!-- Gripper description -->
+    <joint name="${prefix}gripper_base_joint" type="fixed">
+      <origin xyz="0 0 0" rpy="0 0 0" />
+      <parent link="${parent}" />
+      <child link="${prefix}gripper_base_link" />
+      <axis xyz="0 0 0" />
+    </joint>
+    <link name="${prefix}gripper_base_link">
+      <inertial>
+        <origin xyz="4.03E-06 1.08E-05 0.041397" rpy="0 0 0" />
+        <mass value="0.1395" />
+        <inertia ixx="0.00011614" ixy="1E-08" ixz="4E-08" iyy="0.00010327" iyz="0" izz="9.707E-05" />
+      </inertial>
+      <visual>
+        <origin xyz="0 0 0" rpy="0 0 0" />
+        <geometry>
+          <mesh filename="file://$(find kortex_description)/grippers/gen3_lite_2f/meshes/gripper_base_link.STL" />
+        </geometry>
+        <material name="">
+          <color rgba="0.803 0.824 0.820 1" />
+        </material>
+      </visual>
+      <collision>
+        <origin xyz="0 0 0" rpy="0 0 0" />
+        <geometry>
+          <mesh filename="file://$(find kortex_description)/grippers/gen3_lite_2f/meshes/gripper_base_link.STL" />
+        </geometry>
+      </collision>
+    </link>
+    <gazebo reference="${prefix}gripper_base_link">
+      <material>Kortex/Gray</material>
+    </gazebo>
+    <link name="${prefix}right_finger_prox_link">
+    <inertial>
+      <origin xyz="0.020257 0.0063483 6.991E-05" rpy="0 0 0" />
+      <mass value="0.018385" />
+      <inertia ixx="2.29E-06" ixy="1.43E-06" ixz="0" iyy="4.56E-06" iyz="0" izz="4.77E-06" />
+    </inertial>
+    <visual>
+      <origin xyz="0 0 0" rpy="0 0 0" />
+      <geometry>
+        <mesh filename="file://$(find kortex_description)/grippers/gen3_lite_2f/meshes/right_finger_prox_link.STL" />
+      </geometry>
+      <material name="">
+          <color rgba="0.803 0.824 0.820 1" />
+      </material>
+    </visual>
+    <collision>
+      <origin xyz="0 0 0" rpy="0 0 0" />
+      <geometry>
+        <mesh filename="file://$(find kortex_description)/grippers/gen3_lite_2f/meshes/right_finger_prox_link.STL" />
+      </geometry>
+    </collision>
+    </link>
+    <gazebo reference="${prefix}right_finger_prox_link">
+      <material>Kortex/Gray</material>
+    </gazebo>
+    <!-- TODO(MarqRazz) look into why the joint and limits needed to be flipped and modified -->
+    <joint name="${prefix}right_finger_bottom_joint" type="revolute">
+      <origin xyz="0 -0.030501 0.070003" rpy="1.571 0.611 1.571" />
+      <parent link="${prefix}gripper_base_link" />
+      <child link="${prefix}right_finger_prox_link" />
+      <axis xyz="0 0 -1" />
+      <limit lower="0.0" upper="0.85" effort="50" velocity="0.6" />
+    </joint>
+    <link name="${prefix}right_finger_dist_link">
+      <inertial>
+        <origin xyz="0.018488 0.0011091 0" rpy="0 0 0" />
+        <mass value="0.010748" />
+        <inertia ixx="6.3E-07" ixy="3.2E-07" ixz="0" iyy="1.83E-06" iyz="0" izz="1.61E-06" />
+      </inertial>
+      <visual>
+        <origin xyz="0 0 0" rpy="0 0 0" />
+        <geometry>
+          <mesh filename="file://$(find kortex_description)/grippers/gen3_lite_2f/meshes/right_finger_dist_link.STL" />
+        </geometry>
+        <material name="">
+          <color rgba="0 0.055 0.525 1" />
+        </material>
+      </visual>
+      <collision>
+        <origin xyz="0 0 0" rpy="0 0 0" />
+        <geometry>
+          <mesh filename="file://$(find kortex_description)/grippers/gen3_lite_2f/meshes/right_finger_dist_link.STL" />
+        </geometry>
+      </collision>
+    </link>
+    <gazebo reference="${prefix}right_finger_dist_link">
+      <material>Kortex/Blue</material>
+    </gazebo>
+    <joint name="${prefix}right_finger_tip_joint" type="revolute">
+      <origin xyz="-0.045636 0.020423 0" rpy="0 0 0" />
+      <parent link="${prefix}right_finger_prox_link" />
+      <child link="${prefix}right_finger_dist_link" />
+      <axis xyz="0 0 1" />
+      <limit lower="-0.50" upper="0.21" effort="1000" velocity="1000" /> <!--limit lower="-1.03" upper="0.21" effort="1000" velocity="1000" /-->
+      <mimic joint="${prefix}right_finger_bottom_joint" multiplier="-0.676" offset="0.149" />
+    </joint>
+    <link name="${prefix}left_finger_prox_link">
+      <inertial>
+        <origin xyz="0.020257 0.0063483 6.99E-05" rpy="0 0 0" />
+        <mass value="0.018385" />
+        <inertia ixx="2.29E-06" ixy="1.43E-06" ixz="0" iyy="4.56E-06" iyz="0" izz="4.77E-06" />
+      </inertial>
+      <visual>
+        <origin xyz="0 0 0" rpy="0 0 0" />
+        <geometry>
+          <mesh filename="file://$(find kortex_description)/grippers/gen3_lite_2f/meshes/left_finger_prox_link.STL" />
+        </geometry>
+        <material name="">
+          <color rgba="0.803 0.824 0.820 1" />
+        </material>
+      </visual>
+      <collision>
+        <origin xyz="0 0 0" rpy="0 0 0" />
+        <geometry>
+          <mesh filename="file://$(find kortex_description)/grippers/gen3_lite_2f/meshes/left_finger_prox_link.STL" />
+        </geometry>
+      </collision>
+    </link>
+    <gazebo reference="${prefix}left_finger_prox_link">
+      <material>Kortex/Gray</material>
+    </gazebo>
+    <joint name="${prefix}left_finger_bottom_joint" type="revolute">
+      <origin xyz="0 0.0305 0.070003" rpy="-1.571 0.611 -1.571" />
+      <parent link="${prefix}gripper_base_link" />
+      <child link="${prefix}left_finger_prox_link" />
+      <axis xyz="0 0 1" />
+      <limit lower="0.0" upper="0.85" effort="1000" velocity="1000" />
+      <mimic joint="${prefix}right_finger_bottom_joint" multiplier="1.0" offset="0.0" />
+    </joint>
+    <link name="${prefix}left_finger_dist_link">
+      <inertial>
+        <origin xyz="-0.018488 0.0011091 0" rpy="0 0 0" />
+        <mass value="0.010748" />
+        <inertia ixx="6.3E-07" ixy="3.2E-07" ixz="0" iyy="1.83E-06" iyz="0" izz="1.61E-06" />
+      </inertial>
+      <visual>
+        <origin xyz="0 0 0" rpy="0 0 0" />
+        <geometry>
+          <mesh filename="file://$(find kortex_description)/grippers/gen3_lite_2f/meshes/left_finger_dist_link.STL" />
+        </geometry>
+        <material name="">
+          <color rgba="0 0.055 0.525 1" />
+        </material>
+      </visual>
+      <collision>
+        <origin xyz="0 0 0" rpy="0 0 0" />
+        <geometry>
+          <mesh filename="file://$(find kortex_description)/grippers/gen3_lite_2f/meshes/left_finger_dist_link.STL" />
+        </geometry>
+      </collision>
+    </link>
+    <gazebo reference="${prefix}left_finger_dist_link">
+      <material>Kortex/Blue</material>
+    </gazebo>
+    <joint name="${prefix}left_finger_tip_joint" type="revolute">
+      <origin xyz="-0.045636 -0.020423 6.9901E-05" rpy="0 0 0" />
+      <parent link="${prefix}left_finger_prox_link" />
+      <child link="${prefix}left_finger_dist_link" />
+      <axis xyz="0 0 -1" />
+      <limit lower="-0.50" upper="0.21" effort="1000" velocity="1000" /> <!--limit lower="-1.03" upper="0.21" effort="1000" velocity="1000" /-->
+      <mimic joint="${prefix}right_finger_bottom_joint" multiplier="-0.676" offset="0.149" />
+    </joint>
+  </xacro:unless>
   </xacro:macro>
 </robot>

Commit message: Other renames

File: kortex_description/arms/gen3_lite/6dof/urdf/kortex.ros2_control.xacro (robot description, xacro)
@@ -144,5 +144,5 @@
         <state_interface name="effort"/>
       </joint>
-      <xacro:unless value="${use_fake_hardware or sim_isaac or sim_ignition}">
+      <xacro:unless value="${use_fake_hardware or sim_isaac or sim_gazebo}">
         <xacro:unless value="${moveit_active}">
           <joint name="${prefix}right_finger_bottom_joint">

File: kortex_description/grippers/gen3_lite_2f/urdf/gen3_lite_2f_macro.xacro (robot description, xacro)
@@ -13,15 +13,15 @@
     use_internal_bus_gripper_comm:=true
     moveit_active:=false">
-  <xacro:if value="${use_fake_hardware or sim_isaac or sim_ignition}">
+  <xacro:if value="${use_fake_hardware or sim_isaac or sim_gazebo}">
     <xacro:unless value="${moveit_active}">
     <!-- ros2 control include -->
       <xacro:include filename="$(find kortex_description)/grippers/gen3_lite_2f/urdf/gen3_lite_2f.ros2_control.xacro" />
-      <xacro:if value="${sim_ignition or sim_gazebo}">
-        <xacro:property name="ros2_control_name" value="IgnitionSystem"/>
+      <xacro:if value="${sim_gazebo}">
+        <xacro:property name="ros2_control_name" value="GazeboSimSystem"/>
       </xacro:if>
       <xacro:if value="${use_fake_hardware}">
         <xacro:property name="ros2_control_name" value="GenericSystem"/>
       </xacro:if>
-      <xacro:unless value="${use_fake_hardware or sim_ignition or sim_gazebo}">
+      <xacro:unless value="${use_fake_hardware or sim_gazebo}">
         <xacro:property name="ros2_control_name" value="${prefix}KortexMultiInterfaceHardware"/>
       </xacro:unless>
@@ -30,5 +30,5 @@
         use_fake_hardware="${use_fake_hardware}"
         fake_sensor_commands="${fake_sensor_commands}"
-        sim_ignition="${sim_ignition}"
+        sim_gazebo="${sim_gazebo}"
         sim_isaac="${sim_isaac}"
         isaac_joint_commands="${isaac_joint_commands}"
@@ -207,5 +207,5 @@
     </xacro:unless>
   </xacro:if>
-  <xacro:unless value="${use_fake_hardware or sim_isaac or sim_ignition}">
+  <xacro:unless value="${use_fake_hardware or sim_isaac or sim_gazebo}">
     <xacro:unless value="${moveit_active}">
         <!-- Tool frame used by the arm -->

Commit message: Modifications to fix moveit issues while controlling Gen3_lite

File: kortex_description/arms/gen3_lite/6dof/urdf/kortex.ros2_control.xacro (robot description, xacro)
@@ -153,5 +153,5 @@
         </xacro:unless>
       </xacro:unless>
-      <xacro:if value="${moveit_active}">
+      <!--<xacro:if value="${moveit_active}">-->
         <joint name="${prefix}right_finger_bottom_joint">
           <command_interface name="position"/>
@@ -159,5 +159,5 @@
           <state_interface name="velocity"/>
         </joint>
-      </xacro:if>
+      <!--</xacro:if>-->
     </ros2_control>
   </xacro:macro>

File: kortex_description/grippers/gen3_lite_2f/urdf/gen3_lite_2f_macro.xacro (robot description, xacro)
@@ -139,4 +139,5 @@
         <axis xyz="0 0 1" />
         <limit lower="-0.50" upper="0.21" effort="1000" velocity="1000" /> <!--limit lower="-1.03" upper="0.21" effort="1000" velocity="1000" /-->
+        <mimic joint="${prefix}right_finger_bottom_joint" multiplier="-0.276" offset="-0.1" />
       </joint>
       <link name="${prefix}left_finger_prox_link">
@@ -172,4 +173,5 @@
         <limit lower="-0.96" upper="0.09" effort="10" velocity="0.6" />
         <dynamics damping="0.1" friction="1"/>
+        <mimic joint="${prefix}right_finger_bottom_joint" multiplier="-1.0" offset="0.0" />
       </joint>
       <link name="${prefix}left_finger_dist_link">
@@ -204,4 +206,5 @@
         <axis xyz="0 0 -1" />
         <limit lower="-0.50" upper="0.21" effort="1000" velocity="1000" /> <!--limit lower="-1.03" upper="0.21" effort="1000" velocity="1000" /-->
+        <mimic joint="${prefix}right_finger_bottom_joint" multiplier="-0.276" offset="-0.1" />
       </joint>
     </xacro:unless>

Commit message: fixed gen3_lite moveit issues

File: kortex_description/arms/gen3_lite/6dof/urdf/kortex.ros2_control.xacro (robot description, xacro)
@@ -144,6 +144,7 @@
         <state_interface name="effort"/>
       </joint>
-      <xacro:unless value="${use_fake_hardware or sim_isaac or sim_gazebo}">
-        <xacro:unless value="${moveit_active}">
+      <!--<xacro:unless value="${use_fake_hardware or sim_isaac or sim_gazebo}">-->
+        <!--<xacro:unless value="${moveit_active}">-->
+        <!--
           <joint name="${prefix}right_finger_bottom_joint">
             <command_interface name="position"/>
@@ -151,6 +152,7 @@
             <state_interface name="velocity"/>
           </joint>
-        </xacro:unless>
-      </xacro:unless>
+        -->
+       <!-- </xacro:unless> -->
+      <!-- </xacro:unless> -->
       <!--<xacro:if value="${moveit_active}">-->
         <joint name="${prefix}right_finger_bottom_joint">

File: kortex_description/grippers/gen3_lite_2f/urdf/gen3_lite_2f_macro.xacro (robot description, xacro)
@@ -101,9 +101,9 @@
       </gazebo>
       <joint name="${prefix}right_finger_bottom_joint" type="revolute">
-        <origin xyz="0 -0.030501 0.070003" rpy="0 1.5708 0" />
+        <origin xyz="0 -0.030501 0.070003" rpy="1.571 0.611 1.571" />
         <parent link="${prefix}gripper_base_link" />
         <child link="${prefix}right_finger_prox_link" />
-        <axis xyz="0 0 1" />
-        <limit lower="-0.09" upper="0.96" effort="10" velocity="0.6" />
+        <axis xyz="0 0 -1" />
+        <limit lower="-0.1" upper="0.96" effort="10" velocity="0.6" />
         <dynamics damping="0.1" friction="1"/>
       </joint>
@@ -167,11 +167,11 @@
       </gazebo>
       <joint name="${prefix}left_finger_bottom_joint" type="revolute">
-        <origin xyz="0 0.0305 0.070003" rpy="0 1.5708 0" />
+        <origin xyz="0 0.0305 0.070003" rpy="-1.571 0.611 -1.571" />
         <parent link="${prefix}gripper_base_link" />
         <child link="${prefix}left_finger_prox_link" />
         <axis xyz="0 0 1" />
-        <limit lower="-0.96" upper="0.09" effort="10" velocity="0.6" />
+        <limit lower="-0.1" upper="0.96" effort="10" velocity="0.6" />
         <dynamics damping="0.1" friction="1"/>
-        <mimic joint="${prefix}right_finger_bottom_joint" multiplier="-1.0" offset="0.0" />
+        <mimic joint="${prefix}right_finger_bottom_joint" multiplier="1.0" offset="0.0" />
       </joint>
       <link name="${prefix}left_finger_dist_link">
