Commit message: reverse gripper joints in URDF

File: kortex_description/grippers/gen3_lite_2f/urdf/gen3_lite_2f_macro.xacro (robot description, xacro)
@@ -67,10 +67,11 @@
       <material>Kortex/Gray</material>
     </gazebo>
+    <!-- TODO(MarqRazz) look into why the joint and limits needed to be flipped and modified -->
     <joint name="${prefix}right_finger_bottom_joint" type="revolute">
-      <origin xyz="0 -0.030501 0.070003" rpy="0 1.5708 0" />
+      <origin xyz="0 -0.030501 0.070003" rpy="1.571 0.611 1.571" />
       <parent link="${prefix}gripper_base_link" />
       <child link="${prefix}right_finger_prox_link" />
-      <axis xyz="0 0 1" />
-      <limit lower="-0.09" upper="0.96" effort="1000" velocity="0.6" />
+      <axis xyz="0 0 -1" />
+      <limit lower="0.0" upper="0.85" effort="1000" velocity="0.6" />
     </joint>
     <link name="${prefix}right_finger_dist_link">
@@ -133,10 +134,10 @@
     </gazebo>
     <joint name="${prefix}left_finger_bottom_joint" type="revolute">
-      <origin xyz="0 0.0305 0.070003" rpy="0 1.5708 0" />
+      <origin xyz="0 0.0305 0.070003" rpy="-1.571 0.611 -1.571" />
       <parent link="${prefix}gripper_base_link" />
       <child link="${prefix}left_finger_prox_link" />
       <axis xyz="0 0 1" />
-      <limit lower="-0.96" upper="0.09" effort="1000" velocity="1000" />
-      <mimic joint="${prefix}right_finger_bottom_joint" multiplier="-1.0" offset="0.0" />
+      <limit lower="0.0" upper="0.85" effort="1000" velocity="1000" />
+      <mimic joint="${prefix}right_finger_bottom_joint" multiplier="1.0" offset="0.0" />
     </joint>
     <link name="${prefix}left_finger_dist_link">

Commit message: Fixed the Gen3_Lite_fingers closing motion

File: kortex_description/grippers/gen3_lite_2f/urdf/gen3_lite_2f_macro.xacro (robot description, xacro)
@@ -105,5 +105,6 @@
         <child link="${prefix}right_finger_prox_link" />
         <axis xyz="0 0 1" />
-        <limit lower="-0.09" upper="0.96" effort="1000" velocity="0.6" />
+        <limit lower="-0.09" upper="0.96" effort="10" velocity="0.6" />
+        <dynamics damping="0.1" friction="1"/>
       </joint>
       <link name="${prefix}right_finger_dist_link">
@@ -169,5 +170,6 @@
         <child link="${prefix}left_finger_prox_link" />
         <axis xyz="0 0 1" />
-        <limit lower="-0.96" upper="0.09" effort="1000" velocity="1000" />
+        <limit lower="-0.96" upper="0.09" effort="10" velocity="0.6" />
+        <dynamics damping="0.1" friction="1"/>
       </joint>
       <link name="${prefix}left_finger_dist_link">

Commit message: Rectified the mimiced fingertip joints angles for a better rviz visualization

File: kortex_description/grippers/gen3_lite_2f/urdf/gen3_lite_2f_macro.xacro (robot description, xacro)
@@ -313,5 +313,5 @@
         <axis xyz="0 0 1" />
         <limit lower="-0.50" upper="0.21" effort="1000" velocity="1000" /> <!--limit lower="-1.03" upper="0.21" effort="1000" velocity="1000" /-->
-        <mimic joint="${prefix}right_finger_bottom_joint" multiplier="-0.676" offset="0.149" />
+        <mimic joint="${prefix}right_finger_bottom_joint" multiplier="-0.276" offset="-0.1" />
       </joint>
       <link name="${prefix}left_finger_prox_link">
@@ -379,5 +379,5 @@
         <axis xyz="0 0 -1" />
         <limit lower="-0.50" upper="0.21" effort="1000" velocity="1000" /> <!--limit lower="-1.03" upper="0.21" effort="1000" velocity="1000" /-->
-        <mimic joint="${prefix}right_finger_bottom_joint" multiplier="-0.676" offset="0.149" />
+        <mimic joint="${prefix}right_finger_bottom_joint" multiplier="-0.276" offset="-0.1" />
       </joint>
     </xacro:unless>

Commit message: Update gen3_lite_2f_macro.xacro

File: kortex_description/grippers/gen3_lite_2f/urdf/gen3_lite_2f_macro.xacro (robot description, xacro)
@@ -59,5 +59,5 @@
           <origin xyz="0 0 0" rpy="0 0 0" />
           <geometry>
-            <mesh filename="file://$(find kortex_description)/grippers/gen3_lite_2f/meshes/gripper_base_link.STL" />
+            <mesh filename="package://kortex_description/grippers/gen3_lite_2f/meshes/gripper_base_link.STL" />
           </geometry>
           <material name="">
@@ -68,5 +68,5 @@
           <origin xyz="0 0 0" rpy="0 0 0" />
           <geometry>
-            <mesh filename="file://$(find kortex_description)/grippers/gen3_lite_2f/meshes/gripper_base_link.STL" />
+            <mesh filename="package://kortex_description/grippers/gen3_lite_2f/meshes/gripper_base_link.STL" />
           </geometry>
         </collision>
@@ -84,5 +84,5 @@
         <origin xyz="0 0 0" rpy="0 0 0" />
         <geometry>
-          <mesh filename="file://$(find kortex_description)/grippers/gen3_lite_2f/meshes/right_finger_prox_link.STL" />
+          <mesh filename="package://kortex_description/grippers/gen3_lite_2f/meshes/right_finger_prox_link.STL" />
         </geometry>
         <material name="">
@@ -93,5 +93,5 @@
         <origin xyz="0 0 0" rpy="0 0 0" />
         <geometry>
-          <mesh filename="file://$(find kortex_description)/grippers/gen3_lite_2f/meshes/right_finger_prox_link.STL" />
+          <mesh filename="package://kortex_description/grippers/gen3_lite_2f/meshes/right_finger_prox_link.STL" />
         </geometry>
       </collision>
@@ -117,5 +117,5 @@
           <origin xyz="0 0 0" rpy="0 0 0" />
           <geometry>
-            <mesh filename="file://$(find kortex_description)/grippers/gen3_lite_2f/meshes/right_finger_dist_link.STL" />
+            <mesh filename="package://kortex_description/grippers/gen3_lite_2f/meshes/right_finger_dist_link.STL" />
           </geometry>
           <material name="">
@@ -126,5 +126,5 @@
           <origin xyz="0 0 0" rpy="0 0 0" />
           <geometry>
-            <mesh filename="file://$(find kortex_description)/grippers/gen3_lite_2f/meshes/right_finger_dist_link.STL" />
+            <mesh filename="package://kortex_description/grippers/gen3_lite_2f/meshes/right_finger_dist_link.STL" />
           </geometry>
         </collision>
@@ -149,5 +149,5 @@
           <origin xyz="0 0 0" rpy="0 0 0" />
           <geometry>
-            <mesh filename="file://$(find kortex_description)/grippers/gen3_lite_2f/meshes/left_finger_prox_link.STL" />
+            <mesh filename="package://kortex_description/grippers/gen3_lite_2f/meshes/left_finger_prox_link.STL" />
           </geometry>
           <material name="">
@@ -158,5 +158,5 @@
           <origin xyz="0 0 0" rpy="0 0 0" />
           <geometry>
-            <mesh filename="file://$(find kortex_description)/grippers/gen3_lite_2f/meshes/left_finger_prox_link.STL" />
+            <mesh filename="package://kortex_description/grippers/gen3_lite_2f/meshes/left_finger_prox_link.STL" />
           </geometry>
         </collision>
@@ -182,5 +182,5 @@
           <origin xyz="0 0 0" rpy="0 0 0" />
           <geometry>
-            <mesh filename="file://$(find kortex_description)/grippers/gen3_lite_2f/meshes/left_finger_dist_link.STL" />
+            <mesh filename="package://kortex_description/grippers/gen3_lite_2f/meshes/left_finger_dist_link.STL" />
           </geometry>
           <material name="">
@@ -191,5 +191,5 @@
           <origin xyz="0 0 0" rpy="0 0 0" />
           <geometry>
-            <mesh filename="file://$(find kortex_description)/grippers/gen3_lite_2f/meshes/left_finger_dist_link.STL" />
+            <mesh filename="package://kortex_description/grippers/gen3_lite_2f/meshes/left_finger_dist_link.STL" />
           </geometry>
         </collision>
@@ -233,5 +233,5 @@
           <origin xyz="0 0 0" rpy="0 0 0" />
           <geometry>
-            <mesh filename="file://$(find kortex_description)/grippers/gen3_lite_2f/meshes/gripper_base_link.STL" />
+            <mesh filename="package://kortex_description/grippers/gen3_lite_2f/meshes/gripper_base_link.STL" />
           </geometry>
           <material name="">
@@ -242,5 +242,5 @@
           <origin xyz="0 0 0" rpy="0 0 0" />
           <geometry>
-            <mesh filename="file://$(find kortex_description)/grippers/gen3_lite_2f/meshes/gripper_base_link.STL" />
+            <mesh filename="package://kortex_description/grippers/gen3_lite_2f/meshes/gripper_base_link.STL" />
           </geometry>
         </collision>
@@ -258,5 +258,5 @@
         <origin xyz="0 0 0" rpy="0 0 0" />
         <geometry>
-          <mesh filename="file://$(find kortex_description)/grippers/gen3_lite_2f/meshes/right_finger_prox_link.STL" />
+          <mesh filename="package://kortex_description/grippers/gen3_lite_2f/meshes/right_finger_prox_link.STL" />
         </geometry>
         <material name="">
@@ -267,5 +267,5 @@
         <origin xyz="0 0 0" rpy="0 0 0" />
         <geometry>
-          <mesh filename="file://$(find kortex_description)/grippers/gen3_lite_2f/meshes/right_finger_prox_link.STL" />
+          <mesh filename="package://kortex_description/grippers/gen3_lite_2f/meshes/right_finger_prox_link.STL" />
         </geometry>
       </collision>
@@ -291,5 +291,5 @@
           <origin xyz="0 0 0" rpy="0 0 0" />
           <geometry>
-            <mesh filename="file://$(find kortex_description)/grippers/gen3_lite_2f/meshes/right_finger_dist_link.STL" />
+            <mesh filename="package://kortex_description/grippers/gen3_lite_2f/meshes/right_finger_dist_link.STL" />
           </geometry>
           <material name="">
@@ -300,5 +300,5 @@
           <origin xyz="0 0 0" rpy="0 0 0" />
           <geometry>
-            <mesh filename="file://$(find kortex_description)/grippers/gen3_lite_2f/meshes/right_finger_dist_link.STL" />
+            <mesh filename="package://kortex_description/grippers/gen3_lite_2f/meshes/right_finger_dist_link.STL" />
           </geometry>
         </collision>
@@ -324,5 +324,5 @@
           <origin xyz="0 0 0" rpy="0 0 0" />
           <geometry>
-            <mesh filename="file://$(find kortex_description)/grippers/gen3_lite_2f/meshes/left_finger_prox_link.STL" />
+            <mesh filename="package://kortex_description/grippers/gen3_lite_2f/meshes/left_finger_prox_link.STL" />
           </geometry>
           <material name="">
@@ -333,5 +333,5 @@
           <origin xyz="0 0 0" rpy="0 0 0" />
           <geometry>
-            <mesh filename="file://$(find kortex_description)/grippers/gen3_lite_2f/meshes/left_finger_prox_link.STL" />
+            <mesh filename="package://kortex_description/grippers/gen3_lite_2f/meshes/left_finger_prox_link.STL" />
           </geometry>
         </collision>
@@ -357,5 +357,5 @@
           <origin xyz="0 0 0" rpy="0 0 0" />
           <geometry>
-            <mesh filename="file://$(find kortex_description)/grippers/gen3_lite_2f/meshes/left_finger_dist_link.STL" />
+            <mesh filename="package://kortex_description/grippers/gen3_lite_2f/meshes/left_finger_dist_link.STL" />
           </geometry>
           <material name="">
@@ -366,5 +366,5 @@
           <origin xyz="0 0 0" rpy="0 0 0" />
           <geometry>
-            <mesh filename="file://$(find kortex_description)/grippers/gen3_lite_2f/meshes/left_finger_dist_link.STL" />
+            <mesh filename="package://kortex_description/grippers/gen3_lite_2f/meshes/left_finger_dist_link.STL" />
           </geometry>
         </collision>
